Commit message: Added torso laser
git-svn-id: https://roboticssrv.wtb.tue.nl/svn/ros/code/tue-ros-pkg/trunk/amigo2_common/amigo2_description@18272 3a3c2cfb-d3b9-409e-9e75-db8fcdbcaac6

File: urdf/xacro/arms/arm.urdf.xacro (robot description, xacro)
@@ -38,5 +38,5 @@
 </xacro:my_link>
 <!--the upper arm-->
-<xacro:my_link_texturedmesh name="upper_arm_${whichside}" mass="2.95" texture="amigo_description/white">
+<xacro:my_link_texturedmesh name="upper_arm_${whichside}" mass="2.95" texture="white">
    <origin xyz="0.0 -0.2 0.0" rpy="0 0 0"/>
    <origin xyz="-0.00959 -0.19131 -0.00001" rpy="0 0 3.1415" />
@@ -53,5 +53,5 @@
 </xacro:my_link>
 <!--the forearm-->
-<xacro:my_link_texturedmesh name="fore_arm_${whichside}" mass="0.85" texture="amigo_description/white">
+<xacro:my_link_texturedmesh name="fore_arm_${whichside}" mass="0.85" texture="white">
    <origin xyz="0.0 -0.14 0.0" rpy="0.0 0 0"/>
    <origin xyz="0.00425 -0.14868 0.00547" rpy="0 -1.5708 0" />

File: urdf/xacro/kinect/top_kinect.urdf.xacro (robot description, xacro)
@@ -21,7 +21,7 @@
       <origin xyz=" 0 0 0 " rpy="0 0 0" />
       <geometry>
-		<box size="0.001 0.001 0.001"/><!--Changed to 0.001 because otherwise it doesn't work-->
+		<!--<box size="0.001 0.001 0.001"/>--><!--Changed to 0.001 because otherwise it doesn't work-->
         <!--mesh filename="package://amigo_description/kinect/meshes/kinect.dae" scale="0.001 0.001 0.001"/-->
-        <!--<mesh filename="package://amigo2_description/kinect/meshes/kinect_without_base.dae"/>-->
+        <mesh filename="package://amigo2_description/media/meshes/kinect_without_base.dae"/>
       </geometry>
     </visual>

File: urdf/xacro/robot.urdf.xacro (robot description, xacro)
@@ -30,3 +30,4 @@
     <!--========BUILD LASER======-->
     <include filename="$(find amigo2_description)/urdf/xacro/laser/laser.urdf.xacro" />
+    <include filename="$(find amigo2_description)/urdf/xacro/laser/torso_laser.urdf.xacro" />
 </robot>
