Commit message: Fixed joint limits
git-svn-id: https://roboticssrv.wtb.tue.nl/svn/ros/code/tue-ros-pkg/trunk/amigo2_common/amigo2_description@18649 3a3c2cfb-d3b9-409e-9e75-db8fcdbcaac6

File: urdf/amigo2.urdf (robot description, URDF)
Before this commit: robot amigo, 56 links, 55 joints
Joints:
- joint ankle_joint: limit lower=0.0 upper=1.57 effort=13.4 velocity=1.0 -> lower=0.0 upper=1.57 effort=1000 velocity=10
- joint hip_joint: limit lower=0.0 upper=1.57 effort=13.4 velocity=1.0 -> lower=0.0 upper=1.57 effort=1000 velocity=10
- joint knee_joint: limit lower=0.0 upper=1.57 effort=13.4 velocity=1.0 -> lower=0.0 upper=1.57 effort=1000 velocity=10

File: urdf/xacro/torso/torso.urdf.xacro (robot description, xacro)
@@ -42,5 +42,5 @@
         <dynamics damping="6.0" friction="4.87"/><!-- ToDo: adjust dynamics-->
         <axis xyz="0 -1 0"/><!--ToDo: DH parameters?-->
-        <limit effort="13.4" velocity="1.0" lower="0.0" upper="1.57" /> <!--ToDo: adjust parameters-->
+        <limit effort="1000" velocity="10" lower="0.0" upper="1.57" /> <!--ToDo: adjust parameters-->
     </xacro:my_joint>
     <xacro:my_joint name="knee_joint" type="revolute" parent="lower_rear_leg" child="upper_leg">
@@ -48,5 +48,5 @@
         <dynamics damping="6.0" friction="4.87"/><!-- ToDo: adjust dynamics-->
         <axis xyz="0 -1 0"/><!--ToDo: DH parameters?-->
-        <limit effort="13.4" velocity="1.0" lower="0.0" upper="1.57" /> <!--ToDo: adjust parameters-->
+        <limit effort="1000" velocity="10" lower="0.0" upper="1.57" /> <!--ToDo: adjust parameters-->
     </xacro:my_joint>
     <xacro:my_joint name="hip_joint" type="revolute" parent="upper_leg" child="trunk">
@@ -54,5 +54,5 @@
         <dynamics damping="6.0" friction="4.87"/><!-- ToDo: adjust dynamics-->
         <axis xyz="0 -1 0"/><!--ToDo: DH parameters?-->
-        <limit effort="13.4" velocity="1.0" lower="0.0" upper="1.57" /> <!--ToDo: adjust parameters-->
+        <limit effort="1000" velocity="10" lower="0.0" upper="1.57" /> <!--ToDo: adjust parameters-->
     </xacro:my_joint>
 </robot>

Commit message: amigo2 now has head
git-svn-id: https://roboticssrv.wtb.tue.nl/svn/ros/code/tue-ros-pkg/trunk/amigo2_common/amigo2_description@18651 3a3c2cfb-d3b9-409e-9e75-db8fcdbcaac6

File: urdf/amigo2.urdf (robot description, URDF)
Before this commit: robot amigo, 56 links, 55 joints
Links:
- link lower_rear_leg: mass 0.1 -> 5
- link trunk: mass 0.1 -> 10
- link upper_leg: mass 0.1 -> 5
Joints:
- joint head_mount_joint: origin xyz=0.6 0.0 0.0 rpy=3.14 0.0 0.0 -> xyz=0.5 0.0 0.0 rpy=3.14 0.0 0.0

File: urdf/xacro/head/head.urdf.xacro (robot description, xacro)
@@ -17,5 +17,5 @@
   <child link="head_mount"/>
   <axis xyz="0 0 1"/>
-  <origin xyz="0.6 0.0 0.0" rpy="3.14 0.0 0.0"/><!-- Check length -->
+  <origin xyz="0.5 0.0 0.0" rpy="3.14 0.0 0.0"/><!-- Check length -->
 </joint>
 <!-- the link that represents the panning part of the neck, is below neck_tilt -->

File: urdf/xacro/torso/torso.urdf.xacro (robot description, xacro)
@@ -12,5 +12,5 @@
     </xacro:my_link>
     <!-- Lower rear leg -->
-    <xacro:my_link name="lower_rear_leg" mass="0.1" color="White"><!--ToDo: estimate mass-->
+    <xacro:my_link name="lower_rear_leg" mass="5" color="White"><!--ToDo: estimate mass-->
         <box size="0.390 0.200 0.05" /><!--ToDo: check dimensions, adjust height-->
         <origin xyz="0.195 0.0 0.0" rpy="0 0 0"/><!--ToDo: check dimensions, adjust height-->
@@ -19,5 +19,5 @@
     </xacro:my_link>
     <!-- Upper leg (part from lower rear leg joint to trunk joint) -->
-    <xacro:my_link name="upper_leg" mass="0.1" color="White"><!--ToDo: estimate mass-->
+    <xacro:my_link name="upper_leg" mass="5" color="White"><!--ToDo: estimate mass-->
         <box size="0.4115 0.200 0.1" /><!--ToDo: check dimensions, adjust height-->
         <origin xyz="0.20575 0.0 0.0" rpy="0 0 0"/><!--ToDo: check dimensions, adjust height-->
@@ -26,5 +26,5 @@
     </xacro:my_link>
     <!-- Trunk -->
-    <xacro:my_link name="trunk" mass="0.1" color="White"><!--ToDo: estimate mass-->
+    <xacro:my_link name="trunk" mass="10" color="White"><!--ToDo: estimate mass-->
         <box size="0.445 0.200 0.15" /><!--ToDo: check dimensions, adjust height-->
         <origin xyz="0.2225 0.0 0.0" rpy="0 0 0"/><!--ToDo: check dimensions, adjust height-->

Commit message: Temporarily fixed torso joints
git-svn-id: https://roboticssrv.wtb.tue.nl/svn/ros/code/tue-ros-pkg/trunk/amigo2_common/amigo2_description@19531 3a3c2cfb-d3b9-409e-9e75-db8fcdbcaac6

File: urdf/amigo2.urdf (robot description, URDF)
Before this commit: robot amigo, 56 links, 55 joints
Joints:
- joint ankle_joint: limit lower=0.0 upper=1.57 effort=1000 velocity=10 -> lower=0.87 upper=0.87 effort=1000 velocity=10
- joint hip_joint: limit lower=0.0 upper=1.57 effort=1000 velocity=10 -> lower=2.36 upper=2.36 effort=1000 velocity=10
- joint knee_joint: limit lower=0.0 upper=1.57 effort=1000 velocity=10 -> lower=2.0 upper=2.0 effort=1000 velocity=10

File: urdf/xacro/torso/torso.urdf.xacro (robot description, xacro)
@@ -42,5 +42,6 @@
         <dynamics damping="6.0" friction="4.87"/><!-- ToDo: adjust dynamics-->
         <axis xyz="0 -1 0"/><!--ToDo: DH parameters?-->
-        <limit effort="1000" velocity="10" lower="0.0" upper="1.57" /> <!--ToDo: adjust parameters-->
+        <!--<limit effort="1000" velocity="10" lower="0.0" upper="1.57" />--> <!--ToDo: adjust parameters-->
+        <limit effort="1000" velocity="10" lower="0.87" upper="0.87" /> <!--TEMP: fixed joint positions until control is fixed-->
     </xacro:my_joint>
     <xacro:my_joint name="knee_joint" type="revolute" parent="lower_rear_leg" child="upper_leg">
@@ -48,5 +49,6 @@
         <dynamics damping="6.0" friction="4.87"/><!-- ToDo: adjust dynamics-->
         <axis xyz="0 -1 0"/><!--ToDo: DH parameters?-->
-        <limit effort="1000" velocity="10" lower="0.0" upper="1.57" /> <!--ToDo: adjust parameters-->
+        <!--<limit effort="1000" velocity="10" lower="0.0" upper="1.57" />--> <!--ToDo: adjust parameters -->
+        <limit effort="1000" velocity="10" lower="2.0" upper="2.0" /> <!--TEMP: fixed joint positions until control is fixed -->
     </xacro:my_joint>
     <xacro:my_joint name="hip_joint" type="revolute" parent="upper_leg" child="trunk">
@@ -54,5 +56,6 @@
         <dynamics damping="6.0" friction="4.87"/><!-- ToDo: adjust dynamics-->
         <axis xyz="0 -1 0"/><!--ToDo: DH parameters?-->
-        <limit effort="1000" velocity="10" lower="0.0" upper="1.57" /> <!--ToDo: adjust parameters-->
+        <!--<limit effort="1000" velocity="10" lower="0.0" upper="1.57" />--> <!--ToDo: adjust parameters -->
+        <limit effort="1000" velocity="10" lower="2.36" upper="2.36" /> <!--TEMP: fixed joint positions until control is fixed-->
     </xacro:my_joint>
 </robot>
