Commit message: Did some more renaming
git-svn-id: https://roboticssrv.wtb.tue.nl/svn/ros/code/tue-ros-pkg/trunk/sergio_common/sergio_description@25341 3a3c2cfb-d3b9-409e-9e75-db8fcdbcaac6

File: urdf/sergio.urdf (robot description, URDF)
Before this commit: robot sergio, 56 links, 55 joints
Links:
- link top_kinect/openni_camera: geometry visual mesh filename=package://sergio_description/media/meshes/kinect_without_ba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

File: urdf/xacro/gazebo.urdf.xacro (robot description, xacro)
@@ -208,12 +208,12 @@
 <gazebo>
     <plugin name="position_controller" filename="libPositionController.so">
-		<package>amigo2_description</package>
+		<package>sergio_description</package>
 		<group_summary_file>custom/joint_groups.yaml</group_summary_file>
     </plugin>
-    <plugin name="base_controller" filename="libAmigo2BaseController.so">
-		<package>amigo2_controller_configuration_gazebo</package>
+    <plugin name="base_controller" filename="libSergioBaseController.so">
+		<package>sergio_controller_configuration_gazebo</package>
 		<parameter_file>/parameters/base_controller.yaml</parameter_file>
 		<node_namespace>base</node_namespace>
-        <odomTopic>odom</odomTopic>
+        <odomTopic>/sergio/base/measurements</odomTopic>
     </plugin>
 </gazebo>

File: urdf/xacro/kinect/top_kinect.urdf.xacro (robot description, xacro)
@@ -23,5 +23,5 @@
 		<!--<box size="0.001 0.001 0.001"/>--><!--Changed to 0.001 because otherwise it doesn't work-->
         <!--mesh filename="package://amigo_description/kinect/meshes/kinect.dae" scale="0.001 0.001 0.001"/-->
-        <mesh filename="package://amigo2_description/media/meshes/kinect_without_base.dae"/>
+        <mesh filename="package://sergio_description/media/meshes/kinect_without_base.dae"/>
       </geometry>
     </visual>

Commit message: Torso joints are now in control
git-svn-id: https://roboticssrv.wtb.tue.nl/svn/ros/code/tue-ros-pkg/trunk/sergio_common/sergio_description@25378 3a3c2cfb-d3b9-409e-9e75-db8fcdbcaac6

File: urdf/sergio.urdf (robot description, URDF)
Before this commit: robot sergio, 56 links, 55 joints
Joints:
- joint ankle_joint: limit lower=0.87 upper=0.87 effort=1000 velocity=10 -> lower=0.0 upper=1.059 effort=1000 velocity=0.264
- joint hip_joint: limit lower=2.36 upper=2.36 effort=1000 velocity=10 -> lower=0.85 upper=2.36 effort=1000 velocity=0.375
- joint knee_joint: limit lower=2.0 upper=2.0 effort=1000 velocity=10 -> lower=0.0 upper=2.158 effort=1000 velocity=0.539

File: urdf/xacro/torso/torso.urdf.xacro (robot description, xacro)
@@ -42,6 +42,6 @@
         <dynamics damping="6.0" friction="4.87"/><!-- ToDo: adjust dynamics-->
         <axis xyz="0 -1 0"/><!--ToDo: DH parameters?-->
-        <!--<limit effort="1000" velocity="10" lower="0.0" upper="1.57" />--> <!--ToDo: adjust parameters-->
-        <limit effort="1000" velocity="10" lower="0.87" upper="0.87" /> <!--TEMP: fixed joint positions until control is fixed-->
+        <limit effort="1000" velocity="0.265" lower="0.0" upper="1.059" /> <!--ToDo: adjust parameters-->
+        <!--<limit effort="1000" velocity="10" lower="0.87" upper="0.87" />--> <!--TEMP: fixed joint positions until control is fixed-->
     </xacro:my_joint>
     <xacro:my_joint name="knee_joint" type="revolute" parent="lower_rear_leg" child="upper_leg">
@@ -49,6 +49,6 @@
         <dynamics damping="6.0" friction="4.87"/><!-- ToDo: adjust dynamics-->
         <axis xyz="0 -1 0"/><!--ToDo: DH parameters?-->
-        <!--<limit effort="1000" velocity="10" lower="0.0" upper="1.57" />--> <!--ToDo: adjust parameters -->
-        <limit effort="1000" velocity="10" lower="2.0" upper="2.0" /> <!--TEMP: fixed joint positions until control is fixed -->
+        <limit effort="1000" velocity="0.539" lower="0.0" upper="2.158" /> <!--ToDo: adjust parameters -->
+        <!--<limit effort="1000" velocity="10" lower="2.0" upper="2.0" />--> <!--TEMP: fixed joint positions until control is fixed -->
     </xacro:my_joint>
     <xacro:my_joint name="hip_joint" type="revolute" parent="upper_leg" child="trunk">
@@ -56,6 +56,6 @@
         <dynamics damping="6.0" friction="4.87"/><!-- ToDo: adjust dynamics-->
         <axis xyz="0 -1 0"/><!--ToDo: DH parameters?-->
-        <!--<limit effort="1000" velocity="10" lower="0.0" upper="1.57" />--> <!--ToDo: adjust parameters -->
-        <limit effort="1000" velocity="10" lower="2.36" upper="2.36" /> <!--TEMP: fixed joint positions until control is fixed-->
+        <limit effort="1000" velocity="0.375" lower="0.85" upper="2.36" /> <!--ToDo: adjust parameters --><!--Velocity: move in 4 s-->
+        <!--<limit effort="1000" velocity="10" lower="2.36" upper="2.36" />--> <!--TEMP: fixed joint positions until control is fixed-->
     </xacro:my_joint>
 </robot>

Commit message: sergio_description catkinized
git-svn-id: https://roboticssrv.wtb.tue.nl/svn/ros/trunk/sergio_description@27784 3a3c2cfb-d3b9-409e-9e75-db8fcdbcaac6

File: urdf/sergio.urdf (robot description, URDF)
Before this commit: robot sergio, 56 links, 55 joints
Joints:
- joint ankle_joint: limit lower=0.0 upper=1.059 effort=1000 velocity=0.264 -> lower=0.0 upper=1.059 effort=1000 velocity=0.265

File: urdf/xacro/sergio.urdf.xacro (robot description, xacro)
@@ -11,25 +11,25 @@
     <!--Definitions from default package?-->
     <!--get link & joint definitions -->
-    <!--<include filename="$(find amigo_robot_model)/description/definitions.xacro" />-->
-    <include filename="$(find amigo_description)/urdf/xacro/macro_definitions.xacro" />
+    <!--<xacro:include filename="$(find amigo_robot_model)/description/definitions.xacro" />-->
+    <xacro:include filename="$(find amigo_description)/urdf/xacro/macro_definitions.xacro" />
     <!--get custom materials -->
-    <!--<include filename="$(find amigo_robot_model)/description/materials.urdf.xacro" />-->
-    <include filename="$(find amigo_description)/urdf/xacro/materials.urdf.xacro" />
+    <!--<xacro:include filename="$(find amigo_robot_model)/description/materials.urdf.xacro" />-->
+    <xacro:include filename="$(find amigo_description)/urdf/xacro/materials.urdf.xacro" />
     <!--========BUILD BASE======-->
-    <include filename="$(find sergio_description)/urdf/xacro/base/base.urdf.xacro" />
+    <xacro:include filename="$(find sergio_description)/urdf/xacro/base/base.urdf.xacro" />
     <!--========BUILD TORSO======-->
-    <include filename="$(find sergio_description)/urdf/xacro/torso/torso.urdf.xacro" />
+    <xacro:include filename="$(find sergio_description)/urdf/xacro/torso/torso.urdf.xacro" />
     <!--========BUILD ARMS======-->
-    <include filename="$(find sergio_description)/urdf/xacro/arms/arm.urdf.xacro" />
+    <xacro:include filename="$(find sergio_description)/urdf/xacro/arms/arm.urdf.xacro" />
     <xacro:arm whichside="right" sidesign="+1.0" rollsign="+"/>
     <xacro:arm whichside="left"  sidesign="-1.0" rollsign="-"/>
     <!--========BUILD HEAD======-->
-    <include filename="$(find sergio_description)/urdf/xacro/head/head.urdf.xacro" />
+    <xacro:include filename="$(find sergio_description)/urdf/xacro/head/head.urdf.xacro" />
     <!--========BUILD KINECT======-->
-    <include filename="$(find sergio_description)/urdf/xacro/kinect/top_kinect.urdf.xacro" />
+    <xacro:include filename="$(find sergio_description)/urdf/xacro/kinect/top_kinect.urdf.xacro" />
     <!--========BUILD LASER======-->
-    <include filename="$(find sergio_description)/urdf/xacro/laser/laser.urdf.xacro" />
-    <include filename="$(find sergio_description)/urdf/xacro/laser/torso_laser.urdf.xacro" />
+    <xacro:include filename="$(find sergio_description)/urdf/xacro/laser/laser.urdf.xacro" />
+    <xacro:include filename="$(find sergio_description)/urdf/xacro/laser/torso_laser.urdf.xacro" />
     <!-- GAZEBO -->
-    <include filename="$(find sergio_description)/urdf/xacro/gazebo.urdf.xacro"/>
+    <xacro:include filename="$(find sergio_description)/urdf/xacro/gazebo.urdf.xacro"/>
 </robot>

Commit message: Prepared dummy joint state publisher for current use
git-svn-id: https://roboticssrv.wtb.tue.nl/svn/ros/trunk/sergio_description@28398 3a3c2cfb-d3b9-409e-9e75-db8fcdbcaac6

File: urdf/sergio.urdf (robot description, URDF)
Before this commit: robot sergio, 56 links, 55 joints
Joints:
- joint base_laser_joint: origin xyz=0.35 0.0 -0.06 rpy=3.14 0 0 -> xyz=0.35 0.0 0.175 rpy=0 0 0

File: urdf/xacro/laser/laser.urdf.xacro (robot description, xacro)
@@ -1,5 +1,5 @@
 <?xml version="1.0"?>
 <robot xmlns:xacro="http://ros.org/wiki/xacro">
-   <author>Kris van Tienhoven</author>
+   <author>Janno Lunenburg</author>
    <license>BSD</license>
    <review status="unreviewed" notes=""/>
@@ -12,5 +12,5 @@
 </xacro:my_link>
 <xacro:my_joint name="base_laser_joint" type="fixed" parent="base" child="base_laser">
-   <origin xyz="0.35 0.0 -0.06" rpy="3.14 0 0"/><!-- ToDO: determine location -->
+   <origin xyz="0.35 0.0 0.175" rpy="0 0 0"/><!-- ToDO: determine location -->
    <dynamics damping="0.1" friction="0"/>
    <axis xyz="0 1 0"/>

Commit message: updated urdf model to the 3d design in inventor

File: urdf/sergio.urdf (robot description, URDF)
Before this commit: robot sergio, 56 links, 55 joints
Links:
- added link lasermount, mass 0.01; collision box size=0.01 0.06 0.035; visual box size=0.01 0.06 0.035
- link base: geometry collision box size=0.713 0.500 0.11; visual box size=0.713 0.500 0.11
- link base_laser: geometry collision box size=0.06 0.06 0.077; visual box size=0.06 0.06 0.077
- link head_mount: mass 0.001 -> 0.05; geometry collision box size=0.061 0.08 0.08; visual box size=0.061 0.08 0.08
- link lasertop: geometry collision box size=0.06 0.06 0.01; visual box size=0.06 0.06 0.01
- link neck_pan: geometry collision cylinder length=0.02 radius=0.015; visual cylinder length=0.02 radius=0.015
- link neck_tilt: geometry collision box size=0.03 0.03 0.036; visual box size=0.03 0.03 0.036
- link sidepot_left: geometry collision box size=0.400 0.0615 0.1; visual box size=0.400 0.0615 0.1
- link sidepot_right: geometry collision box size=0.400 0.0615 0.1; visual box size=0.400 0.0615 0.1
- link trunk: geometry collision box size=0.470 0.200 0.15; visual box size=0.470 0.200 0.15
Joints:
- added joint lasermount_joint: type fixed, parent base_laser, child lasermount
- joint ankle_joint: origin xyz=-0.185 0.0 0.045 rpy=0 0 0 -> xyz=-0.185 0.0 0.0565 rpy=0 0 0
- joint base_laser_joint: origin xyz=0.35 0.0 0.175 rpy=0 0 0 -> xyz=0.3295 0.0 0.145 rpy=0 0 0
- joint base_link_joint: origin xyz=0.0 0.0 0.075 rpy=0 0 0 -> xyz=0.0 0.0 0.085 rpy=0 0 0
- joint base_mount_joint: origin xyz=0.0 0.0 0.05 rpy=0 0 0.0 -> xyz=0.0 0.0 0.055 rpy=0 0 0.0
- joint head_joint: origin (none) -> xyz=0.0 0.0 0.036 rpy=0.0 0.0 0.0
- joint head_mount_joint: origin xyz=0.5 0.0 0.0 rpy=3.14 0.0 0.0 -> xyz=0.6057 0.0 -0.01017 rpy=3.14 0.065 0.0
- joint neck_tilt_joint: limit lower=-2.0 upper=2.0 effort=13.4 velocity=1.0 -> lower=-0.98 upper=0.98 effort=13.4 velocity=1.0; origin xyz=0.0 0.0 0.0445 rpy=0.0 0.0 0.0 -> xyz=0.0 0.0 0.0 rpy=0.0 0.0 0.0
- joint shoulder_mount_joint_left: origin xyz=0.445 0.22 0.0 rpy=3.14 0 0.0 -> xyz=0.470 0.22 0.0 rpy=3.14 0 0.0
- joint shoulder_mount_joint_right: origin xyz=0.445 -0.22 0.0 rpy=3.14 0 0.0 -> xyz=0.470 -0.22 0.0 rpy=3.14 0 0.0
- joint sidepot_left_joint: origin xyz=0.0 0.275 0.0 rpy=0 0 0 -> xyz=0.0 0.28075 0.0 rpy=0 0 0
- joint sidepot_right_joint: origin xyz=0.0 -0.275 0.0 rpy=0 0 0 -> xyz=0.0 -0.28075 0.0 rpy=0 0 0
- joint top_kinect/base_kinect_joint: origin xyz=0.07 0 0.07 rpy=0 0 0 -> xyz=0.019 0.0 0.017 rpy=0 0 0

File: urdf/xacro/arms/arm.urdf.xacro (robot description, xacro)
@@ -158,5 +158,5 @@
     <parent link="trunk"/>
     <child link="shoulder_mount_${whichside}"/>
-    <origin xyz="0.445 ${sidesign*-0.22} 0.0" rpy="3.14 0 0.0"/><!-- Check length -->
+    <origin xyz="0.470 ${sidesign*-0.22} 0.0" rpy="3.14 0 0.0"/><!-- Check length -->
   </joint>
 <xacro:my_joint name="shoulder_yaw_joint_${whichside}" type="revolute" parent="shoulder_mount_${whichside}" child="shoulder_link1_${whichside}">

File: urdf/xacro/base/base.urdf.xacro (robot description, xacro)
@@ -13,12 +13,12 @@
     <!--base block-->
     <xacro:my_link name="base" mass="0.1" color="White"><!--ToDo: estimate mass-->
-        <box size="0.700 0.500 0.1" /><!--ToDo: check dimensions, adjust height-->
-        <origin xyz="0.0 0.0 0.0" rpy="0 0 0"/>
-        <origin xyz="0.0 0.0 0.0" rpy="0 0 0"/>
+        <box size="0.713 0.500 0.11" /><!--ToDo: check dimensions, adjust height-->
+        <origin xyz="-0.0235 0.0 0.0" rpy="0 0 0"/>
+        <origin xyz="-0.0235 0.0 0.0" rpy="0 0 0"/>
         <inertia ixx="0.001"  ixy="0"  ixz="0" iyy="0.001" iyz="0" izz="0.001" /><!--Estimate inertia-->
     </xacro:my_link>
     <!-- side pots -->
     <xacro:my_link name="sidepot_left" mass="0.1" color="White"><!--ToDo: estimate mass-->
-        <box size="0.400 0.050 0.1" /><!--ToDo: check dimensions, adjust height-->
+        <box size="0.400 0.0615 0.1" /><!--ToDo: check dimensions, adjust height-->
         <origin xyz="0.0 0.0 0.0" rpy="0 0 0"/>
         <origin xyz="0.0 0.0 0.0" rpy="0 0 0"/>
@@ -26,5 +26,5 @@
     </xacro:my_link>
     <xacro:my_link name="sidepot_right" mass="0.1" color="White"><!--ToDo: estimate mass-->
-        <box size="0.400 0.050 0.1" /><!--ToDo: check dimensions, adjust height-->
+        <box size="0.400 0.0615 0.1" /><!--ToDo: check dimensions, adjust height-->
         <origin xyz="0.0 0.0 0.0" rpy="0 0 0"/>
         <origin xyz="0.0 0.0 0.0" rpy="0 0 0"/>
@@ -43,5 +43,5 @@
         <child link="base"/>
         <axis xyz="1 0 0"/>
-        <origin xyz="0.0 0.0 0.075" rpy="0 0 0"/><!--ToDO: adjust height-->
+        <origin xyz="0.0 0.0 0.085" rpy="0 0 0"/><!--ToDO: adjust height-->
     </joint>
     <joint name="sidepot_left_joint" type="fixed">
@@ -49,5 +49,5 @@
         <child link="sidepot_left"/>
         <axis xyz="1 0 0"/>
-        <origin xyz="0.0 0.275 0.0" rpy="0 0 0"/><!--ToDO: adjust distance-->
+        <origin xyz="0.0 0.28075 0.0" rpy="0 0 0"/><!--ToDO: adjust distance-->
     </joint>
     <joint name="sidepot_right_joint" type="fixed">
@@ -55,10 +55,10 @@
         <child link="sidepot_right"/>
         <axis xyz="1 0 0"/>
-        <origin xyz="0.0 -0.275 0.0" rpy="0 0 0"/><!--ToDO: adjust distance-->
+        <origin xyz="0.0 -0.28075 0.0" rpy="0 0 0"/><!--ToDO: adjust distance-->
     </joint>
     <joint name="base_mount_joint" type="fixed">
         <parent link="base"/>
         <child link="base_torso_mount"/>
-        <origin xyz="0.0 0.0 0.05" rpy="0 0 0.0"/><!--ToDo: adjust height-->
+        <origin xyz="0.0 0.0 0.055" rpy="0 0 0.0"/><!--ToDo: adjust height-->
     </joint>
 </robot>

File: urdf/xacro/gazebo.urdf.xacro (robot description, xacro)
@@ -174,5 +174,5 @@
           <frameName>base_laser</frameName>
         </plugin>
-        <pose>0.310000 0.000000 0.240000 3.140000 0.000000 0.000000</pose>
+        <pose>0.329500 0.000000 0.230000 3.140000 0.000000 0.000000</pose>
       </sensor>
 </gazebo>

File: urdf/xacro/head/head.urdf.xacro (robot description, xacro)
@@ -6,22 +6,22 @@
 <!--head-->
 <!-- !!!!!!!!!something without a visual not sure what this is!!!!!!!!!!!! -->
-<link name="head_mount">
-  <inertial>
-    <origin xyz="0.0 0.0 0.0" rpy="0 0 0"/>
-    <mass value="0.001"/>
+<xacro:my_link name="head_mount" mass="0.05" color="White">
+    <box size="0.061 0.08 0.08" /><!-- Fill in -->
+    <origin xyz="-0.0505 0.0 0.0" rpy="0 0 0"/>
+    <origin xyz="-0.0505 0.0 0.0" rpy="0 0 0"/>
     <inertia ixx="0.0001"  ixy="0"  ixz="0" iyy="0.0001" iyz="0" izz="0.0001" />
-  </inertial>
-</link>
+    <color rgba="0.25 0.25 0.25 1.0"/>
+</xacro:my_link>
 <joint name="head_mount_joint" type="fixed">
   <parent link="trunk"/>
   <child link="head_mount"/>
   <axis xyz="0 0 1"/>
-  <origin xyz="0.5 0.0 0.0" rpy="3.14 0.0 0.0"/><!-- Check length -->
+  <origin xyz="0.6057 0.0 -0.01017" rpy="3.14 0.065 0.0"/><!-- Check length -->
 </joint>
 <!-- the link that represents the panning part of the neck, is below neck_tilt -->
 <xacro:my_link name="neck_pan" mass="0.05" color="White">
-   <cylinder radius="0.015" length="0.0525" />
-   <origin xyz="0.0 0.0 0.0335" rpy="0 0 0"/>
-   <origin xyz="0.0 0.0 0.0335" rpy="0 0 0" />
+   <cylinder radius="0.015" length="0.02" />
+   <origin xyz="0.0 0.0 -0.01" rpy="0 0 0"/>
+   <origin xyz="0.0 0.0 -0.01" rpy="0 0 0" />
    <inertia ixx="0.0001"  ixy="0"  ixz="0" iyy="0.0001" iyz="0" izz="0.0001" />
    <color rgba="0.25 0.25 0.25 1.0"/>
@@ -35,7 +35,7 @@
 </xacro:my_link_texturedmesh>-->
 <xacro:my_link name="neck_tilt" mass="0.05" color="White">
-   <box size="0.001 0.001 0.001" /><!-- Fill in -->
-   <origin xyz="0.0 -0.0 0.0285" rpy="0 0 0"/>
-   <origin xyz="0.0 -0.0 0.015" rpy="0 0 0" />
+   <box size="0.03 0.03 0.036" /><!-- Fill in -->
+   <origin xyz="0.0 -0.0 0.018" rpy="0 0 0"/>
+   <origin xyz="0.0 -0.0 0.018" rpy="0 0 0" />
    <inertia ixx="0.001"  ixy="0"  ixz="0" iyy="0.001" iyz="0" izz="0.001" />
 </xacro:my_link>
@@ -49,5 +49,5 @@
   <my_link name="head" mass="0" color="White">
     <box size="0.001 0.001 0.001" /><!-- Fill in -->
-   <origin xyz="0 0 0.041" rpy="0 0 0"/>
+   <origin xyz="0.0 0.0 0.041" rpy="0 0 0"/>
    <origin xyz="0.0 0.0 0.141" rpy="0 0 -1.5708"/>
    <inertia ixx="0"  ixy="0"  ixz="0" iyy="0" iyz="0" izz="0" />
@@ -56,4 +56,5 @@
     <parent link="neck_tilt"/>
     <child link="head"/>
+    <origin xyz="0.0 0.0 0.036" rpy="0.0 0.0 0.0"/>
   </joint>
 <!-- the tilt and pan joints-->
@@ -65,8 +66,8 @@
 </xacro:my_joint>
 <xacro:my_joint name="neck_tilt_joint" type="revolute" parent="neck_pan" child="neck_tilt">
-   <origin xyz="0.0 0.0 0.0445" rpy="0.0 0.0 0.0"/>
+   <origin xyz="0.0 0.0 0.0" rpy="0.0 0.0 0.0"/>
    <dynamics damping="0.1" friction="0.0"/>
    <axis xyz="0 1 0"/>
-   <limit effort="13.4" velocity="1.0" lower="-2.0" upper="2.0" />
+   <limit effort="13.4" velocity="1.0" lower="-0.98" upper="0.98" />
 </xacro:my_joint>
 </robot>

File: urdf/xacro/kinect/top_kinect.urdf.xacro (robot description, xacro)
@@ -6,5 +6,5 @@
   <property name="M_PI" value="3.14159"/>
   <joint name="top_kinect/base_kinect_joint" type="fixed">
-    <origin xyz="0.07 0 0.07" rpy="0 0 0" /> <!-- THESE VALUES ARE ROUGH ESTIMATES!! -->
+    <origin xyz="0.019 0.0 0.017" rpy="0 0 0" /> <!-- THESE VALUES ARE ROUGH ESTIMATES!! -->
     <parent link="head" />
     <child link="top_kinect/openni_camera" />

File: urdf/xacro/laser/laser.urdf.xacro (robot description, xacro)
@@ -6,11 +6,12 @@
 <!--the laser at the base of the robot -->
 <xacro:my_link name="base_laser" mass="0.5" color="Black">
-   <box size="0.05 0.065 0.12" />
-   <origin xyz="0.0 0.0 0.0" rpy="0 0 0"/>
-   <origin xyz="-0.005 0.0 -0.065" rpy="0 0 0" />
+   <box size="0.06 0.06 0.077" />
+   <origin xyz="0.0 0.0 -0.0165" rpy="0 0 0"/>
+   <origin xyz="0.0 0.0 -0.0165" rpy="0 0 0" />
    <inertia ixx="0.0001"  ixy="0"  ixz="0" iyy="0.0001" iyz="0" izz="0.0001" />
 </xacro:my_link>
+<!-- origin of the laser range finder, from technical drawing -->
 <xacro:my_joint name="base_laser_joint" type="fixed" parent="base" child="base_laser">
-   <origin xyz="0.35 0.0 0.175" rpy="0 0 0"/><!-- ToDO: determine location -->
+   <origin xyz="0.3295 0.0 0.145" rpy="0 0 0"/><!-- ToDO: determine location -->
    <dynamics damping="0.1" friction="0"/>
    <axis xyz="0 1 0"/>
@@ -25,7 +26,7 @@
 </xacro:my_link_textured>-->
 <xacro:my_link name="lasertop" mass="0.01" color="Red"><!--Changed color to red to make it work-->
-   <box size="0.05 0.065 0.01" />
-   <origin xyz="0.0 0.0 0.0" rpy="0 0 0"/>
-   <origin xyz="-0.005 0.0 0.0" rpy="0 0 0" />
+   <box size="0.06 0.06 0.01" />
+   <origin xyz="0.0 0.0 0.027" rpy="0 0 0"/>
+   <origin xyz="0.0 0.0 0.027" rpy="0 0 0" />
    <inertia ixx="0.0001"  ixy="0"  ixz="0" iyy="0.0001" iyz="0" izz="0.0001" />
 </xacro:my_link>
@@ -33,4 +34,14 @@
     <parent link="base_laser"/>
     <child link="lasertop"/>
+</joint>
+<xacro:my_link name="lasermount" mass="0.01" color="White">
+   <box size="0.01 0.06 0.035" />
+   <origin xyz="-0.025 0.0 -0.0725" rpy="0 0 0"/>
+   <origin xyz="-0.025 0.0 -0.0725" rpy="0 0 0" />
+   <inertia ixx="0.0001"  ixy="0"  ixz="0" iyy="0.0001" iyz="0" izz="0.0001" />
+</xacro:my_link>
+<joint name="lasermount_joint" type="fixed">
+    <parent link="base_laser"/>
+    <child link="lasermount"/>
 </joint>
 <!--the tue logo in front of the laser-->

File: urdf/xacro/torso/torso.urdf.xacro (robot description, xacro)
@@ -27,7 +27,7 @@
     <!-- Trunk -->
     <xacro:my_link name="trunk" mass="10" color="White"><!--ToDo: estimate mass-->
-        <box size="0.445 0.200 0.15" /><!--ToDo: check dimensions, adjust height-->
-        <origin xyz="0.2225 0.0 0.0" rpy="0 0 0"/><!--ToDo: check dimensions, adjust height-->
-        <origin xyz="0.2225 0.0 0.0" rpy="0 0 0"/><!--ToDo: check dimensions, adjust height-->
+        <box size="0.470 0.200 0.15" /><!--ToDo: check dimensions, adjust height-->
+        <origin xyz="0.235 0.0 0.0" rpy="0 0 0"/><!--ToDo: check dimensions, adjust height-->
+        <origin xyz="0.235 0.0 0.0" rpy="0 0 0"/><!--ToDo: check dimensions, adjust height-->
         <inertia ixx="0.001"  ixy="0"  ixz="0" iyy="0.001" iyz="0" izz="0.001" /><!--Estimate inertia-->
     </xacro:my_link>
@@ -39,5 +39,5 @@
     </joint>
     <xacro:my_joint name="ankle_joint" type="revolute" parent="torso_mounting_frame" child="lower_rear_leg">
-        <origin xyz="-0.185 0.0 0.045" rpy="0 0 0"/><!-- ToDo: adjust height-->
+        <origin xyz="-0.185 0.0 0.0565" rpy="0 0 0"/><!-- ToDo: adjust height-->
         <dynamics damping="6.0" friction="4.87"/><!-- ToDo: adjust dynamics-->
         <axis xyz="0 -1 0"/><!--ToDo: DH parameters?-->
