Commit message: 5 ultrasone sensors added to the base

File: urdf/sergio.urdf (robot description, URDF)
Before this commit: robot sergio, 57 links, 56 joints
Links:
- added link base_sonar1, mass 0.05; collision cylinder length=0.01 radius=0.005; visual cylinder length=0.01 radius=0.005
- added link base_sonar2, mass 0.05; collision cylinder length=0.01 radius=0.005; visual cylinder length=0.01 radius=0.005
- added link base_sonar3, mass 0.05; collision cylinder length=0.01 radius=0.005; visual cylinder length=0.01 radius=0.005
- added link base_sonar4, mass 0.05; collision cylinder length=0.01 radius=0.005; visual cylinder length=0.01 radius=0.005
- added link base_sonar5, mass 0.05; collision cylinder length=0.01 radius=0.005; visual cylinder length=0.01 radius=0.005
Joints:
- added joint base_sonar1_joint: type fixed, parent base, child base_sonar1, origin xyz=-0.380 0.0 0.0 rpy=0.0 0 3.14
- added joint base_sonar2_joint: type fixed, parent base, child base_sonar2, origin xyz=-0.380 0.311 0.0 rpy=0.0 0 3.14
- added joint base_sonar3_joint: type fixed, parent base, child base_sonar3, origin xyz=-0.380 -0.311 0.0 rpy=0.0 0 3.14
- added joint base_sonar4_joint: type fixed, parent base, child base_sonar4, origin xyz=-0.370 -0.3115 0.0 rpy=0.0 0 -1.57
- added joint base_sonar5_joint: type fixed, parent base, child base_sonar5, origin xyz=-0.370 0.3115 0.0 rpy=0.0 0 1.57
- joint base_laser_joint: origin xyz=0.3295 0.0 0.145 rpy=0 0 0 -> xyz=0.3295 0.0 0.145 rpy=0.0 0 0

File: urdf/xacro/laser/laser.urdf.xacro (robot description, xacro)
@@ -13,5 +13,5 @@
 <!-- origin of the laser range finder, from technical drawing -->
 <xacro:my_joint name="base_laser_joint" type="fixed" parent="base" child="base_laser">
-   <origin xyz="0.3295 0.0 0.145" rpy="0 0 0"/><!-- ToDO: determine location -->
+   <origin xyz="0.3295 0.0 0.145" rpy="0.0 0 0"/><!-- ToDO: determine location -->
    <dynamics damping="0.1" friction="0"/>
    <axis xyz="0 1 0"/>

File: urdf/xacro/sergio.urdf.xacro (robot description, xacro)
@@ -31,4 +31,6 @@
     <xacro:include filename="$(find sergio_description)/urdf/xacro/laser/laser.urdf.xacro" />
     <xacro:include filename="$(find sergio_description)/urdf/xacro/laser/torso_laser.urdf.xacro" />
+    <!--========BUILD ULTRASONE======-->
+    <xacro:include filename="$(find sergio_description)/urdf/xacro/ultrasone/ultrasone.urdf.xacro" />
     <!-- GAZEBO -->
     <xacro:include filename="$(find sergio_description)/urdf/xacro/gazebo.urdf.xacro"/>

Commit message: new sergio urdf model working

File: urdf/sergio.urdf (robot description, URDF)
Before this commit: robot sergio, 57 links, 56 joints
Links:
- removed link lasermount
- removed link lasertop
- added link base_lasertop, mass 0.01; collision box size=0.06 0.06 0.018; visual box size=0.06 0.06 0.018
- added link laser_mount, mass 0.01; collision box size=0.01 0.06 0.035; visual box size=0.01 0.06 0.035
- added link torso_laser_mount, mass 0.01; collision box size=0.06 0.06 0.018; visual box size=0.06 0.06 0.018
- link base_laser: geometry collision box size=0.06 0.06 0.069; visual box size=0.06 0.06 0.069
- link torso_laser: geometry collision box size=0.06 0.06 0.069; visual box size=0.06 0.06 0.069
- link torso_lasertop: geometry collision box size=0.06 0.06 0.018; visual box size=0.06 0.06 0.018
Joints:
- removed joint base_laser_joint
- removed joint lasermount_joint
- removed joint lasertop_joint
- removed joint torso_laser_joint
- added joint base_lasercenter_joint: type fixed, parent laser_mount, child base_laser, origin xyz=0.03 0.0 0.09 rpy=0.0 0.0 0.0
- added joint base_lasertop_joint: type fixed, parent base_laser, child base_lasertop, origin xyz=0.0 0.0 0.023 rpy=0 0 0
- added joint laser_mount_joint: type fixed, parent base, child laser_mount, origin xyz=0.2995 0.0 0.055 rpy=0.0 0.0 0.0
- added joint laser_tilt_joint: type revolute, parent trunk, child torso_laser_mount, origin xyz=0.3163 0.0 -0.0671 rpy=3.14 1.57 0.0 , axis 0 1 0, limit lower=-0.3 upper=0.3 effort=13.4 velocity=1.0
- added joint torso_lasercenter_joint: type fixed, parent torso_laser_mount, child torso_laser, origin xyz=0.0 0.0 0.0015 rpy=0.0 0.0 0.0
- joint top_kinect/base_kinect_joint: origin xyz=0.019 0.0 0.017 rpy=0 0 0 -> xyz=0.03 0.0 0.017 rpy=0 0 0
- joint torso_lasertop_joint: origin (none) -> xyz=0.0 0.0 0.023 rpy=0 0 0

File: urdf/xacro/base/base.urdf.xacro (robot description, xacro)
@@ -38,4 +38,11 @@
        <inertia ixx="0"  ixy="0"  ixz="0" iyy="0" iyz="0" izz="0" />
     </xacro:my_link>
+    <!-- base - laser interface -->
+    <xacro:my_link name="laser_mount" mass="0.01" color="White">
+       <box size="0.01 0.06 0.035" />
+       <origin xyz="0.005 0.0 0.0175" rpy="0 0 0"/>
+       <origin xyz="0.005 0.0 0.0175" rpy="0 0 0" />
+        <inertia ixx="0.0001"  ixy="0"  ixz="0" iyy="0.0001" iyz="0" izz="0.0001" />
+    </xacro:my_link>
     <!-- joints -->
     <joint name="base_link_joint" type="fixed">
@@ -62,3 +69,8 @@
         <origin xyz="0.0 0.0 0.055" rpy="0 0 0.0"/><!--ToDo: adjust height-->
     </joint>
+    <joint name="laser_mount_joint" type="fixed">
+        <parent link="base"/>
+        <child link="laser_mount"/>
+        <origin xyz="0.2995 0.0 0.055" rpy="0.0 0.0 0.0"/>
+    </joint>
 </robot>

File: urdf/xacro/kinect/top_kinect.urdf.xacro (robot description, xacro)
@@ -6,5 +6,5 @@
   <property name="M_PI" value="3.14159"/>
   <joint name="top_kinect/base_kinect_joint" type="fixed">
-    <origin xyz="0.019 0.0 0.017" rpy="0 0 0" /> <!-- THESE VALUES ARE ROUGH ESTIMATES!! -->
+    <origin xyz="0.03 0.0 0.017" rpy="0 0 0" /> <!-- THESE VALUES ARE ROUGH ESTIMATES!! -->
     <parent link="head" />
     <child link="top_kinect/openni_camera" />

File: urdf/xacro/laser/laser.urdf.xacro (robot description, xacro)
@@ -1,58 +1,40 @@
 <?xml version="1.0"?>
 <robot xmlns:xacro="http://ros.org/wiki/xacro">
-   <author>Janno Lunenburg</author>
+   <author>Ton Peters</author>
    <license>BSD</license>
    <review status="unreviewed" notes=""/>
-<!--the laser at the base of the robot -->
-<xacro:my_link name="base_laser" mass="0.5" color="Black">
-   <box size="0.06 0.06 0.077" />
-   <origin xyz="0.0 0.0 -0.0165" rpy="0 0 0"/>
-   <origin xyz="0.0 0.0 -0.0165" rpy="0 0 0" />
+<!--Start of the macro
+@param laser_name, is used to locate the sensor
+@param laser_parent, parent
+@param laser_xyz, transform from parent to laser center (center is at l=0.3 w=0.3 h=55)
+@param laser_rpy, rotation from parent to laser center (x points forward, z to the top)
+-->
+ <xacro:macro name="laser" params="laser_name laser_parent laser_xyz laser_rpy">
+<!-- link visualize the black part of the laser-->
+<xacro:my_link name="${laser_name}_laser" mass="0.5" color="Black">
+   <box size="0.06 0.06 0.069" />
+   <origin xyz="0.0 0.0 -0.0205" rpy="0 0 0"/>
+   <origin xyz="0.0 0.0 -0.0205" rpy="0 0 0" />
    <inertia ixx="0.0001"  ixy="0"  ixz="0" iyy="0.0001" iyz="0" izz="0.0001" />
 </xacro:my_link>
-<!-- origin of the laser range finder, from technical drawing -->
-<xacro:my_joint name="base_laser_joint" type="fixed" parent="base" child="base_laser">
-   <origin xyz="0.3295 0.0 0.145" rpy="0 0 0"/><!-- ToDO: determine location -->
-   <dynamics damping="0.1" friction="0"/>
-   <axis xyz="0 1 0"/>
-   <limit effort="13.4" velocity="1.0" lower="-0.7809" upper="1.5708" />
-</xacro:my_joint>
-<!--the orange top of the laser-->
-<!--<xacro:my_link_textured name="lasertop" mass="0.01" texture="orange">
-   <box size="0.05 0.065 0.01" />
+<!-- joint origin of the laser range finder -->
+<joint name="${laser_name}_lasercenter_joint" type="fixed">
+    <parent link="${laser_parent}"/>
+    <child link="${laser_name}_laser"/>
+    <origin xyz="${laser_xyz}" rpy="${laser_rpy}"/>
+</joint>
+<!-- joint origin of the orange top -->
+<joint name="${laser_name}_lasertop_joint" type="fixed">
+    <parent link="${laser_name}_laser"/>
+    <child link="${laser_name}_lasertop"/>
+    <origin xyz="0.0 0.0 0.023" rpy="0 0 0"/>
+</joint>
+<!-- link visual of the orange top -->
+<xacro:my_link name="${laser_name}_lasertop" mass="0.01" color="Orange"><!--Changed color to red to make it work-->
+   <box size="0.06 0.06 0.018" />
    <origin xyz="0.0 0.0 0.0" rpy="0 0 0"/>
-   <origin xyz="-0.005 0.0 0.0" rpy="0 0 0" />
-   <inertia ixx="0.0001"  ixy="0"  ixz="0" iyy="0.0001" iyz="0" izz="0.0001" />
-</xacro:my_link_textured>-->
-<xacro:my_link name="lasertop" mass="0.01" color="Red"><!--Changed color to red to make it work-->
-   <box size="0.06 0.06 0.01" />
-   <origin xyz="0.0 0.0 0.027" rpy="0 0 0"/>
-   <origin xyz="0.0 0.0 0.027" rpy="0 0 0" />
+   <origin xyz="0.0 0.0 0.0" rpy="0 0 0" />
    <inertia ixx="0.0001"  ixy="0"  ixz="0" iyy="0.0001" iyz="0" izz="0.0001" />
 </xacro:my_link>
-<joint name="lasertop_joint" type="fixed">
-    <parent link="base_laser"/>
-    <child link="lasertop"/>
-</joint>
-<xacro:my_link name="lasermount" mass="0.01" color="White">
-   <box size="0.01 0.06 0.035" />
-   <origin xyz="-0.025 0.0 -0.0725" rpy="0 0 0"/>
-   <origin xyz="-0.025 0.0 -0.0725" rpy="0 0 0" />
-   <inertia ixx="0.0001"  ixy="0"  ixz="0" iyy="0.0001" iyz="0" izz="0.0001" />
-</xacro:my_link>
-<joint name="lasermount_joint" type="fixed">
-    <parent link="base_laser"/>
-    <child link="lasermount"/>
-</joint>
-<!--the tue logo in front of the laser-->
-<!--<xacro:my_link_texturedmesh name="logo" mass="0.01" texture="amigo_description/logo">
-   <origin xyz="0.0 0.0 0.0" rpy="0 0 0"/>
-   <origin xyz="0.025 0.0 -0.14" rpy="0 0 3.1415" />
-   <inertia ixx="0.0001"  ixy="0"  ixz="0" iyy="0.0001" iyz="0" izz="0.0001" />
-   <mesh filename="package://amigo2_description/media/meshes/logo.dae" scale="0.0016 0.0016 0.0016"/>
-</xacro:my_link_texturedmesh>
-  <joint name="logo_joint" type="fixed">
-    <parent link="base_laser"/>
-    <child link="logo"/>
-  </joint>-->
+</xacro:macro>
 </robot>

File: urdf/xacro/sergio.urdf.xacro (robot description, xacro)
@@ -28,7 +28,11 @@
     <!--========BUILD KINECT======-->
     <xacro:include filename="$(find sergio_description)/urdf/xacro/kinect/top_kinect.urdf.xacro" />
-    <!--========BUILD LASER======-->
+    <!--========BUILD TORSO LASER JOINT======-->
+    <xacro:include filename="$(find sergio_description)/urdf/xacro/laser/torso_laser_joint.urdf.xacro" />
+    <!--========BUILD LASERS======-->
+    <!--<xacro:include filename="$(find sergio_description)/urdf/xacro/laser/base_laser.urdf.xacro" />-->
     <xacro:include filename="$(find sergio_description)/urdf/xacro/laser/laser.urdf.xacro" />
-    <xacro:include filename="$(find sergio_description)/urdf/xacro/laser/torso_laser.urdf.xacro" />
+    <xacro:laser laser_name="base" laser_parent="laser_mount" laser_xyz="0.03 0.0 0.09" laser_rpy="0.0 0.0 0.0"  />
+    <xacro:laser laser_name="torso" laser_parent="torso_laser_mount" laser_xyz="0.0 0.0 0.0015" laser_rpy="0.0 0.0 0.0"  />
     <!-- GAZEBO -->
     <xacro:include filename="$(find sergio_description)/urdf/xacro/gazebo.urdf.xacro"/>

Commit message: added documentation to the urdf model

File: urdf/sergio.urdf (robot description, URDF)
Before this commit: robot sergio, 58 links, 57 joints
Joints:
- joint hip_joint: origin xyz=0.4115 0.0 0. rpy=3.14 3.14 0 -> xyz=0.4115 0.0 0.0 rpy=3.14 3.14 0.0
- joint knee_joint: origin xyz=0.390 0.0 0. rpy=3.14 3.14 0 -> xyz=0.390 0.0 0.0 rpy=3.14 3.14 0.0

File: urdf/xacro/torso/torso.urdf.xacro (robot description, xacro)
@@ -46,5 +46,5 @@
     </xacro:my_joint>
     <xacro:my_joint name="knee_joint" type="revolute" parent="lower_rear_leg" child="upper_leg">
-        <origin xyz="0.390 0.0 0." rpy="3.14 3.14 0"/><!-- ToDo: adjust height-->
+        <origin xyz="0.390 0.0 0.0" rpy="3.14 3.14 0.0"/><!-- ToDo: adjust height-->
         <dynamics damping="6.0" friction="4.87"/><!-- ToDo: adjust dynamics-->
         <axis xyz="0 -1 0"/><!--ToDo: DH parameters?-->
@@ -53,5 +53,5 @@
     </xacro:my_joint>
     <xacro:my_joint name="hip_joint" type="revolute" parent="upper_leg" child="trunk">
-        <origin xyz="0.4115 0.0 0." rpy="3.14 3.14 0"/><!-- ToDo: adjust height-->
+        <origin xyz="0.4115 0.0 0.0" rpy="3.14 3.14 0.0"/><!-- ToDo: adjust height-->
         <dynamics damping="6.0" friction="4.87"/><!-- ToDo: adjust dynamics-->
         <axis xyz="0 -1 0"/><!--ToDo: DH parameters?-->

Commit message: renamed torso_laser_joint to laser_tilt_joint

File: urdf/sergio.urdf (robot description, URDF)
Before this commit: robot sergio, 56 links, 55 joints
Joints:
- removed joint torso_laser_joint
- added joint laser_tilt_joint: type revolute, parent trunk, child torso_laser, origin xyz=0.22 0.0 -0.1 rpy=3.14 1.57 0.0 , axis 0 1 0, limit lower=-0.7809 upper=1.5708 effort=13.4 velocity=1.0

File: urdf/xacro/laser/torso_laser.urdf.xacro (robot description, xacro)
@@ -11,5 +11,5 @@
    <inertia ixx="0.0001"  ixy="0"  ixz="0" iyy="0.0001" iyz="0" izz="0.0001" />
 </xacro:my_link>
-<xacro:my_joint name="torso_laser_joint" type="revolute" parent="trunk" child="torso_laser">
+<xacro:my_joint name="laser_tilt_joint" type="revolute" parent="trunk" child="torso_laser">
    <origin xyz="0.22 0.0 -0.1" rpy="3.14 1.57 0.0 "/><!-- ToDo: replace position -->
    <dynamics damping="0.1" friction="0"/><!--ToDo: update-->

Commit message: ultrasone sensors working

File: urdf/sergio.urdf (robot description, URDF)
Before this commit: robot sergio, 56 links, 55 joints
Links:
- added link base_sonar1, mass 0.05; collision cylinder length=0.01 radius=0.005; visual cylinder length=0.01 radius=0.005
- added link base_sonar2, mass 0.05; collision cylinder length=0.01 radius=0.005; visual cylinder length=0.01 radius=0.005
- added link base_sonar3, mass 0.05; collision cylinder length=0.01 radius=0.005; visual cylinder length=0.01 radius=0.005
- added link base_sonar4, mass 0.05; collision cylinder length=0.01 radius=0.005; visual cylinder length=0.01 radius=0.005
- added link base_sonar5, mass 0.05; collision cylinder length=0.01 radius=0.005; visual cylinder length=0.01 radius=0.005
- added link lasermount, mass 0.01; collision box size=0.01 0.06 0.035; visual box size=0.01 0.06 0.035
- link base: geometry collision box size=0.713 0.500 0.11; visual box size=0.713 0.500 0.11
- link base_laser: geometry collision box size=0.06 0.06 0.077; visual box size=0.06 0.06 0.077
- link head_mount: mass 0.001 -> 0.05; geometry collision box size=0.061 0.08 0.08; visual box size=0.061 0.08 0.08
- link lasertop: geometry collision box size=0.06 0.06 0.01; visual box size=0.06 0.06 0.01
- link neck_pan: geometry collision cylinder length=0.02 radius=0.015; visual cylinder length=0.02 radius=0.015
- link neck_tilt: geometry collision box size=0.03 0.03 0.036; visual box size=0.03 0.03 0.036
- link sidepot_left: geometry collision box size=0.400 0.0615 0.1; visual box size=0.400 0.0615 0.1
- link sidepot_right: geometry collision box size=0.400 0.0615 0.1; visual box size=0.400 0.0615 0.1
- link trunk: geometry collision box size=0.470 0.200 0.15; visual box size=0.470 0.200 0.15
Joints:
- added joint base_sonar1_joint: type fixed, parent base, child base_sonar1, origin xyz=-0.380 0.0 0.0 rpy=0.0 0 3.14
- added joint base_sonar2_joint: type fixed, parent base, child base_sonar2, origin xyz=-0.380 0.311 0.0 rpy=0.0 0 3.14
- added joint base_sonar3_joint: type fixed, parent base, child base_sonar3, origin xyz=-0.380 -0.311 0.0 rpy=0.0 0 3.14
- added joint base_sonar4_joint: type fixed, parent base, child base_sonar4, origin xyz=-0.370 -0.3115 0.0 rpy=0.0 0 -1.57
- added joint base_sonar5_joint: type fixed, parent base, child base_sonar5, origin xyz=-0.370 0.3115 0.0 rpy=0.0 0 1.57
- added joint lasermount_joint: type fixed, parent base_laser, child lasermount
- joint ankle_joint: origin xyz=-0.185 0.0 0.045 rpy=0 0 0 -> xyz=-0.185 0.0 0.0565 rpy=0 0 0
- joint base_laser_joint: origin xyz=0.35 0.0 0.175 rpy=0 0 0 -> xyz=0.3295 0.0 0.145 rpy=0.0 0 0
- joint base_link_joint: origin xyz=0.0 0.0 0.075 rpy=0 0 0 -> xyz=0.0 0.0 0.085 rpy=0 0 0
- joint base_mount_joint: origin xyz=0.0 0.0 0.05 rpy=0 0 0.0 -> xyz=0.0 0.0 0.055 rpy=0 0 0.0
- joint head_joint: origin (none) -> xyz=0.0 0.0 0.036 rpy=0.0 0.0 0.0
- joint head_mount_joint: origin xyz=0.5 0.0 0.0 rpy=3.14 0.0 0.0 -> xyz=0.6057 0.0 -0.01017 rpy=3.14 0.065 0.0
- joint neck_tilt_joint: limit lower=-2.0 upper=2.0 effort=13.4 velocity=1.0 -> lower=-0.98 upper=0.98 effort=13.4 velocity=1.0; origin xyz=0.0 0.0 0.0445 rpy=0.0 0.0 0.0 -> xyz=0.0 0.0 0.0 rpy=0.0 0.0 0.0
- joint shoulder_mount_joint_left: origin xyz=0.445 0.22 0.0 rpy=3.14 0 0.0 -> xyz=0.470 0.22 0.0 rpy=3.14 0 0.0
- joint shoulder_mount_joint_right: origin xyz=0.445 -0.22 0.0 rpy=3.14 0 0.0 -> xyz=0.470 -0.22 0.0 rpy=3.14 0 0.0
- joint sidepot_left_joint: origin xyz=0.0 0.275 0.0 rpy=0 0 0 -> xyz=0.0 0.28075 0.0 rpy=0 0 0
- joint sidepot_right_joint: origin xyz=0.0 -0.275 0.0 rpy=0 0 0 -> xyz=0.0 -0.28075 0.0 rpy=0 0 0
- joint top_kinect/base_kinect_joint: origin xyz=0.07 0 0.07 rpy=0 0 0 -> xyz=0.019 0.0 0.017 rpy=0 0 0

File: urdf/xacro/gazebo.urdf.xacro (robot description, xacro)
@@ -174,8 +174,8 @@
           <frameName>base_laser</frameName>
         </plugin>
-        <pose>0.310000 0.000000 0.240000 3.140000 0.000000 0.000000</pose>
+        <pose>0.329500 0.000000 0.230000 0.00000 0.000000 0.000000</pose>
       </sensor>
 </gazebo>
-<gazebo reference="neck_tilt">
+<gazebo reference="head">
       <sensor name='openni_camera' type='depth'>
         <update_rate>20.000000</update_rate>
@@ -203,5 +203,5 @@
           <frameName>top_kinect/openni_depth_optical_frame</frameName>
         </plugin>
-        <pose>0.070000 0.000000 0.070000 0.000000 0.000000 0.000000</pose>
+        <pose>0.019000 0.000000 0.017000 0.000000 0.000000 0.000000</pose>
       </sensor>
 </gazebo>

File: urdf/xacro/laser/laser.urdf.xacro (robot description, xacro)
@@ -6,11 +6,12 @@
 <!--the laser at the base of the robot -->
 <xacro:my_link name="base_laser" mass="0.5" color="Black">
-   <box size="0.05 0.065 0.12" />
-   <origin xyz="0.0 0.0 0.0" rpy="0 0 0"/>
-   <origin xyz="-0.005 0.0 -0.065" rpy="0 0 0" />
+   <box size="0.06 0.06 0.077" />
+   <origin xyz="0.0 0.0 -0.0165" rpy="0 0 0"/>
+   <origin xyz="0.0 0.0 -0.0165" rpy="0 0 0" />
    <inertia ixx="0.0001"  ixy="0"  ixz="0" iyy="0.0001" iyz="0" izz="0.0001" />
 </xacro:my_link>
+<!-- origin of the laser range finder, from technical drawing -->
 <xacro:my_joint name="base_laser_joint" type="fixed" parent="base" child="base_laser">
-   <origin xyz="0.35 0.0 0.175" rpy="0 0 0"/><!-- ToDO: determine location -->
+   <origin xyz="0.3295 0.0 0.145" rpy="0.0 0 0"/><!-- ToDO: determine location -->
    <dynamics damping="0.1" friction="0"/>
    <axis xyz="0 1 0"/>
@@ -25,7 +26,7 @@
 </xacro:my_link_textured>-->
 <xacro:my_link name="lasertop" mass="0.01" color="Red"><!--Changed color to red to make it work-->
-   <box size="0.05 0.065 0.01" />
-   <origin xyz="0.0 0.0 0.0" rpy="0 0 0"/>
-   <origin xyz="-0.005 0.0 0.0" rpy="0 0 0" />
+   <box size="0.06 0.06 0.01" />
+   <origin xyz="0.0 0.0 0.027" rpy="0 0 0"/>
+   <origin xyz="0.0 0.0 0.027" rpy="0 0 0" />
    <inertia ixx="0.0001"  ixy="0"  ixz="0" iyy="0.0001" iyz="0" izz="0.0001" />
 </xacro:my_link>
@@ -33,4 +34,14 @@
     <parent link="base_laser"/>
     <child link="lasertop"/>
+</joint>
+<xacro:my_link name="lasermount" mass="0.01" color="White">
+   <box size="0.01 0.06 0.035" />
+   <origin xyz="-0.025 0.0 -0.0725" rpy="0 0 0"/>
+   <origin xyz="-0.025 0.0 -0.0725" rpy="0 0 0" />
+   <inertia ixx="0.0001"  ixy="0"  ixz="0" iyy="0.0001" iyz="0" izz="0.0001" />
+</xacro:my_link>
+<joint name="lasermount_joint" type="fixed">
+    <parent link="base_laser"/>
+    <child link="lasermount"/>
 </joint>
 <!--the tue logo in front of the laser-->

Commit message: Modified the color orange of the laser + cleaned up some components

File: urdf/sergio.urdf (robot description, URDF)
Before this commit: robot sergio, 58 links, 57 joints
Links:
- link torso_laser_mount: geometry collision box size=0.0 0.0 0.0; visual box size=0.0 0.0 0.0

File: urdf/xacro/sergio.urdf.xacro (robot description, xacro)
@@ -14,5 +14,4 @@
     <xacro:include filename="$(find amigo_description)/urdf/xacro/macro_definitions.xacro" />
     <!--get custom materials -->
-    <!--<xacro:include filename="$(find amigo_robot_model)/description/materials.urdf.xacro" />-->
     <xacro:include filename="$(find amigo_description)/urdf/xacro/materials.urdf.xacro" />
     <!--========BUILD BASE======-->
@@ -28,6 +27,4 @@
     <!--========BUILD KINECT======-->
     <xacro:include filename="$(find sergio_description)/urdf/xacro/kinect/top_kinect.urdf.xacro" />
-    <!--========BUILD TORSO LASER JOINT======-->
-    <xacro:include filename="$(find sergio_description)/urdf/xacro/laser/torso_laser_joint.urdf.xacro" />
     <!--========BUILD LASERS======-->
     <!--<xacro:include filename="$(find sergio_description)/urdf/xacro/laser/base_laser.urdf.xacro" />-->

File: urdf/xacro/torso/torso.urdf.xacro (robot description, xacro)
@@ -32,4 +32,11 @@
         <inertia ixx="0.001"  ixy="0"  ixz="0" iyy="0.001" iyz="0" izz="0.001" /><!--Estimate inertia-->
     </xacro:my_link>
+    <!-- torso laser joint (center is the center of rotation of the laser)-->
+	<xacro:my_link name="torso_laser_mount" mass="0.01" color="Black">
+	   <box size="0.0 0.0 0.0" />
+	   <origin xyz="0.0 0.0 0.0" rpy="0 0 0"/>
+	   <origin xyz="0.0 0.0 0.0" rpy="0 0 0" />
+	   <inertia ixx="0.0001"  ixy="0"  ixz="0" iyy="0.0001" iyz="0" izz="0.0001" />
+	</xacro:my_link>
     <!-- joints -->
     <joint name="torso_mount_joint" type="fixed">
@@ -59,3 +66,11 @@
         <!--<limit effort="1000" velocity="10" lower="2.36" upper="2.36" />--> <!--TEMP: fixed joint positions until control is fixed-->
     </xacro:my_joint>
+    <joint name="laser_tilt_joint" type="revolute" >
+	   <parent link="trunk" />
+	   <child link="torso_laser_mount"/>
+	   <origin xyz="0.3163 0.0 -0.0671" rpy="3.14 1.57 0.0 "/>
+	   <dynamics damping="0.1" friction="0"/><!--ToDo: update-->
+	   <axis xyz="0 1 0"/>
+	   <limit effort="13.4" velocity="1.0" lower="-0.3" upper="0.3" /> <!--ToDo: update-->
+	</joint>
 </robot>
