Commit message: Adjusted the torso joint limits on the basis of the torso calibration. Set the initial position of the torso (by publish_jointstates.py) to a more natural looking position

File: urdf/sergio.urdf (robot description, URDF)
Before this commit: robot sergio, 58 links, 57 joints
Joints:
- joint ankle_joint: limit lower=0.0 upper=1.059 effort=1000 velocity=0.265 -> lower=0.05 upper=1.001 effort=1000 velocity=0.265
- joint hip_joint: limit lower=0.85 upper=2.36 effort=1000 velocity=0.375 -> lower=1.01 upper=2.31 effort=1000 velocity=0.375
- joint knee_joint: limit lower=0.0 upper=2.158 effort=1000 velocity=0.539 -> lower=0.18 upper=2.06 effort=1000 velocity=0.539

File: urdf/xacro/torso/torso.urdf.xacro (robot description, xacro)
@@ -49,5 +49,5 @@
         <dynamics damping="6.0" friction="4.87"/><!-- ToDo: adjust dynamics-->
         <axis xyz="0 -1 0"/><!--ToDo: DH parameters?-->
-        <limit effort="1000" velocity="0.265" lower="0.0" upper="1.059" /> <!--ToDo: adjust parameters-->
+        <limit effort="1000" velocity="0.265" lower="0.05" upper="1.001" /> <!--ToDo: adjust parameters-->
         <!--<limit effort="1000" velocity="10" lower="0.87" upper="0.87" />--> <!--TEMP: fixed joint positions until control is fixed-->
     </xacro:my_joint>
@@ -56,5 +56,5 @@
         <dynamics damping="6.0" friction="4.87"/><!-- ToDo: adjust dynamics-->
         <axis xyz="0 -1 0"/><!--ToDo: DH parameters?-->
-        <limit effort="1000" velocity="0.539" lower="0.0" upper="2.158" /> <!--ToDo: adjust parameters -->
+        <limit effort="1000" velocity="0.539" lower="0.18" upper="2.06" /> <!--ToDo: adjust parameters -->
         <!--<limit effort="1000" velocity="10" lower="2.0" upper="2.0" />--> <!--TEMP: fixed joint positions until control is fixed -->
     </xacro:my_joint>
@@ -63,5 +63,5 @@
         <dynamics damping="6.0" friction="4.87"/><!-- ToDo: adjust dynamics-->
         <axis xyz="0 -1 0"/><!--ToDo: DH parameters?-->
-        <limit effort="1000" velocity="0.375" lower="0.85" upper="2.36" /> <!--ToDo: adjust parameters --><!--Velocity: move in 4 s-->
+        <limit effort="1000" velocity="0.375" lower="1.01" upper="2.31" /> <!--ToDo: adjust parameters --><!--Velocity: move in 4 s-->
         <!--<limit effort="1000" velocity="10" lower="2.36" upper="2.36" />--> <!--TEMP: fixed joint positions until control is fixed-->
     </xacro:my_joint>

Commit message: moved sonar sensors to the side

File: urdf/sergio.urdf (robot description, URDF)
Before this commit: robot sergio, 63 links, 62 joints
Links:
- removed link base_sonar5
Joints:
- removed joint base_sonar5_joint
- joint base_sonar1_joint: origin xyz=-0.380 0.0 0.0 rpy=0.0 0 3.14 -> xyz=0.370 0.3115 0.0 rpy=0.0 0 1.57
- joint base_sonar2_joint: origin xyz=-0.380 0.311 0.0 rpy=0.0 0 3.14 -> xyz=0.124 0.3115 0.0 rpy=0.0 0 1.57
- joint base_sonar3_joint: origin xyz=-0.380 -0.311 0.0 rpy=0.0 0 3.14 -> xyz=-0.124 0.3115 0.0 rpy=0.0 0 1.57
- joint base_sonar4_joint: origin xyz=-0.370 -0.3115 0.0 rpy=0.0 0 -1.57 -> xyz=-0.370 0.3115 0.0 rpy=0.0 0 1.57

File: urdf/xacro/ultrasone/ultrasone.urdf.xacro (robot description, xacro)
@@ -8,5 +8,6 @@
     <parent link="base"/>
     <child link="base_sonar1"/>
-    <origin xyz="-0.380 0.0 0.0" rpy="0.0 0 3.14"/>
+    <!--<origin xyz="-0.380 0.0 0.0" rpy="0.0 0 3.14"/>-->
+    <origin xyz="0.370 0.3115 0.0" rpy="0.0 0 1.57"/>
 </joint>
 <!-- visual of the ultrasone sensor -->
@@ -21,5 +22,6 @@
     <parent link="base"/>
     <child link="base_sonar2"/>
-    <origin xyz="-0.380 0.311 0.0" rpy="0.0 0 3.14"/>
+    <!--<origin xyz="-0.380 0.311 0.0" rpy="0.0 0 3.14"/>-->
+    <origin xyz="0.124 0.3115 0.0" rpy="0.0 0 1.57"/>
 </joint>
 <!-- visual of the ultrasone sensor -->
@@ -34,5 +36,6 @@
     <parent link="base"/>
     <child link="base_sonar3"/>
-    <origin xyz="-0.380 -0.311 0.0" rpy="0.0 0 3.14"/>
+    <!--<origin xyz="-0.380 -0.311 0.0" rpy="0.0 0 3.14"/>-->
+    <origin xyz="-0.124 0.3115 0.0" rpy="0.0 0 1.57"/>
 </joint>
 <!-- visual of the ultrasone sensor -->
@@ -47,5 +50,5 @@
     <parent link="base"/>
     <child link="base_sonar4"/>
-    <origin xyz="-0.370 -0.3115 0.0" rpy="0.0 0 -1.57"/>
+    <origin xyz="-0.370 0.3115 0.0" rpy="0.0 0 1.57"/>
 </joint>
 <!-- visual of the ultrasone sensor -->
@@ -56,16 +59,3 @@
    <inertia ixx="0.0001"  ixy="0"  ixz="0" iyy="0.0001" iyz="0" izz="0.0001" />
 </xacro:my_link>
-<!-- origin of the ultrasone sensor-->
-<joint name="base_sonar5_joint" type="fixed" >
-    <parent link="base"/>
-    <child link="base_sonar5"/>
-    <origin xyz="-0.370 0.3115 0.0" rpy="0.0 0 1.57"/>
-</joint>
-<!-- visual of the ultrasone sensor -->
-<xacro:my_link name="base_sonar5" mass="0.05" color="Red">
-   <cylinder radius="0.005" length="0.01" />
-   <origin xyz="0.005 0.0 0.0" rpy="0 0.0 0"/>
-   <origin xyz="0.005 0.0 0.0" rpy="0 1.57 0" />
-   <inertia ixx="0.0001"  ixy="0"  ixz="0" iyy="0.0001" iyz="0" izz="0.0001" />
-</xacro:my_link>
 </robot>

Commit message: Corrected laser offset from 0.055 to 0.0605 as found in the specifications online

File: urdf/sergio.urdf (robot description, URDF)
Before this commit: robot sergio, 58 links, 57 joints
Joints:
- joint base_lasercenter_joint: origin xyz=0.03 0.0 0.09 rpy=0.0 0.0 0.0 -> xyz=0.03 0.0 0.0955 rpy=0.0 0.0 0.0
- joint base_lasertop_joint: origin xyz=0.0 0.0 0.023 rpy=0 0 0 -> xyz=0.0 0.0 0.0175 rpy=0 0 0
- joint torso_lasercenter_joint: origin xyz=0.0 0.0 0.0015 rpy=0.0 0.0 0.0 -> xyz=0.0 0.0 -0.004 rpy=0.0 0.0 0.0
- joint torso_lasertop_joint: origin xyz=0.0 0.0 0.023 rpy=0 0 0 -> xyz=0.0 0.0 0.0175 rpy=0 0 0

File: urdf/xacro/laser/laser.urdf.xacro (robot description, xacro)
@@ -7,15 +7,8 @@
 @param laser_name, is used to locate the sensor
 @param laser_parent, parent
-@param laser_xyz, transform from parent to laser center (center is at l=0.3 w=0.3 h=55)
+@param laser_xyz, transform from parent to laser center (center is at l=0.3 w=0.3 h=60.5)
 @param laser_rpy, rotation from parent to laser center (x points forward, z to the top)
 -->
  <xacro:macro name="laser" params="laser_name laser_parent laser_xyz laser_rpy">
-<!-- link visualize the black part of the laser-->
-<xacro:my_link name="${laser_name}_laser" mass="0.5" color="Black">
-   <box size="0.06 0.06 0.069" />
-   <origin xyz="0.0 0.0 -0.0205" rpy="0 0 0"/>
-   <origin xyz="0.0 0.0 -0.0205" rpy="0 0 0" />
-   <inertia ixx="0.0001"  ixy="0"  ixz="0" iyy="0.0001" iyz="0" izz="0.0001" />
-</xacro:my_link>
 <!-- joint origin of the laser range finder -->
 <joint name="${laser_name}_lasercenter_joint" type="fixed">
@@ -24,12 +17,22 @@
     <origin xyz="${laser_xyz}" rpy="${laser_rpy}"/>
 </joint>
+<!-- link visualize the black part of the laser-->
+<xacro:my_link name="${laser_name}_laser" mass="0.5" color="Black">
+   <box size="0.06 0.06 0.069" />
+   <!--<origin xyz="0.0 0.0 -0.0205" rpy="0 0 0"/>
+   <origin xyz="0.0 0.0 -0.0205" rpy="0 0 0" />-->
+   <origin xyz="0.0 0.0 -0.026" rpy="0 0 0"/>
+   <origin xyz="0.0 0.0 -0.026" rpy="0 0 0" />
+   <inertia ixx="0.0001"  ixy="0"  ixz="0" iyy="0.0001" iyz="0" izz="0.0001" />
+</xacro:my_link>
 <!-- joint origin of the orange top -->
 <joint name="${laser_name}_lasertop_joint" type="fixed">
     <parent link="${laser_name}_laser"/>
     <child link="${laser_name}_lasertop"/>
-    <origin xyz="0.0 0.0 0.023" rpy="0 0 0"/>
+    <!--<origin xyz="0.0 0.0 0.023" rpy="0 0 0"/>-->
+    <origin xyz="0.0 0.0 0.0175" rpy="0 0 0"/>
 </joint>
 <!-- link visual of the orange top -->
-<xacro:my_link name="${laser_name}_lasertop" mass="0.01" color="Orange"><!--Changed color to red to make it work-->
+<xacro:my_link name="${laser_name}_lasertop" mass="0.01" color="Orange">
    <box size="0.06 0.06 0.018" />
    <origin xyz="0.0 0.0 0.0" rpy="0 0 0"/>

File: urdf/xacro/sergio.urdf.xacro (robot description, xacro)
@@ -30,6 +30,6 @@
     <!--<xacro:include filename="$(find sergio_description)/urdf/xacro/laser/base_laser.urdf.xacro" />-->
     <xacro:include filename="$(find sergio_description)/urdf/xacro/laser/laser.urdf.xacro" />
-    <xacro:laser laser_name="base" laser_parent="laser_mount" laser_xyz="0.03 0.0 0.09" laser_rpy="0.0 0.0 0.0"  />
-    <xacro:laser laser_name="torso" laser_parent="torso_laser_mount" laser_xyz="0.0 0.0 0.0015" laser_rpy="0.0 0.0 0.0"  />
+    <xacro:laser laser_name="base" laser_parent="laser_mount" laser_xyz="0.03 0.0 0.0955" laser_rpy="0.0 0.0 0.0"  />
+    <xacro:laser laser_name="torso" laser_parent="torso_laser_mount" laser_xyz="0.0 0.0 -0.004" laser_rpy="0.0 0.0 0.0"  />
     <!-- GAZEBO -->
     <xacro:include filename="$(find sergio_description)/urdf/xacro/gazebo.urdf.xacro"/>

Commit message: calibrated the torso laser

File: urdf/sergio.urdf (robot description, URDF)
Before this commit: robot sergio, 58 links, 57 joints
Joints:
- joint laser_tilt_joint: limit lower=-0.3 upper=0.3 effort=13.4 velocity=1.0 -> lower=0.0 upper=0.3173 effort=13.4 velocity=1.0; origin xyz=0.3163 0.0 -0.0671 rpy=3.14 1.57 0.0  -> xyz=0.3163 0.0 -0.0671 rpy=3.14 1.406 0.0 

File: urdf/xacro/torso/torso.urdf.xacro (robot description, xacro)
@@ -69,8 +69,8 @@
 	   <parent link="trunk" />
 	   <child link="torso_laser_mount"/>
-	   <origin xyz="0.3163 0.0 -0.0671" rpy="3.14 1.57 0.0 "/>
+	   <origin xyz="0.3163 0.0 -0.0671" rpy="3.14 1.406 0.0 "/>
 	   <dynamics damping="0.1" friction="0"/><!--ToDo: update-->
 	   <axis xyz="0 1 0"/>
-	   <limit effort="13.4" velocity="1.0" lower="-0.3" upper="0.3" /> <!--ToDo: update-->
+	   <limit effort="13.4" velocity="1.0" lower="0.0" upper="0.3173" /> <!--ToDo: update-->
 	</joint>
 </robot>

Commit message: Sergio has larger base visual for better self-filtering

File: urdf/sergio.urdf (robot description, URDF)
Before this commit: robot sergio, 58 links, 57 joints
Links:
- link base: geometry collision box size=0.713 0.650 0.3; visual box size=0.713 0.650 0.3

File: urdf/xacro/base/base.urdf.xacro (robot description, xacro)
@@ -13,5 +13,7 @@
     <!--base block-->
     <xacro:my_link name="base" mass="0.1" color="White"><!--ToDo: estimate mass-->
-        <box size="0.713 0.500 0.11" /><!--ToDo: check dimensions, adjust height-->
+        <!--box size="0.713 0.500 0.11" /--><!--ToDo: check dimensions, adjust height-->
+        <!-- Large box for better self-filtering -->
+        <box size="0.713 0.650 0.3" />
         <origin xyz="-0.0235 0.0 0.0" rpy="0 0 0"/>
         <origin xyz="-0.0235 0.0 0.0" rpy="0 0 0"/>

Commit message: Now complete independent of amigo_description

File: urdf/sergio.urdf (robot description, URDF)
Before this commit: robot sergio, 58 links, 57 joints
Links:
- link fore_arm_left: geometry collision mesh filename=package://sergio_description/media/meshes/forearmtextured.d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 scale=0.0004 0.0004 0.0004; visual mesh filename=package://sergio_description/media/meshes/forearmtextured.d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 scale=0.0004 0.0004 0.0004
- link fore_arm_right: geometry collision mesh filename=package://sergio_description/media/meshes/forearmtextured.d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 scale=0.0004 0.0004 0.0004; visual mesh filename=package://sergio_description/media/meshes/forearmtextured.d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 scale=0.0004 0.0004 0.0004
- link upper_arm_left: geometry collision mesh filename=package://sergio_description/media/meshes/upperarmtextured.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 scale=0.0004 0.0004 0.0004; visual mesh filename=package://sergio_description/media/meshes/upperarmtextured.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 scale=0.0004 0.0004 0.0004
- link upper_arm_right: geometry collision mesh filename=package://sergio_description/media/meshes/upperarmtextured.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 scale=0.0004 0.0004 0.0004; visual mesh filename=package://sergio_description/media/meshes/upperarmtextured.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 scale=0.0004 0.0004 0.0004

File: urdf/xacro/arms/arm.urdf.xacro (robot description, xacro)
@@ -42,5 +42,5 @@
    <origin xyz="-0.00959 -0.19131 -0.00001" rpy="0 0 3.1415" />
    <inertia ixx="0.027"  ixy="0"  ixz="0" iyy="0.45993" iyz="0" izz="0.004" />
-   <mesh filename="package://amigo_description/media/meshes/upperarmtextured.dae" scale="0.0004 0.0004 0.0004"/>
+   <mesh filename="package://sergio_description/media/meshes/upperarmtextured.dae" scale="0.0004 0.0004 0.0004"/>
 </xacro:my_link_texturedmesh>
 <!--the elbow
@@ -57,5 +57,5 @@
    <origin xyz="0.00425 -0.14868 0.00547" rpy="0 -1.5708 0" />
    <inertia ixx="0.001"  ixy="0"  ixz="0" iyy="0.5" iyz="0" izz="0.001" />
-   <mesh filename="package://amigo_description/media/meshes/forearmtextured.dae" scale="0.0004 0.0004 0.0004"/>
+   <mesh filename="package://sergio_description/media/meshes/forearmtextured.dae" scale="0.0004 0.0004 0.0004"/>
 </xacro:my_link_texturedmesh>
 <!--the wrist

File: urdf/xacro/head/head.urdf.xacro (robot description, xacro)
@@ -32,5 +32,5 @@
    <origin xyz="0.0 -0.0 0.015" rpy="0 0 0" />
    <inertia ixx="0.001"  ixy="0"  ixz="0" iyy="0.001" iyz="0" izz="0.001" />
-   <mesh filename="package://amigo_description/media/meshes/necktilttextured.dae" scale="0.004 0.004 0.004"/>
+   <mesh filename="package://sergio_description/media/meshes/necktilttextured.dae" scale="0.004 0.004 0.004"/>
 </xacro:my_link_texturedmesh>-->
 <xacro:my_link name="neck_tilt" mass="0.05" color="White">
@@ -45,5 +45,5 @@
    <origin xyz="0.0 0.0 0.141" rpy="0 0 -1.5708"/>
    <inertia ixx="0"  ixy="0"  ixz="0" iyy="0" iyz="0" izz="0" />
-   <mesh filename="package://amigo_description/media/meshes/headtextured.dae" scale="0.0004 0.0004 0.0004"/>
+   <mesh filename="package://sergio_description/media/meshes/headtextured.dae" scale="0.0004 0.0004 0.0004"/>
   </my_link_texturedmesh>-->
   <my_link name="head" mass="0" color="White">

File: urdf/xacro/kinect/top_kinect.urdf.xacro (robot description, xacro)
@@ -22,5 +22,5 @@
       <geometry>
 		<!--<box size="0.001 0.001 0.001"/>--><!--Changed to 0.001 because otherwise it doesn't work-->
-        <!--mesh filename="package://amigo_description/kinect/meshes/kinect.dae" scale="0.001 0.001 0.001"/-->
+        <!--mesh filename="package://sergio_description/kinect/meshes/kinect.dae" scale="0.001 0.001 0.001"/-->
         <mesh filename="package://sergio_description/media/meshes/kinect_without_base.dae"/>
       </geometry>

File: urdf/xacro/macro_definitions.xacro (robot description, xacro)
@@ -46,5 +46,5 @@
      <xacro:insert_block name="type" />
      </geometry>
-     <material name="${texture}">
+     <material name="amigo_description/${texture}">
      </material>
     </visual>
@@ -57,5 +57,5 @@
   </link>
 <gazebo reference="${name}">
-      <material>sergio_robot_model/${texture}</material>
+      <material>amigo_description/${texture}</material>
       <turnGravityOff>false</turnGravityOff>
     </gazebo>
@@ -124,5 +124,5 @@
      <xacro:insert_block name="mesh" />
      </geometry>
-     <material name="${texture}"/>
+     <material name="amigo_description/${texture}"/>
     </visual>
     <collision>
@@ -134,5 +134,5 @@
   </link>
 <gazebo reference="${name}">
-	  <material>sergio_robot_model/${texture}</material>
+	  <material>amigo_description/${texture}</material>
       <turnGravityOff>false</turnGravityOff>
     </gazebo>
@@ -151,5 +151,5 @@
      <xacro:insert_block name="mesh" />
      </geometry>
-     <material name="${texture}"/>
+     <material name="amigo_description/${texture}"/>
     </visual>
     <collision>
@@ -161,5 +161,5 @@
   </link>
 <gazebo reference="${name}">
-	  <material>sergio_robot_model/${texture}</material>
+	  <material>amigo_description/${texture}</material>
       <turnGravityOff>false</turnGravityOff>
     </gazebo>

File: urdf/xacro/sergio.urdf.xacro (robot description, xacro)
@@ -11,8 +11,8 @@
     <!--Definitions from default package?-->
     <!--get link & joint definitions -->
-    <!--<xacro:include filename="$(find amigo_robot_model)/description/definitions.xacro" />-->
-    <xacro:include filename="$(find amigo_description)/urdf/xacro/macro_definitions.xacro" />
+    <!--<xacro:include filename="$(find sergio_robot_model)/description/definitions.xacro" />-->
+    <xacro:include filename="$(find sergio_description)/urdf/xacro/macro_definitions.xacro" />
     <!--get custom materials -->
-    <xacro:include filename="$(find amigo_description)/urdf/xacro/materials.urdf.xacro" />
+    <xacro:include filename="$(find sergio_description)/urdf/xacro/materials.urdf.xacro" />
     <!--========BUILD BASE======-->
     <xacro:include filename="$(find sergio_description)/urdf/xacro/base/base.urdf.xacro" />

Commit message: modified torso limits to meet the current hardware settings

File: urdf/sergio.urdf (robot description, URDF)
Before this commit: robot sergio, 58 links, 57 joints
Joints:
- joint ankle_joint: limit lower=0.05 upper=1.001 effort=1000 velocity=0.265 -> lower=0.152 upper=1.00 effort=1000 velocity=0.265
- joint hip_joint: limit lower=1.01 upper=2.31 effort=1000 velocity=0.375 -> lower=1.007 upper=2.31 effort=1000 velocity=0.375
- joint knee_joint: limit lower=0.18 upper=2.06 effort=1000 velocity=0.539 -> lower=0.419 upper=2.059 effort=1000 velocity=0.539

File: urdf/xacro/torso/torso.urdf.xacro (robot description, xacro)
@@ -49,5 +49,5 @@
         <dynamics damping="6.0" friction="4.87"/><!-- ToDo: adjust dynamics-->
         <axis xyz="0 -1 0"/><!--ToDo: DH parameters?-->
-        <limit effort="1000" velocity="0.265" lower="0.05" upper="1.001" /> <!--ToDo: adjust parameters-->
+        <limit effort="1000" velocity="0.265" lower="0.152" upper="1.00" /> <!--ToDo: adjust parameters-->
         <!--<limit effort="1000" velocity="10" lower="0.87" upper="0.87" />--> <!--TEMP: fixed joint positions until control is fixed-->
     </xacro:my_joint>
@@ -56,5 +56,5 @@
         <dynamics damping="6.0" friction="4.87"/><!-- ToDo: adjust dynamics-->
         <axis xyz="0 -1 0"/><!--ToDo: DH parameters?-->
-        <limit effort="1000" velocity="0.539" lower="0.18" upper="2.06" /> <!--ToDo: adjust parameters -->
+        <limit effort="1000" velocity="0.539" lower="0.419" upper="2.059" /> <!--ToDo: adjust parameters -->
         <!--<limit effort="1000" velocity="10" lower="2.0" upper="2.0" />--> <!--TEMP: fixed joint positions until control is fixed -->
     </xacro:my_joint>
@@ -63,5 +63,5 @@
         <dynamics damping="6.0" friction="4.87"/><!-- ToDo: adjust dynamics-->
         <axis xyz="0 -1 0"/><!--ToDo: DH parameters?-->
-        <limit effort="1000" velocity="0.375" lower="1.01" upper="2.31" /> <!--ToDo: adjust parameters --><!--Velocity: move in 4 s-->
+        <limit effort="1000" velocity="0.375" lower="1.007" upper="2.31" /> <!--ToDo: adjust parameters --><!--Velocity: move in 4 s-->
         <!--<limit effort="1000" velocity="10" lower="2.36" upper="2.36" />--> <!--TEMP: fixed joint positions until control is fixed-->
     </xacro:my_joint>

Commit message: Reduced base block

File: urdf/sergio.urdf (robot description, URDF)
Before this commit: robot sergio, 58 links, 57 joints
Links:
- link base: geometry collision box size=0.713 0.500 0.11; visual box size=0.713 0.500 0.11

File: urdf/xacro/base/base.urdf.xacro (robot description, xacro)
@@ -13,7 +13,7 @@
     <!--base block-->
     <xacro:my_link name="base" mass="0.1" color="White"><!--ToDo: estimate mass-->
-        <!--box size="0.713 0.500 0.11" /--><!--ToDo: check dimensions, adjust height-->
+        <box size="0.713 0.500 0.11"/><!--ToDo: check dimensions, adjust height-->
         <!-- Large box for better self-filtering -->
-        <box size="0.713 0.650 0.3" />
+        <!--<box size="0.713 0.650 0.3" />-->
         <origin xyz="-0.0235 0.0 0.0" rpy="0 0 0"/>
         <origin xyz="-0.0235 0.0 0.0" rpy="0 0 0"/>
