Commit message: Added wheels

File: urdf/sergio.urdf (robot description, URDF)
Before this commit: robot sergio, 58 links, 57 joints
Links:
- added link wheel_left_front, mass 0; collision cylinder length=0.06 radius=0.075; visual cylinder length=0.06 radius=0.075
- added link wheel_left_rear, mass 0; collision cylinder length=0.06 radius=0.075; visual cylinder length=0.06 radius=0.075
- added link wheel_right_front, mass 0; collision cylinder length=0.06 radius=0.075; visual cylinder length=0.06 radius=0.075
- added link wheel_right_rear, mass 0; collision cylinder length=0.06 radius=0.075; visual cylinder length=0.06 radius=0.075
Joints:
- added joint wheel_left_front_joint: type fixed, parent base_link, child wheel_left_front, origin xyz=0.275 0.275 0.075 rpy=1.57 0.0 0.0
- added joint wheel_left_rear_joint: type fixed, parent base_link, child wheel_left_rear, origin xyz=-0.275 0.275 0.075 rpy=1.57 0.0 0.0
- added joint wheel_right_front_joint: type fixed, parent base_link, child wheel_right_front, origin xyz=0.275 -0.275 0.075 rpy=1.57 0.0 0.0
- added joint wheel_right_rear_joint: type fixed, parent base_link, child wheel_right_rear, origin xyz=-0.275 -0.275 0.075 rpy=1.57 0.0 0.0

File: urdf/xacro/base/base.urdf.xacro (robot description, xacro)
@@ -47,4 +47,29 @@
         <inertia ixx="0.0001"  ixy="0"  ixz="0" iyy="0.0001" iyz="0" izz="0.0001" />
     </xacro:my_link>
+    <!-- wheels -->
+    <xacro:my_link name="wheel_right_front" mass="0" color="DarkGrey">
+       <cylinder radius="0.075" length="0.06" />
+       <origin xyz="0.0 0.0 0.0" rpy="0.0 0 0"/>
+       <origin xyz="0.0 0.0 0.0" rpy="0.0 0 0" />
+       <inertia ixx="0"  ixy="0"  ixz="0" iyy="0" iyz="0" izz="0" />
+    </xacro:my_link>
+    <xacro:my_link name="wheel_left_front" mass="0" color="DarkGrey">
+       <cylinder radius="0.075" length="0.06" />
+       <origin xyz="0.0 0.0 0.0" rpy="0.0 0 0"/>
+       <origin xyz="0.0 0.0 0.0" rpy="0.0 0 0" />
+       <inertia ixx="0"  ixy="0"  ixz="0" iyy="0" iyz="0" izz="0" />
+    </xacro:my_link>
+    <xacro:my_link name="wheel_right_rear" mass="0" color="DarkGrey">
+       <cylinder radius="0.075" length="0.06" />
+       <origin xyz="0.0 0.0 0.0" rpy="0.0 0 0"/>
+       <origin xyz="0.0 0.0 0.0" rpy="0.0 0 0" />
+       <inertia ixx="0"  ixy="0"  ixz="0" iyy="0" iyz="0" izz="0" />
+    </xacro:my_link>
+    <xacro:my_link name="wheel_left_rear" mass="0" color="DarkGrey">
+       <cylinder radius="0.075" length="0.06" />
+       <origin xyz="0.0 0.0 0.0" rpy="0.0 0 0"/>
+       <origin xyz="0.0 0.0 0.0" rpy="0.0 0 0" />
+       <inertia ixx="0"  ixy="0"  ixz="0" iyy="0" iyz="0" izz="0" />
+    </xacro:my_link>
     <!-- joints -->
     <joint name="base_link_joint" type="fixed">
@@ -76,3 +101,23 @@
         <origin xyz="0.2995 0.0 0.055" rpy="0.0 0.0 0.0"/>
     </joint>
+    <joint name="wheel_right_front_joint" type="fixed">
+        <parent link="base_link"/>
+        <child link="wheel_right_front"/>
+        <origin xyz="0.275 -0.275 0.075" rpy="1.57 0.0 0.0"/>
+    </joint>
+    <joint name="wheel_left_front_joint" type="fixed">
+        <parent link="base_link"/>
+        <child link="wheel_left_front"/>
+        <origin xyz="0.275 0.275 0.075" rpy="1.57 0.0 0.0"/>
+    </joint>
+    <joint name="wheel_right_rear_joint" type="fixed">
+        <parent link="base_link"/>
+        <child link="wheel_right_rear"/>
+        <origin xyz="-0.275 -0.275 0.075" rpy="1.57 0.0 0.0"/>
+    </joint>
+    <joint name="wheel_left_rear_joint" type="fixed">
+        <parent link="base_link"/>
+        <child link="wheel_left_rear"/>
+        <origin xyz="-0.275 0.275 0.075" rpy="1.57 0.0 0.0"/>
+    </joint>
 </robot>

File: urdf/xacro/materials.urdf.xacro (robot description, xacro)
@@ -29,4 +29,7 @@
     <color rgba="0.6 0.6 0.6 1.0"/>
   </material>
+  <material name="DarkGrey">
+    <color rgba="0.25 0.25 0.25 1.0"/>
+  </material>
   <material name="Orange">
     <color rgba="1.0 0.33 0.0 1.0"/>

Commit message: Updated arm description

File: urdf/sergio.urdf (robot description, URDF)
Before this commit: robot sergio, 62 links, 61 joints
Links:
- added link elbow_extra_block2_left, mass 0.01; collision cylinder length=0.08 radius=0.03; visual cylinder length=0.08 radius=0.03
- added link elbow_extra_block2_right, mass 0.01; collision cylinder length=0.08 radius=0.03; visual cylinder length=0.08 radius=0.03
- added link elbow_extra_block_left, mass 0.01; collision box size=0.015 0.08 0.06; visual box size=0.015 0.08 0.06
- added link elbow_extra_block_right, mass 0.01; collision box size=0.015 0.08 0.06; visual box size=0.015 0.08 0.06
- added link fore_arm_top_left, mass 0.01; collision cylinder length=0.01 radius=0.037; visual cylinder length=0.01 radius=0.037
- added link fore_arm_top_right, mass 0.01; collision cylinder length=0.01 radius=0.037; visual cylinder length=0.01 radius=0.037
- added link pitch_axis_left, mass 0.15; collision cylinder length=0.220 radius=0.035; visual cylinder length=0.220 radius=0.035
- added link pitch_axis_right, mass 0.15; collision cylinder length=0.220 radius=0.035; visual cylinder length=0.220 radius=0.035
- added link upper_arm_top_left, mass 0.01; collision cylinder length=0.02 radius=0.0561; visual cylinder length=0.02 radius=0.0561
- added link upper_arm_top_right, mass 0.01; collision cylinder length=0.02 radius=0.0561; visual cylinder length=0.02 radius=0.0561
- added link wrist_to_hand_block_left, mass 0.01; collision box size=0.03 0.02 0.038; visual box size=0.03 0.02 0.038
- added link wrist_to_hand_block_right, mass 0.01; collision box size=0.03 0.02 0.038; visual box size=0.03 0.02 0.038
- added link wrist_visual_left, mass 0.01; collision cylinder length=0.06 radius=0.018; visual cylinder length=0.06 radius=0.018
- added link wrist_visual_right, mass 0.01; collision cylinder length=0.06 radius=0.018; visual cylinder length=0.06 radius=0.018
- link shoulder_mount_left: geometry collision cylinder length=0.160 radius=0.075; visual cylinder length=0.160 radius=0.075
- link shoulder_mount_right: geometry collision cylinder length=0.160 radius=0.075; visual cylinder length=0.160 radius=0.075
Joints:
- added joint elbow_extra_block2_joint_left: type fixed, parent upper_arm_left, child elbow_extra_block2_left, origin xyz=0.0 -0.31 0.0 rpy=-1.5708 0 0
- added joint elbow_extra_block2_joint_right: type fixed, parent upper_arm_right, child elbow_extra_block2_right, origin xyz=0.0 -0.31 0.0 rpy=-1.5708 0 0
- added joint elbow_extra_block_joint_left: type fixed, parent upper_arm_left, child elbow_extra_block_left, origin xyz=0.0 -0.31 0.0 rpy=-1.5708 0 0
- added joint elbow_extra_block_joint_right: type fixed, parent upper_arm_right, child elbow_extra_block_right, origin xyz=0.0 -0.31 0.0 rpy=-1.5708 0 0
- added joint fore_arm_top_joint_left: type fixed, parent fore_arm_left, child fore_arm_top_left, origin xyz=0.002 -0.011 0.0 rpy=1.5708 0 0
- added joint fore_arm_top_joint_right: type fixed, parent fore_arm_right, child fore_arm_top_right, origin xyz=0.002 -0.011 0.0 rpy=1.5708 0 0
- added joint pitch_axis_joint_left: type fixed, parent trunk, child pitch_axis_left, origin xyz=0.470 0.22 0.0 rpy=3.14 0 0.0
- added joint pitch_axis_joint_right: type fixed, parent trunk, child pitch_axis_right, origin xyz=0.470 -0.22 0.0 rpy=3.14 0 0.0
- added joint upper_arm_top_joint_left: type fixed, parent upper_arm_left, child upper_arm_top_left, origin xyz=-0.01 -0.1 0.0 rpy=1.5708 0 0.0
- added joint upper_arm_top_joint_right: type fixed, parent upper_arm_right, child upper_arm_top_right, origin xyz=-0.01 -0.1 0.0 rpy=1.5708 0 0.0
- added joint wrist_to_hand_block_joint_left: type fixed, parent wrist_link6_left, child wrist_to_hand_block_left, origin xyz=0.0 0.0 0.0 rpy=0 0 0
- added joint wrist_to_hand_block_joint_right: type fixed, parent wrist_link6_right, child wrist_to_hand_block_right, origin xyz=0.0 0.0 0.0 rpy=0 0 0
- added joint wrist_visual_joint_left: type fixed, parent wrist_link6_left, child wrist_visual_left, origin xyz=-0.02 0.0 0.0 rpy=1.5708 0 0
- added joint wrist_visual_joint_right: type fixed, parent wrist_link6_right, child wrist_visual_right, origin xyz=-0.02 0.0 0.0 rpy=1.5708 0 0

File: urdf/xacro/arms/arm.urdf.xacro (robot description, xacro)
@@ -17,5 +17,5 @@
 <!--the end of the clavicle, yaw rotation-->
 <xacro:my_link name="shoulder_mount_${whichside}" mass="0.15" color="White">
-   <cylinder radius="0.075" length="0.140" /><!-- Length of tube should be correct (see report), origin depends on placement -->
+   <cylinder radius="0.075" length="0.160" /><!-- Length of tube should be correct (see report), origin depends on placement -->
    <origin xyz="0.0 ${sidesign*-0.155} 0.0" rpy="1.57 0 0"/>
    <origin xyz="0.0 ${sidesign*-0.155} 0.0" rpy="1.57 0 0 " />

File: urdf/xacro/sergio.urdf.xacro (robot description, xacro)
@@ -23,4 +23,8 @@
     <xacro:arm whichside="right" sidesign="+1.0" rollsign="+"/>
     <xacro:arm whichside="left"  sidesign="-1.0" rollsign="-"/>
+    <!--extra arm visuals-->
+    <xacro:include filename="$(find sergio_description)/urdf/xacro/arms/arm_extra.urdf.xacro" />
+    <xacro:arm_extra whichside="right" sidesign="+1.0" rollsign="+"/>
+    <xacro:arm_extra whichside="left"  sidesign="-1.0" rollsign="-"/>
     <!--========BUILD HEAD======-->
     <xacro:include filename="$(find sergio_description)/urdf/xacro/head/head.urdf.xacro" />

Commit message: Included meshes of torso and upperleg and use large base mesh

File: urdf/sergio.urdf (robot description, URDF)
Before this commit: robot sergio, 76 links, 75 joints
Links:
- added link trunk_inside, mass 0.001; collision box size=0.470 0.200 0.075; visual box size=0.470 0.200 0.075
- added link upper_leg_inside, mass 0.001; collision box size=0.5115 0.200 0.06; visual box size=0.5115 0.200 0.06
- link base: geometry collision mesh filename=package://sergio_description/media/meshes/Base2.dae scale=0.01 0.01 0.01; visual mesh filename=package://sergio_description/media/meshes/Base2.dae scale=0.01 0.01 0.01
- link shoulder_mount_left: geometry collision cylinder length=0.210 radius=0.075; visual cylinder length=0.210 radius=0.075
- link shoulder_mount_right: geometry collision cylinder length=0.210 radius=0.075; visual cylinder length=0.210 radius=0.075
- link trunk: geometry collision mesh filename=package://sergio_description/media/meshes/torso.dae scale=0.01 0.01 0.01; visual mesh filename=package://sergio_description/media/meshes/torso.dae scale=0.01 0.01 0.01
- link upper_leg: geometry collision mesh filename=package://sergio_description/media/meshes/upper_leg_reduced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 scale=0.01 0.01 0.01; visual mesh filename=package://sergio_description/media/meshes/upper_leg_reduced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 scale=0.01 0.01 0.01
- link wheel_left_front: geometry collision cylinder length=0.055 radius=0.075; visual cylinder length=0.055 radius=0.075
- link wheel_left_rear: geometry collision cylinder length=0.055 radius=0.075; visual cylinder length=0.055 radius=0.075
- link wheel_right_front: geometry collision cylinder length=0.055 radius=0.075; visual cylinder length=0.055 radius=0.075
- link wheel_right_rear: geometry collision cylinder length=0.055 radius=0.075; visual cylinder length=0.055 radius=0.075
Joints:
- added joint trunk_inside_joint: type fixed, parent trunk, child trunk_inside, origin xyz=0.0 0.0 0.0 rpy=0 0 0.0
- added joint upper_leg_inside_joint: type fixed, parent upper_leg, child upper_leg_inside, origin xyz=0.0 0.0 0.0 rpy=0 0 0.0

File: urdf/xacro/arms/arm.urdf.xacro (robot description, xacro)
@@ -17,5 +17,5 @@
 <!--the end of the clavicle, yaw rotation-->
 <xacro:my_link name="shoulder_mount_${whichside}" mass="0.15" color="White">
-   <cylinder radius="0.075" length="0.160" /><!-- Length of tube should be correct (see report), origin depends on placement -->
+   <cylinder radius="0.075" length="0.210" /><!-- Length of tube should be correct (see report), origin depends on placement -->
    <origin xyz="0.0 ${sidesign*-0.155} 0.0" rpy="1.57 0 0"/>
    <origin xyz="0.0 ${sidesign*-0.155} 0.0" rpy="1.57 0 0 " />

File: urdf/xacro/base/base.urdf.xacro (robot description, xacro)
@@ -12,12 +12,22 @@
     </xacro:my_link>
     <!--base block-->
-    <xacro:my_link name="base" mass="0.1" color="White"><!--ToDo: estimate mass-->
-        <box size="0.713 0.500 0.11"/><!--ToDo: check dimensions, adjust height-->
-        <!-- Large box for better self-filtering -->
-        <!--<box size="0.713 0.650 0.3" />-->
+    <!--
+    <xacro:my_link name="base" mass="0.1" color="White">
+        <box size="0.713 0.500 0.11"/>
         <origin xyz="-0.0235 0.0 0.0" rpy="0 0 0"/>
         <origin xyz="-0.0235 0.0 0.0" rpy="0 0 0"/>
-        <inertia ixx="0.001"  ixy="0"  ixz="0" iyy="0.001" iyz="0" izz="0.001" /><!--Estimate inertia-->
+        <inertia ixx="0.001"  ixy="0"  ixz="0" iyy="0.001" iyz="0" izz="0.001" />
     </xacro:my_link>
+    -->
+    <!--the base-->
+    <xacro:my_link_texturedmesh name="base" mass="0.1" texture="white">
+        <origin xyz="-0.295 0.10 -0.14" rpy="0 0 1.57"/>
+        <origin xyz="-0.295 0.10 -0.14" rpy="0 0 1.57" />
+        <inertia ixx="0.001"  ixy="0"  ixz="0" iyy="0.001" iyz="0" izz="0.001" />
+        <!--<mesh filename="package://sergio_description/media/meshes/Base2_reduced.dae" scale="0.01 0.01 0.01"/>-->
+        <!--<mesh filename="package://sergio_description/media/meshes/Base2_reduced10000.dae" scale="0.01 0.01 0.01"/>-->
+        <!--<mesh filename="package://sergio_description/media/meshes/BaseWithTexture.dae" scale="0.01 0.01 0.01"/>-->
+        <mesh filename="package://sergio_description/media/meshes/Base2.dae" scale="0.01 0.01 0.01"/>
+    </xacro:my_link_texturedmesh>
     <!-- side pots -->
     <xacro:my_link name="sidepot_left" mass="0.1" color="White"><!--ToDo: estimate mass-->
@@ -49,5 +59,5 @@
     <!-- wheels -->
     <xacro:my_link name="wheel_right_front" mass="0" color="DarkGrey">
-       <cylinder radius="0.075" length="0.06" />
+       <cylinder radius="0.075" length="0.055" />
        <origin xyz="0.0 0.0 0.0" rpy="0.0 0 0"/>
        <origin xyz="0.0 0.0 0.0" rpy="0.0 0 0" />
@@ -55,5 +65,5 @@
     </xacro:my_link>
     <xacro:my_link name="wheel_left_front" mass="0" color="DarkGrey">
-       <cylinder radius="0.075" length="0.06" />
+       <cylinder radius="0.075" length="0.055" />
        <origin xyz="0.0 0.0 0.0" rpy="0.0 0 0"/>
        <origin xyz="0.0 0.0 0.0" rpy="0.0 0 0" />
@@ -61,5 +71,5 @@
     </xacro:my_link>
     <xacro:my_link name="wheel_right_rear" mass="0" color="DarkGrey">
-       <cylinder radius="0.075" length="0.06" />
+       <cylinder radius="0.075" length="0.055" />
        <origin xyz="0.0 0.0 0.0" rpy="0.0 0 0"/>
        <origin xyz="0.0 0.0 0.0" rpy="0.0 0 0" />
@@ -67,5 +77,5 @@
     </xacro:my_link>
     <xacro:my_link name="wheel_left_rear" mass="0" color="DarkGrey">
-       <cylinder radius="0.075" length="0.06" />
+       <cylinder radius="0.075" length="0.055" />
        <origin xyz="0.0 0.0 0.0" rpy="0.0 0 0"/>
        <origin xyz="0.0 0.0 0.0" rpy="0.0 0 0" />

File: urdf/xacro/torso/torso.urdf.xacro (robot description, xacro)
@@ -5,5 +5,5 @@
     <review status="unreviewed" notes=""/>
    <!--mounting frame-->
-    <xacro:my_link name="torso_mounting_frame" mass="0.1" color="White"><!--ToDo: estimate mass-->
+    <xacro:my_link name="torso_mounting_frame" mass="0.1" color="Grey"><!--ToDo: estimate mass-->
         <box size="0.500 0.400 0.05" /><!--ToDo: check dimensions, adjust height-->
         <origin xyz="0.0 0.0 0.025" rpy="0 0 0"/>
@@ -12,5 +12,5 @@
     </xacro:my_link>
     <!-- Lower rear leg -->
-    <xacro:my_link name="lower_rear_leg" mass="5" color="White"><!--ToDo: estimate mass-->
+    <xacro:my_link name="lower_rear_leg" mass="5" color="Grey"><!--ToDo: estimate mass-->
         <box size="0.390 0.200 0.05" /><!--ToDo: check dimensions, adjust height-->
         <origin xyz="0.195 0.0 0.0" rpy="0 0 0"/><!--ToDo: check dimensions, adjust height-->
@@ -19,17 +19,44 @@
     </xacro:my_link>
     <!-- Upper leg (part from lower rear leg joint to trunk joint) -->
-    <xacro:my_link name="upper_leg" mass="5" color="White"><!--ToDo: estimate mass-->
-        <box size="0.4115 0.200 0.1" /><!--ToDo: check dimensions, adjust height-->
-        <origin xyz="0.20575 0.0 0.0" rpy="0 0 0"/><!--ToDo: check dimensions, adjust height-->
-        <origin xyz="0.20575 0.0 0.0" rpy="0 0 0"/><!--ToDo: check dimensions, adjust height-->
-        <inertia ixx="0.001"  ixy="0"  ixz="0" iyy="0.001" iyz="0" izz="0.001" /><!--Estimate inertia-->
+    <!--
+    <xacro:my_link name="upper_leg" mass="5" color="White">
+        <box size="0.4115 0.200 0.1" />
+        <origin xyz="0.20575 0.0 0.0" rpy="0 0 0"/>
+        <origin xyz="0.20575 0.0 0.0" rpy="0 0 0"/>
+        <inertia ixx="0.001"  ixy="0"  ixz="0" iyy="0.001" iyz="0" izz="0.001" />
+    </xacro:my_link>-->
+    <xacro:my_link_texturedmesh name="upper_leg" mass="5" texture="white"><!-- ToDo: estimate mass -->
+        <origin xyz="0.41575 -0.10 -0.02" rpy="0 0 1.57"/>
+        <origin xyz="0.41575 -0.10 -0.02" rpy="0 0 1.57"/>
+        <inertia ixx="0.001"  ixy="0"  ixz="0" iyy="0.001" iyz="0" izz="0.001" /><!-- ToDo: estimate mass -->
+        <mesh filename="package://sergio_description/media/meshes/upper_leg_reduced10000.dae" scale="0.01 0.01 0.01"/>
+    </xacro:my_link_texturedmesh>
+    <xacro:my_link name="upper_leg_inside" mass="0.001" color="Black">
+        <box size="0.5115 0.200 0.06" />
+        <origin xyz="0.20 0.0 0.0" rpy="0 0 0"/>
+        <origin xyz="0.20 0.0 0.0" rpy="0 0 0"/>
+        <inertia ixx="0.001"  ixy="0"  ixz="0" iyy="0.001" iyz="0" izz="0.001" />
     </xacro:my_link>
     <!-- Trunk -->
-    <xacro:my_link name="trunk" mass="10" color="White"><!--ToDo: estimate mass-->
-        <box size="0.470 0.200 0.15" /><!--ToDo: check dimensions, adjust height-->
-        <origin xyz="0.235 0.0 0.0" rpy="0 0 0"/><!--ToDo: check dimensions, adjust height-->
-        <origin xyz="0.235 0.0 0.0" rpy="0 0 0"/><!--ToDo: check dimensions, adjust height-->
-        <inertia ixx="0.001"  ixy="0"  ixz="0" iyy="0.001" iyz="0" izz="0.001" /><!--Estimate inertia-->
-    </xacro:my_link>
+    <!--
+    <xacro:my_link name="trunk" mass="10" color="White">
+        <box size="0.470 0.200 0.15" />
+        <origin xyz="0.235 0.0 0.0" rpy="0 0 0"/>
+        <origin xyz="0.235 0.0 0.0" rpy="0 0 0"/>
+        <inertia ixx="0.001"  ixy="0"  ixz="0" iyy="0.001" iyz="0" izz="0.001" />
+    </xacro:my_link>-->
+    <xacro:my_link_texturedmesh name="trunk" mass="10" texture="white"><!-- ToDo: estimate mass -->
+        <origin xyz="0.16 -0.12 0.0" rpy="3.1415 1.72 0"/>
+        <origin xyz="0.16 -0.12 0.0" rpy="3.1415 1.72 0"/>
+        <inertia ixx="0.001"  ixy="0"  ixz="0" iyy="0.001" iyz="0" izz="0.001" /><!-- ToDo: estimate mass -->
+        <!--<mesh filename="package://sergio_description/media/meshes/torso_reduced10000.dae" scale="0.01 0.01 0.01"/>-->
+        <mesh filename="package://sergio_description/media/meshes/torso.dae" scale="0.01 0.01 0.01"/>
+    </xacro:my_link_texturedmesh>
+    <xacro:my_link name="trunk_inside" mass="0.001" color="Black">
+        <box size="0.470 0.200 0.075" />
+        <origin xyz="0.235 0.0 0.0" rpy="0 0 0"/>
+        <origin xyz="0.235 0.0 0.0" rpy="0 0 0"/>
+        <inertia ixx="0.001"  ixy="0"  ixz="0" iyy="0.001" iyz="0" izz="0.001" />
+    </xacro:my_link>-->
     <!-- torso laser joint (center is the center of rotation of the laser)-->
 	<xacro:my_link name="torso_laser_mount" mass="0.01" color="Black">
@@ -59,4 +86,9 @@
         <!--<limit effort="1000" velocity="10" lower="2.0" upper="2.0" />--> <!--TEMP: fixed joint positions until control is fixed -->
     </xacro:my_joint>
+    <joint name="upper_leg_inside_joint" type="fixed">
+        <parent link="upper_leg"/>
+        <child link="upper_leg_inside"/>
+        <origin xyz="0.0 0.0 0.0" rpy="0 0 0.0"/>
+    </joint>
     <xacro:my_joint name="hip_joint" type="revolute" parent="upper_leg" child="trunk">
         <origin xyz="0.4115 0.0 0.0" rpy="3.14 3.14 0.0"/><!-- ToDo: adjust height-->
@@ -66,4 +98,9 @@
         <!--<limit effort="1000" velocity="10" lower="2.36" upper="2.36" />--> <!--TEMP: fixed joint positions until control is fixed-->
     </xacro:my_joint>
+    <joint name="trunk_inside_joint" type="fixed">
+        <parent link="trunk"/>
+        <child link="trunk_inside"/>
+        <origin xyz="0.0 0.0 0.0" rpy="0 0 0.0"/>
+    </joint>
     <joint name="laser_tilt_joint" type="revolute" >
 	   <parent link="trunk" />

Commit message: Visual updates

File: urdf/sergio.urdf (robot description, URDF)
Before this commit: robot sergio, 78 links, 77 joints
Links:
- link shoulder_mount_left: geometry collision cylinder length=0.190 radius=0.075; visual cylinder length=0.190 radius=0.075
- link shoulder_mount_right: geometry collision cylinder length=0.190 radius=0.075; visual cylinder length=0.190 radius=0.075
Joints:
- joint base_lasercenter_joint: origin xyz=0.03 0.0 0.0955 rpy=0.0 0.0 0.0 -> xyz=0.03 0.0 0.0455 rpy=0.0 0.0 0.0

File: urdf/xacro/arms/arm.urdf.xacro (robot description, xacro)
@@ -17,5 +17,5 @@
 <!--the end of the clavicle, yaw rotation-->
 <xacro:my_link name="shoulder_mount_${whichside}" mass="0.15" color="White">
-   <cylinder radius="0.075" length="0.210" /><!-- Length of tube should be correct (see report), origin depends on placement -->
+   <cylinder radius="0.075" length="0.190" /><!-- Length of tube should be correct (see report), origin depends on placement -->
    <origin xyz="0.0 ${sidesign*-0.155} 0.0" rpy="1.57 0 0"/>
    <origin xyz="0.0 ${sidesign*-0.155} 0.0" rpy="1.57 0 0 " />

File: urdf/xacro/torso/torso.urdf.xacro (robot description, xacro)
@@ -47,6 +47,6 @@
     </xacro:my_link>-->
     <xacro:my_link_texturedmesh name="trunk" mass="10" texture="white"><!-- ToDo: estimate mass -->
-        <origin xyz="0.16 -0.12 0.0" rpy="3.1415 1.72 0"/>
-        <origin xyz="0.16 -0.12 0.0" rpy="3.1415 1.72 0"/>
+        <origin xyz="0.16 -0.11 0.0" rpy="3.1415 1.73 0"/>
+        <origin xyz="0.16 -0.11 0.0" rpy="3.1415 1.73 0"/>
         <inertia ixx="0.001"  ixy="0"  ixz="0" iyy="0.001" iyz="0" izz="0.001" /><!-- ToDo: estimate mass -->
         <!--<mesh filename="package://sergio_description/media/meshes/torso_reduced10000.dae" scale="0.01 0.01 0.01"/>-->
