Commit message: adjusted the dynamixel limits because of hardware changes

File: urdf/sergio.urdf (robot description, URDF)
Before this commit: robot sergio, 58 links, 57 joints
Joints:
- joint laser_tilt_joint: limit lower=0.0 upper=0.3173 effort=13.4 velocity=1.0 -> lower=0.0 upper=0.324 effort=13.4 velocity=1.0
- joint neck_pan_joint: limit lower=-1.5708 upper=1.5708 effort=13.4 velocity=1.0 -> lower=-1.586 upper=1.586 effort=13.4 velocity=1.0
- joint neck_tilt_joint: limit lower=-0.98 upper=0.98 effort=13.4 velocity=1.0 -> lower=-0.994 upper=0.994 effort=13.4 velocity=1.0

File: urdf/xacro/head/head.urdf.xacro (robot description, xacro)
@@ -63,5 +63,5 @@
    <dynamics damping="0.1" friction="0"/>
    <axis xyz="0 0 1"/>
-   <limit effort="13.4" velocity="1.0" lower="-1.5708" upper="1.5708" />
+   <limit effort="13.4" velocity="1.0" lower="-1.586" upper="1.586" />
 </xacro:my_joint>
 <xacro:my_joint name="neck_tilt_joint" type="revolute" parent="neck_pan" child="neck_tilt">
@@ -69,5 +69,5 @@
    <dynamics damping="0.1" friction="0.0"/>
    <axis xyz="0 1 0"/>
-   <limit effort="13.4" velocity="1.0" lower="-0.98" upper="0.98" />
+   <limit effort="13.4" velocity="1.0" lower="-0.994" upper="0.994" />
 </xacro:my_joint>
 </robot>

File: urdf/xacro/torso/torso.urdf.xacro (robot description, xacro)
@@ -72,5 +72,5 @@
 	   <dynamics damping="0.1" friction="0"/><!--ToDo: update-->
 	   <axis xyz="0 1 0"/>
-	   <limit effort="13.4" velocity="1.0" lower="0.0" upper="0.3173" /> <!--ToDo: update-->
+	   <limit effort="13.4" velocity="1.0" lower="0.0" upper="0.324" /> <!--ToDo: update-->
 	</joint>
 </robot>

Commit message: Added batteries

File: urdf/sergio.urdf (robot description, URDF)
Before this commit: robot sergio, 78 links, 77 joints
Links:
- added link batteries, mass 0.1; collision box size=0.332 0.117 0.08; visual box size=0.332 0.117 0.08
Joints:
- added joint battery_joint: type fixed, parent base_link, child batteries, origin xyz=0.0 0.2335 0.194 rpy=0.0 0.0 0.0

File: urdf/xacro/base/base.urdf.xacro (robot description, xacro)
@@ -82,4 +82,11 @@
        <inertia ixx="0"  ixy="0"  ixz="0" iyy="0" iyz="0" izz="0" />
     </xacro:my_link>
+    <!-- Batteries -->
+    <xacro:my_link name="batteries" mass="0.1" color="Black"><!--ToDo: estimate mass-->
+        <box size="0.332 0.117 0.08" /><!--ToDo: check dimensions, adjust height-->
+        <origin xyz="0.0 0.0 0.0" rpy="0 0 0"/>
+        <origin xyz="0.0 0.0 0.0" rpy="0 0 0"/>
+        <inertia ixx="0.001"  ixy="0"  ixz="0" iyy="0.001" iyz="0" izz="0.001" /><!--Estimate inertia-->
+    </xacro:my_link>
     <!-- joints -->
     <joint name="base_link_joint" type="fixed">
@@ -131,3 +138,8 @@
         <origin xyz="-0.275 0.275 0.075" rpy="1.57 0.0 0.0"/>
     </joint>
+    <joint name="battery_joint" type="fixed">
+        <parent link="base_link"/>
+        <child link="batteries"/>
+        <origin xyz="0.0 0.2335 0.194" rpy="0.0 0.0 0.0"/>
+    </joint>
 </robot>

Commit message: Added 0.05 offset to torso

File: urdf/sergio.urdf (robot description, URDF)
Before this commit: robot sergio, 58 links, 57 joints
Joints:
- joint torso_mount_joint: origin xyz=0.0 0.0 0.0 rpy=0 0 0.0 -> xyz=0.0 0.0 0.05 rpy=0 0 0.0

File: urdf/xacro/torso/torso.urdf.xacro (robot description, xacro)
@@ -43,5 +43,5 @@
         <parent link="base_torso_mount"/>
         <child link="torso_mounting_frame"/>
-        <origin xyz="0.0 0.0 0.0" rpy="0 0 0.0"/><!--ToDo: adjust height-->
+        <origin xyz="0.0 0.0 0.05" rpy="0 0 0.0"/><!--ToDo: adjust height-->
     </joint>
     <xacro:my_joint name="ankle_joint" type="revolute" parent="torso_mounting_frame" child="lower_rear_leg">

Commit message: Better velocities and accelerations

File: urdf/sergio.urdf (robot description, URDF)
Before this commit: robot sergio, 79 links, 78 joints
Joints:
- joint ankle_joint: limit lower=0.152 upper=1.00 effort=1000 velocity=0.265 -> lower=0.152 upper=1.00 effort=0.3 velocity=0.265
- joint elbow_pitch_joint_left: limit lower=0.0 upper=2.23 effort=4.5 velocity=1.0 -> lower=0.0 upper=2.23 effort=0.5 velocity=0.8
- joint elbow_pitch_joint_right: limit lower=0.0 upper=2.23 effort=4.5 velocity=1.0 -> lower=0.0 upper=2.23 effort=0.5 velocity=0.8
- joint elbow_roll_joint_left: limit lower=-1.83 upper=1.83 effort=4.5 velocity=1.0 -> lower=-1.83 upper=1.83 effort=0.5 velocity=0.8
- joint elbow_roll_joint_right: limit lower=-1.83 upper=1.83 effort=4.5 velocity=1.0 -> lower=-1.83 upper=1.83 effort=0.5 velocity=0.8
- joint hip_joint: limit lower=1.007 upper=2.31 effort=1000 velocity=0.375 -> lower=1.007 upper=2.31 effort=0.3 velocity=0.375
- joint knee_joint: limit lower=0.419 upper=2.059 effort=1000 velocity=0.539 -> lower=0.419 upper=2.059 effort=0.3 velocity=0.539
- joint shoulder_pitch_joint_left: limit lower=-1.57 upper=1.57 effort=13.4 velocity=1.0 -> lower=-1.57 upper=1.57 effort=0.2 velocity=0.4
- joint shoulder_pitch_joint_right: limit lower=-1.57 upper=1.57 effort=13.4 velocity=1.0 -> lower=-1.57 upper=1.57 effort=0.2 velocity=0.4
- joint shoulder_roll_joint_left: limit lower=-1.57 upper=1.57 effort=9.8 velocity=1.0 -> lower=-1.57 upper=1.57 effort=0.3 velocity=0.6
- joint shoulder_roll_joint_right: limit lower=-1.57 upper=1.57 effort=9.8 velocity=1.0 -> lower=-1.57 upper=1.57 effort=0.3 velocity=0.6
- joint shoulder_yaw_joint_left: limit lower=-1.57 upper=0.0 effort=13.4 velocity=1.0 -> lower=-1.57 upper=0.0 effort=0.2 velocity=0.4
- joint shoulder_yaw_joint_right: limit lower=-1.57 upper=0.0 effort=13.4 velocity=1.0 -> lower=-1.57 upper=0.0 effort=0.2 velocity=0.4
- joint wrist_pitch_joint_left: limit lower=-0.95 upper=0.95 effort=1 velocity=1.0 -> lower=-0.95 upper=0.95 effort=0.5 velocity=1.0
- joint wrist_pitch_joint_right: limit lower=-0.95 upper=0.95 effort=1 velocity=1.0 -> lower=-0.95 upper=0.95 effort=0.5 velocity=1.0
- joint wrist_yaw_joint_left: limit lower=-0.61 upper=0.61 effort=1 velocity=1.0 -> lower=-0.61 upper=0.61 effort=0.5 velocity=1.0
- joint wrist_yaw_joint_right: limit lower=-0.61 upper=0.61 effort=1 velocity=1.0 -> lower=-0.61 upper=0.61 effort=0.5 velocity=1.0

File: urdf/xacro/arms/arm.urdf.xacro (robot description, xacro)
@@ -164,5 +164,5 @@
    <dynamics damping="4.0" friction="4.87"/>
    <axis xyz="${rollsign}1 0 0"/>
-   <limit effort="13.4" velocity="1.0" lower="-1.57" upper="0.0" />
+   <limit effort="0.2" velocity="0.4" lower="-1.57" upper="0.0" />
 </xacro:my_joint>
 <xacro:my_joint name="shoulder_pitch_joint_${whichside}" type="revolute" parent="shoulder_link1_${whichside}" child="shoulder_link2_${whichside}">
@@ -170,5 +170,5 @@
    <dynamics damping="4.0" friction="6.06"/>
    <axis xyz="0 -1 0"/>
-   <limit effort="13.4" velocity="1.0" lower="-1.57" upper="1.57" />
+   <limit effort="0.2" velocity="0.4" lower="-1.57" upper="1.57" />
 </xacro:my_joint>
 <xacro:my_joint name="shoulder_roll_joint_${whichside}" type="revolute" parent="shoulder_link2_${whichside}" child="upper_arm_${whichside}">
@@ -176,5 +176,5 @@
    <dynamics damping="3.8" friction="2.216"/>
    <axis xyz="0 ${sidesign} 0"/>
-   <limit effort="9.8" velocity="1.0" lower="-1.57" upper="1.57"/>
+   <limit effort="0.3" velocity="0.6" lower="-1.57" upper="1.57"/>
 </xacro:my_joint>
 <xacro:my_joint name="elbow_pitch_joint_${whichside}" type="revolute" parent="upper_arm_${whichside}" child="elbow_link4_${whichside}">
@@ -182,5 +182,5 @@
    <dynamics damping="3" friction="1.18"/>
    <axis xyz="0 -1 0"/>
-   <limit effort="4.5" velocity="1.0" lower="0.0" upper="2.23" />
+   <limit effort="0.5" velocity="0.8" lower="0.0" upper="2.23" />
 </xacro:my_joint>
 <xacro:my_joint name="elbow_roll_joint_${whichside}" type="revolute" parent="elbow_link4_${whichside}" child="fore_arm_${whichside}">
@@ -188,5 +188,5 @@
    <dynamics damping="3.5" friction="1.35"/>
    <axis xyz="0 ${sidesign} 0"/>
-   <limit effort="4.5" velocity="1.0" lower="-1.83" upper="1.83"/>
+   <limit effort="0.5" velocity="0.8" lower="-1.83" upper="1.83"/>
 </xacro:my_joint>
 <xacro:my_joint name="wrist_pitch_joint_${whichside}" type="revolute" parent="fore_arm_${whichside}" child="wrist_link6_${whichside}">
@@ -194,5 +194,5 @@
    <dynamics damping="0.35" friction="0.63"/>
    <axis xyz="0 -1 0"/>
-   <limit effort="1" velocity="1.0" lower="-0.95" upper="0.95"/>
+   <limit effort="0.5" velocity="1.0" lower="-0.95" upper="0.95"/>
 </xacro:my_joint>
 <xacro:my_joint name="wrist_yaw_joint_${whichside}" type="revolute" parent="wrist_link6_${whichside}" child="hand_${whichside}">
@@ -200,5 +200,5 @@
    <dynamics damping="0.3" friction="0.68"/>
    <axis xyz="0 0 ${sidesign}1"/>
-   <limit effort="1" velocity="1.0" lower="-0.61" upper="0.61"/>
+   <limit effort="0.5" velocity="1.0" lower="-0.61" upper="0.61"/>
 </xacro:my_joint>
 <xacro:my_joint name="finger1_joint_${whichside}" type="revolute" parent="hand_${whichside}" child="finger1_${whichside}">

File: urdf/xacro/torso/torso.urdf.xacro (robot description, xacro)
@@ -76,5 +76,5 @@
         <dynamics damping="6.0" friction="4.87"/><!-- ToDo: adjust dynamics-->
         <axis xyz="0 -1 0"/><!--ToDo: DH parameters?-->
-        <limit effort="1000" velocity="0.265" lower="0.152" upper="1.00" /> <!--ToDo: adjust parameters-->
+        <limit effort="0.3" velocity="0.265" lower="0.152" upper="1.00" /> <!--ToDo: adjust parameters-->
         <!--<limit effort="1000" velocity="10" lower="0.87" upper="0.87" />--> <!--TEMP: fixed joint positions until control is fixed-->
     </xacro:my_joint>
@@ -83,5 +83,5 @@
         <dynamics damping="6.0" friction="4.87"/><!-- ToDo: adjust dynamics-->
         <axis xyz="0 -1 0"/><!--ToDo: DH parameters?-->
-        <limit effort="1000" velocity="0.539" lower="0.419" upper="2.059" /> <!--ToDo: adjust parameters -->
+        <limit effort="0.3" velocity="0.539" lower="0.419" upper="2.059" /> <!--ToDo: adjust parameters -->
         <!--<limit effort="1000" velocity="10" lower="2.0" upper="2.0" />--> <!--TEMP: fixed joint positions until control is fixed -->
     </xacro:my_joint>
@@ -95,5 +95,5 @@
         <dynamics damping="6.0" friction="4.87"/><!-- ToDo: adjust dynamics-->
         <axis xyz="0 -1 0"/><!--ToDo: DH parameters?-->
-        <limit effort="1000" velocity="0.375" lower="1.007" upper="2.31" /> <!--ToDo: adjust parameters --><!--Velocity: move in 4 s-->
+        <limit effort="0.3" velocity="0.375" lower="1.007" upper="2.31" /> <!--ToDo: adjust parameters --><!--Velocity: move in 4 s-->
         <!--<limit effort="1000" velocity="10" lower="2.36" upper="2.36" />--> <!--TEMP: fixed joint positions until control is fixed-->
     </xacro:my_joint>
