Commit message: Now truly independent of amigo_description

File: urdf/xacro/macro_definitions.xacro (robot description, xacro)
@@ -46,5 +46,5 @@
      <xacro:insert_block name="type" />
      </geometry>
-     <material name="amigo_description/${texture}">
+     <material name="sergio_description/${texture}">
      </material>
     </visual>
@@ -57,5 +57,5 @@
   </link>
 <gazebo reference="${name}">
-      <material>amigo_description/${texture}</material>
+      <material>sergio_description/${texture}</material>
       <turnGravityOff>false</turnGravityOff>
     </gazebo>
@@ -124,5 +124,5 @@
      <xacro:insert_block name="mesh" />
      </geometry>
-     <material name="amigo_description/${texture}"/>
+     <material name="sergio_description/${texture}"/>
     </visual>
     <collision>
@@ -134,5 +134,5 @@
   </link>
 <gazebo reference="${name}">
-	  <material>amigo_description/${texture}</material>
+	  <material>sergio_description/${texture}</material>
       <turnGravityOff>false</turnGravityOff>
     </gazebo>
@@ -151,5 +151,5 @@
      <xacro:insert_block name="mesh" />
      </geometry>
-     <material name="amigo_description/${texture}"/>
+     <material name="sergio_description/${texture}"/>
     </visual>
     <collision>
@@ -161,5 +161,5 @@
   </link>
 <gazebo reference="${name}">
-	  <material>amigo_description/${texture}</material>
+	  <material>sergio_description/${texture}</material>
       <turnGravityOff>false</turnGravityOff>
     </gazebo>

File: urdf/xacro/materials.urdf.xacro (robot description, xacro)
@@ -32,18 +32,18 @@
     <color rgba="1.0 0.33 0.0 1.0"/>
   </material>
-  <material name="amigo_description/bottomcovers">
-    <texture filename="package://amigo_description/media/materials/textures/bottomcovers/finalreduced.jpg" />
+  <material name="sergio_description/bottomcovers">
+    <texture filename="package://sergio_description/media/materials/textures/bottomcovers/finalreduced.jpg" />
   </material>
-    <material name="amigo_description/white">
-    <texture filename="package://amigo_description/media/materials/textures/white/white.jpg" />
+    <material name="sergio_description/white">
+    <texture filename="package://sergio_description/media/materials/textures/white/white.jpg" />
   </material>
-  <material name="amigo_description/logo">
-    <texture filename="package://amigo_description/media/materials/textures/logo/tue.jpg" />
+  <material name="sergio_description/logo">
+    <texture filename="package://sergio_description/media/materials/textures/logo/tue.jpg" />
   </material>
-  <material name="amigo_description/aluminium">
-    <texture filename="package://amigo_description/media/materials/textures/aluminium/aluminium_0001_c.jpg" />
+  <material name="sergio_description/aluminium">
+    <texture filename="package://sergio_description/media/materials/textures/aluminium/aluminium_0001_c.jpg" />
   </material>
-  <material name="amigo_description/orange">
-    <texture filename="package://amigo_description/media/materials/textures/orange/orange.jpg" />
+  <material name="sergio_description/orange">
+    <texture filename="package://sergio_description/media/materials/textures/orange/orange.jpg" />
   </material>
 </robot>
