Commit message: Add prefix like AMIGO

File: urdf/kinect/top_kinect.urdf.xacro (robot description, xacro)
@@ -1,5 +1,5 @@
 <?xml version="1.0"?>
 <robot xmlns:xacro="http://ros.org/wiki/xacro">
-  <property name="M_PI" value="3.14159"/>
+  <xacro:property name="M_PI" value="3.14159"/>
   <joint name="top_kinect/base_kinect_joint" type="fixed">
     <origin xyz="0.03 0.0 0.017" rpy="0 0 0" /> <!-- THESE VALUES ARE ROUGH ESTIMATES!! -->

File: urdf/sergio.urdf.xacro (robot description, xacro)
@@ -4,4 +4,5 @@
     <license>BSD</license>
     <review status="unreviewed" notes=""/>
+    <xacro:property name="prefix" value="sergio/" scope="parent | global"/>
     <!-- ToDo: In general: look at DH conventions-->
     <!--get link & joint definitions -->
