Commit message: Front laser is now upside down and added back laser

File: urdf/base/base.urdf.xacro (robot description, xacro)
@@ -47,4 +47,11 @@
         <inertia ixx="0.0001"  ixy="0"  ixz="0" iyy="0.0001" iyz="0" izz="0.0001" />
     </xacro:my_link>
+    <!-- base - back laser interface -->
+    <xacro:my_link name="back_laser_mount" mass="0.01" color="White">
+       <box size="0.01 0.06 0.035" />
+       <origin xyz="0.005 0.0 0.0175" rpy="0 0 0"/>
+       <origin xyz="0.005 0.0 0.0175" rpy="0 0 0"/>
+       <inertia ixx="0.0001"  ixy="0"  ixz="0" iyy="0.0001" iyz="0" izz="0.0001" />
+    </xacro:my_link>
     <!-- joints -->
     <joint name="base_link_joint" type="fixed">
@@ -74,5 +81,10 @@
         <parent link="base"/>
         <child link="laser_mount"/>
-        <origin xyz="0.2995 0.0 0.055" rpy="0.0 0.0 0.0"/>
+        <origin xyz="0.2995 0.0 0.055" rpy="3.141592653589793 0.0 0.0"/>
+    </joint>
+    <joint name="back_laser_mount_joint" type="fixed">
+        <parent link="base"/>
+        <child link="back_laser_mount"/>
+        <origin xyz="-0.285 0.0 0.27" rpy="0.0 0.0 0.0"/>
     </joint>
 </robot>

File: urdf/sergio.urdf.xacro (robot description, xacro)
@@ -27,5 +27,6 @@
     <!--<xacro:include filename="$(find sergio_description)/urdf/laser/base_laser.urdf.xacro" />-->
     <xacro:include filename="$(find sergio_description)/urdf/laser/laser.urdf.xacro" />
-    <xacro:laser laser_name="base" laser_parent="laser_mount" laser_xyz="0.03 0.0 0.0955" laser_rpy="0.0 0.0 0.0"  />
+    <xacro:laser laser_name="base" laser_parent="laser_mount" laser_xyz="0.03 0.0 0.078" laser_rpy="0.0 0.0 0.0"  />
+    <xacro:laser laser_name="back" laser_parent="back_laser_mount" laser_xyz="0.0 0.0 0.0" laser_rpy="0.0 0.0 3.141592653589793"  />
     <xacro:laser laser_name="torso" laser_parent="torso_laser_mount" laser_xyz="0.0 0.0 -0.004" laser_rpy="0.0 0.0 0.0"  />
 </robot>

Commit message: Change back laser position

File: urdf/base/base.urdf.xacro (robot description, xacro)
@@ -81,10 +81,10 @@
         <parent link="base"/>
         <child link="laser_mount"/>
-        <origin xyz="0.2995 0.0 0.055" rpy="3.141592653589793 0.0 0.0"/>
+        <origin xyz="0.2995 0.0 0.05" rpy="3.141592653589793 0.0 0.0"/>
     </joint>
     <joint name="back_laser_mount_joint" type="fixed">
         <parent link="base"/>
         <child link="back_laser_mount"/>
-        <origin xyz="-0.285 0.0 0.27" rpy="0.0 0.0 0.0"/>
+        <origin xyz="-0.20 0.0 0.291" rpy="0.0 0.0 0.0"/>
     </joint>
 </robot>

Commit message: Change back laser mount box size

File: urdf/base/base.urdf.xacro (robot description, xacro)
@@ -49,5 +49,5 @@
     <!-- base - back laser interface -->
     <xacro:my_link name="back_laser_mount" mass="0.01" color="White">
-       <box size="0.01 0.06 0.035" />
+       <box size="0.01 0.06 0.03" />
        <origin xyz="0.005 0.0 0.0175" rpy="0 0 0"/>
        <origin xyz="0.005 0.0 0.0175" rpy="0 0 0"/>

Commit message: Change back laser position

File: urdf/base/base.urdf.xacro (robot description, xacro)
@@ -86,5 +86,5 @@
         <parent link="base"/>
         <child link="back_laser_mount"/>
-        <origin xyz="-0.20 0.0 0.291" rpy="0.0 0.0 0.0"/>
+        <origin xyz="-0.20 0.0 0.206" rpy="0.0 0.0 0.0"/>
     </joint>
 </robot>

Commit message: Update pos of lasers and new look

File: urdf/base/base.urdf.xacro (robot description, xacro)
@@ -15,20 +15,26 @@
         <!--box size="0.713 0.500 0.11" /--><!--ToDo: check dimensions, adjust height-->
         <!-- Large box for better self-filtering -->
-        <box size="0.713 0.650 0.3" />
-        <origin xyz="-0.0235 0.0 0.0" rpy="0 0 0"/>
-        <origin xyz="-0.0235 0.0 0.0" rpy="0 0 0"/>
+        <box size="0.73 0.650 0.14" />
+        <origin xyz="-0.02 0.0 -0.015" rpy="0 0 0"/>
+        <origin xyz="-0.02 0.0 -0.015" rpy="0 0 0"/>
         <inertia ixx="0.001"  ixy="0"  ixz="0" iyy="0.001" iyz="0" izz="0.001" /><!--Estimate inertia-->
     </xacro:my_link>
     <!-- side pots -->
     <xacro:my_link name="sidepot_left" mass="0.1" color="White"><!--ToDo: estimate mass-->
-        <box size="0.400 0.0615 0.1" /><!--ToDo: check dimensions, adjust height-->
-        <origin xyz="0.0 0.0 0.0" rpy="0 0 0"/>
-        <origin xyz="0.0 0.0 0.0" rpy="0 0 0"/>
+        <box size="0.43 0.165 0.13" /><!--ToDo: check dimensions, adjust height-->
+        <origin xyz="0.0 0.0 0.065" rpy="0 0 0"/>
+        <origin xyz="0.0 0.0 0.065" rpy="0 0 0"/>
         <inertia ixx="0.001"  ixy="0"  ixz="0" iyy="0.001" iyz="0" izz="0.001" /><!--Estimate inertia-->
     </xacro:my_link>
     <xacro:my_link name="sidepot_right" mass="0.1" color="White"><!--ToDo: estimate mass-->
-        <box size="0.400 0.0615 0.1" /><!--ToDo: check dimensions, adjust height-->
-        <origin xyz="0.0 0.0 0.0" rpy="0 0 0"/>
-        <origin xyz="0.0 0.0 0.0" rpy="0 0 0"/>
+        <box size="0.43 0.165 0.13" /><!--ToDo: check dimensions, adjust height-->
+        <origin xyz="0.0 0.0 0.065" rpy="0 0 0"/>
+        <origin xyz="0.0 0.0 0.065" rpy="0 0 0"/>
+        <inertia ixx="0.001"  ixy="0"  ixz="0" iyy="0.001" iyz="0" izz="0.001" /><!--Estimate inertia-->
+    </xacro:my_link>
+    <xacro:my_link name="sidepot_back" mass="0.1" color="White"><!--ToDo: estimate mass-->
+        <box size="0.16 0.65 0.13" /><!--ToDo: check dimensions, adjust height-->
+        <origin xyz="0.0 0.0 0.065" rpy="0 0 0"/>
+        <origin xyz="0.0 0.0 0.065" rpy="0 0 0"/>
         <inertia ixx="0.001"  ixy="0"  ixz="0" iyy="0.001" iyz="0" izz="0.001" /><!--Estimate inertia-->
     </xacro:my_link>
@@ -49,7 +55,7 @@
     <!-- base - back laser interface -->
     <xacro:my_link name="back_laser_mount" mass="0.01" color="White">
-       <box size="0.01 0.06 0.03" />
-       <origin xyz="0.005 0.0 0.0175" rpy="0 0 0"/>
-       <origin xyz="0.005 0.0 0.0175" rpy="0 0 0"/>
+       <box size="0.06 0.28 0.01" />
+       <origin xyz="0.0 0.0 -0.005" rpy="0 0 0"/>
+       <origin xyz="0.0 0.0 -0.005" rpy="0 0 0"/>
        <inertia ixx="0.0001"  ixy="0"  ixz="0" iyy="0.0001" iyz="0" izz="0.0001" />
     </xacro:my_link>
@@ -65,5 +71,5 @@
         <child link="sidepot_left"/>
         <axis xyz="1 0 0"/>
-        <origin xyz="0.0 0.28075 0.0" rpy="0 0 0"/><!--ToDO: adjust distance-->
+        <origin xyz="-0.01 0.2425 0.045" rpy="0 0 0"/><!--ToDO: adjust distance-->
     </joint>
     <joint name="sidepot_right_joint" type="fixed">
@@ -71,20 +77,26 @@
         <child link="sidepot_right"/>
         <axis xyz="1 0 0"/>
-        <origin xyz="0.0 -0.28075 0.0" rpy="0 0 0"/><!--ToDO: adjust distance-->
+        <origin xyz="-0.01 -0.2425 0.045" rpy="0 0 0"/><!--ToDO: adjust distance-->
+    </joint>
+    <joint name="sidepot_back_joint" type="fixed">
+        <parent link="base"/>
+        <child link="sidepot_back"/>
+        <axis xyz="1 0 0"/>
+        <origin xyz="-0.305 0.0 0.045" rpy="0 0 0"/><!--ToDO: adjust distance-->
     </joint>
     <joint name="base_mount_joint" type="fixed">
         <parent link="base"/>
         <child link="base_torso_mount"/>
-        <origin xyz="0.0 0.0 0.055" rpy="0 0 0.0"/><!--ToDo: adjust height-->
+        <origin xyz="0.0 0.0 0.01" rpy="0 0 0.0"/><!--ToDo: adjust height 12-11-16 Matthijs: -4.5cm -->
     </joint>
     <joint name="laser_mount_joint" type="fixed">
         <parent link="base"/>
         <child link="laser_mount"/>
-        <origin xyz="0.2995 0.0 0.05" rpy="3.141592653589793 0.0 0.0"/>
+        <origin xyz="0.2995 0.0 0.039" rpy="3.141592653589793 0.0 0.0"/>
     </joint>
     <joint name="back_laser_mount_joint" type="fixed">
         <parent link="base"/>
         <child link="back_laser_mount"/>
-        <origin xyz="-0.20 0.0 0.206" rpy="0.0 0.0 0.0"/>
+        <origin xyz="-0.293 0.0 0.157" rpy="0.0 0.0 0.0"/>
     </joint>
 </robot>

File: urdf/sergio.urdf.xacro (robot description, xacro)
@@ -28,5 +28,5 @@
     <xacro:include filename="$(find sergio_description)/urdf/laser/laser.urdf.xacro" />
     <xacro:laser laser_name="base" laser_parent="laser_mount" laser_xyz="0.03 0.0 0.06" laser_rpy="0.0 0.0 0.0"  />
-    <xacro:laser laser_name="back" laser_parent="back_laser_mount" laser_xyz="-0.03 0.0 0.06" laser_rpy="0.0 0.0 3.141592653589793"  />
+    <xacro:laser laser_name="back" laser_parent="back_laser_mount" laser_xyz="0.0 0.0 0.06" laser_rpy="0.0 0.0 3.141592653589793"  />
     <xacro:laser laser_name="torso" laser_parent="torso_laser_mount" laser_xyz="0.0 0.0 -0.004" laser_rpy="0.0 0.0 0.0"  />
 </robot>

File: urdf/torso/torso.urdf.xacro (robot description, xacro)
@@ -33,10 +33,10 @@
     </xacro:my_link>
     <!-- torso laser joint (center is the center of rotation of the laser)-->
-	<xacro:my_link name="torso_laser_mount" mass="0.01" color="Black">
-	   <box size="0.0 0.0 0.0" />
-	   <origin xyz="0.0 0.0 0.0" rpy="0 0 0"/>
-	   <origin xyz="0.0 0.0 0.0" rpy="0 0 0" />
-	   <inertia ixx="0.0001"  ixy="0"  ixz="0" iyy="0.0001" iyz="0" izz="0.0001" />
-	</xacro:my_link>
+    <xacro:my_link name="torso_laser_mount" mass="0.01" color="Black">
+        <box size="0.0 0.0 0.0" />
+        <origin xyz="0.0 0.0 0.0" rpy="0 0 0"/>
+        <origin xyz="0.0 0.0 0.0" rpy="0 0 0" />
+        <inertia ixx="0.0001"  ixy="0"  ixz="0" iyy="0.0001" iyz="0" izz="0.0001" />
+    </xacro:my_link>
     <!-- joints -->
     <joint name="torso_mount_joint" type="fixed">
@@ -67,10 +67,10 @@
     </xacro:my_joint>
     <joint name="laser_tilt_joint" type="revolute" >
-	   <parent link="trunk" />
-	   <child link="torso_laser_mount"/>
-	   <origin xyz="0.3073 0.0 -0.0871" rpy="3.14 1.406 0.0 "/>
-	   <dynamics damping="0.1" friction="0"/><!--ToDo: update-->
-	   <axis xyz="0 1 0"/>
-	   <limit effort="13.4" velocity="1.0" lower="0.0" upper="0.324" /> <!--ToDo: update-->
-	</joint>
+        <parent link="trunk" />
+        <child link="torso_laser_mount"/>
+        <origin xyz="0.3073 0.0 -0.0871" rpy="3.14 1.406 0.0 "/>
+        <dynamics damping="0.1" friction="0"/><!--ToDo: update-->
+        <axis xyz="0 1 0"/>
+        <limit effort="13.4" velocity="1.0" lower="0.0" upper="0.324" /> <!--ToDo: update-->
+        </joint>
 </robot>

Commit message: update batteries

File: urdf/base/base.urdf.xacro (robot description, xacro)
@@ -90,7 +90,7 @@
     <!-- Batteries -->
     <xacro:my_link name="batteries" mass="0.1" color="Black"><!--ToDo: estimate mass-->
-        <box size="0.332 0.117 0.08" /><!--ToDo: check dimensions, adjust height-->
-        <origin xyz="0.0 0.0 0.0" rpy="0 0 0"/>
-        <origin xyz="0.0 0.0 0.0" rpy="0 0 0"/>
+        <box size="0.332 0.120 0.1" /><!--ToDo: check dimensions, adjust height-->
+        <origin xyz="0.0 0.0 0.05" rpy="0 0 0"/>
+        <origin xyz="0.0 0.0 0.05" rpy="0 0 0"/>
         <inertia ixx="0.001"  ixy="0"  ixz="0" iyy="0.001" iyz="0" izz="0.001" /><!--Estimate inertia-->
     </xacro:my_link>
@@ -156,7 +156,7 @@
     </joint>
     <joint name="battery_joint" type="fixed">
-        <parent link="base_link"/>
+        <parent link="base"/>
         <child link="batteries"/>
-        <origin xyz="0.0 0.2335 0.194" rpy="0.0 0.0 0.0"/>
+        <origin xyz="0.0 0.23 0.055" rpy="0.0 0.0 0.0"/>
     </joint>
 </robot>
