Commit message: New Torso laser possition 20mm front 9mm down

File: urdf/torso/torso.urdf.xacro (robot description, xacro)
@@ -69,5 +69,5 @@
 	   <parent link="trunk" />
 	   <child link="torso_laser_mount"/>
-	   <origin xyz="0.3163 0.0 -0.0671" rpy="3.14 1.406 0.0 "/>
+	   <origin xyz="0.3073 0.0 -0.0871" rpy="3.14 1.406 0.0 "/>
 	   <dynamics damping="0.1" friction="0"/><!--ToDo: update-->
 	   <axis xyz="0 1 0"/>

Commit message: Add dummy matrix frame

File: urdf/torso/torso.urdf.xacro (robot description, xacro)
@@ -39,4 +39,9 @@
         <inertia ixx="0.0001"  ixy="0"  ixz="0" iyy="0.0001" iyz="0" izz="0.0001" />
     </xacro:my_link>
+    <!-- Matrix creator -->
+    <link name="matrix">
+       <origin xyz="0.0 0.0 0.0" rpy="0 0 0" />
+       <inertia ixx="0"  ixy="0"  ixz="0" iyy="0" iyz="0" izz="0" />
+    </link>
     <!-- joints -->
     <joint name="torso_mount_joint" type="fixed">
@@ -74,3 +79,8 @@
         <limit effort="13.4" velocity="1.0" lower="0.0" upper="0.324" /> <!--ToDo: update-->
         </joint>
+    <joint name="trunk_matrix_joint" type="fixed">
+        <parent link="trunk"/>
+        <child link="matrix"/>
+        <origin xyz="0.5 0.0 0.10" rpy="0 1.570796 0"/>
+    </joint>
 </robot>
