Commit message: Add extra arm visuals

File: urdf/arms/arm.urdf.xacro (robot description, xacro)
@@ -1,235 +1,254 @@
 <?xml version="1.0"?>
-<robot 	xmlns:xacro="http://ros.org/wiki/xacro">
-    <author>Rob Janssen, Kris van Tienhoven, Janno Lunenburg</author>
-    <license>BSD</license>
-    <review status="unreviewed" notes=""/>
-    <!--Start of the macro
-    @param whichside is "left"  or "right"
-    @param sidesign is -1 or +1
-    @param rollsign is - or +
-    The reason sidesign is -1 or +1 and not just - or + aswell is because
-    it has to be reversable and xml cannot multiply - or + but can multiply
-     -1 and +1-->
-     <xacro:macro name="arm" params="whichside sidesign rollsign">
-    <!--the end of the clavicle, yaw rotation-->
-    <xacro:my_link name="shoulder_mount_${whichside}" mass="0.15" color="White">
-       <cylinder radius="0.075" length="0.140" /><!-- Length of tube should be correct (see report), origin depends on placement -->
-       <origin xyz="0.0 ${sidesign*-0.155} 0.0" rpy="1.57 0 0"/>
-       <origin xyz="0.0 ${sidesign*-0.155} 0.0" rpy="1.57 0 0 " />
-       <inertia ixx="0.01"  ixy="0"  ixz="0" iyy="0.01" iyz="0" izz="0.01" /> <!-- 0.45993-->
-    </xacro:my_link>
-    <!-- ${sidesign*-0.155} -->
-    <!--the cylinder on the end of the clavicle, pitch rotation-->
-    <xacro:my_link name="shoulder_link1_${whichside}" mass="0.25" color="Black">
-       <cylinder radius="0.045" length="0.015" />
-       <origin xyz="0.0 0.0 0.0" rpy="0 0 0"/>
-       <origin xyz="0.0 0.0 ${sidesign *0.0525}" rpy="0 0 0 " />
-       <inertia ixx="6.0"  ixy="0"  ixz="0" iyy="0.01" iyz="0" izz="0.01" />
-    </xacro:my_link>
-    <!--the box that connects the clavicle to the upper arm, roll rotation-->
-    <xacro:my_link name="shoulder_link2_${whichside}" mass="0.15" color="Black">
-       <box size="0.035 0.01 0.1" />
-       <origin xyz="0.0 0.0 0.0" rpy="0 0 0"/>
-       <origin xyz="0.0 ${-sidesign*0.06} -0.05" rpy="0 0 0" />
-       <inertia ixx="0.01"  ixy="0"  ixz="0" iyy="4.04" iyz="0" izz="0.001" />
-    </xacro:my_link>
-    <!--the upper arm-->
-    <xacro:my_link_texturedmesh name="upper_arm_${whichside}" mass="2.95" texture="white">
-       <origin xyz="0.0 -0.2 0.0" rpy="0 0 0"/>
-       <origin xyz="-0.00959 -0.19131 -0.00001" rpy="0 0 3.1415" />
-       <inertia ixx="0.027"  ixy="0"  ixz="0" iyy="0.45993" iyz="0" izz="0.004" />
-       <mesh filename="package://sergio_description/media/meshes/upperarmtextured.dae" scale="0.0004 0.0004 0.0004"/>
-    </xacro:my_link_texturedmesh>
-    <!--the elbow
-    note: not visible, see arm_extra_visuals for the elbow visuals -->
-    <xacro:my_link name="elbow_link4_${whichside}" mass="0.1" color="Grey">
-       <cylinder radius="0.0" length="0.0"/>
-       <origin xyz="0.0 0.0 0.0" rpy="0 0 0"/>
-       <origin xyz="0.0 0.0 0.0" rpy="0 0 0" />
-       <inertia ixx="0.001"  ixy="0"  ixz="0" iyy="0.6" iyz="0" izz="0.001" />
-    </xacro:my_link>
-    <!--the forearm-->
-    <xacro:my_link_texturedmesh name="fore_arm_${whichside}" mass="0.85" texture="white">
-       <origin xyz="0.0 -0.14 0.0" rpy="0.0 0 0"/>
-       <origin xyz="0.00425 -0.14868 0.00547" rpy="0 -1.5708 0" />
-       <inertia ixx="0.001"  ixy="0"  ixz="0" iyy="0.5" iyz="0" izz="0.001" />
-       <mesh filename="package://sergio_description/media/meshes/forearmtextured.dae" scale="0.0004 0.0004 0.0004"/>
-    </xacro:my_link_texturedmesh>
-    <!--the wrist
-    note: not visible, see arm_extra_visuals for the wrist visuals -->
-    <xacro:my_link name="wrist_link6_${whichside}" mass="0.01" color="Black">
-       <cylinder radius="0.0" length="0.0"/>
-       <origin xyz="0.0 0.0 0.0" rpy="0 0 0"/>
-       <origin xyz="0.0 0.0 0.0" rpy="1.5708 0 0" />
-       <inertia ixx="0.001"  ixy="0"  ixz="0" iyy="0.03322" iyz="0" izz="0.001" />
-    </xacro:my_link>
-    <!--the hand -->
-    <xacro:my_link name="hand_${whichside}" mass="0.20" color="Grey">
-       <box size="0.080 0.085 0.038"/>
-       <origin xyz="0.048 0.0 0.0" rpy="0 0 0"/>
-       <origin xyz="0.048 0.0 0.0" rpy="0 0 0" />
-       <inertia ixx="0.01"  ixy="0"  ixz="0" iyy="0.01" iyz="0" izz="0.0622" />
-    </xacro:my_link>
-    <!--the right finger-->
-    <xacro:my_link name="finger1_${whichside}" mass="0.01" color="Black">
-       <box size="0.018 0.018 0.06"/>
-       <origin xyz="0.0 0.0 -0.03" rpy="0 0 0"/>
-       <origin xyz="0.0 0.0 -0.03" rpy="0 0 0" />
-       <inertia ixx="0.01"  ixy="0"  ixz="0" iyy="0.01" iyz="0" izz="0.01" />
-    </xacro:my_link>
-    <!--the right finger phalanx-->
-    <xacro:my_link name="finger1_phalanx_${whichside}" mass="0.01" color="White">
-       <cylinder length="0.019" radius="0.009"/>
-       <origin xyz="0.0 0.0 0" rpy="0 0 0"/>
-       <origin xyz="0.0 0.0 0" rpy="0 0 0" />
-       <inertia ixx="0.001"  ixy="0"  ixz="0" iyy="0.001" iyz="0" izz="0.001" />
-    </xacro:my_link>
-    <!--the right finger tip-->
-    <xacro:my_link name="finger1_tip_${whichside}" mass="0.01" color="Black">
-       <box size="0.018 0.018 0.06"/>
-       <origin xyz="0.0 0.0 -0.03" rpy="0 0 0"/>
-       <origin xyz="0.0 0.0 -0.03" rpy="0 0 0" />
-       <inertia ixx="0.00037"  ixy="0"  ixz="0" iyy="0.00052" iyz="0" izz="0.00052" />
-    </xacro:my_link>
-    <!--the right finger tip phalanx-->
-    <xacro:my_link name="finger1_tip_phalanx_${whichside}" mass="0.01" color="White">
-       <cylinder length="0.017" radius="0.009"/>
-       <origin xyz="0.0 0.0 0" rpy="0 0 0"/>
-       <origin xyz="0.0 0.0 0" rpy="0 0 0" />
-       <inertia ixx="0.001"  ixy="0"  ixz="0" iyy="0.001" iyz="0" izz="0.001" />
-    </xacro:my_link>
-    <!--the left finger-->
-    <xacro:my_link name="finger2_${whichside}" mass="0.01" color="Black">
-       <box size="0.018 0.018 0.06"/>
-       <origin xyz="0.0 0.0 -0.03" rpy="0 0 0"/>
-       <origin xyz="0.0 0.0 -0.03" rpy="0 0 0" />
-       <inertia ixx="0.01"  ixy="0"  ixz="0" iyy="0.01" iyz="0" izz="0.01" />
-    </xacro:my_link>
-    <!--the left finger phalanx-->
-    <xacro:my_link name="finger2_phalanx_${whichside}" mass="0.01" color="White">
-       <cylinder length="0.019" radius="0.009"/>
-       <origin xyz="0.0 0.0 0" rpy="0 0 0"/>
-       <origin xyz="0.0 0.0 0" rpy="0 0 0" />
-       <inertia ixx="0.001"  ixy="0"  ixz="0" iyy="0.001" iyz="0" izz="0.001" />
-    </xacro:my_link>
-    <!--the left finger tip -->
-    <xacro:my_link name="finger2_tip_${whichside}" mass="0.01" color="Black">
-       <box size="0.018 0.018 0.06"/>
-       <origin xyz="0.0 0.0 -0.03" rpy="0 0 0"/>
-       <origin xyz="0.0 0.0 -0.03" rpy="0 0 0" />
-       <inertia ixx="0.00037"  ixy="0"  ixz="0" iyy="0.00052" iyz="0" izz="0.00052" />
-    </xacro:my_link>
-    <!--the left finger tip phalanx-->
-    <xacro:my_link name="finger2_tip_phalanx_${whichside}" mass="0.01" color="White">
-       <cylinder length="0.017" radius="0.009"/>
-       <origin xyz="0.0 0.0 0" rpy="0 0 0"/>
-       <origin xyz="0.0 0.0 0" rpy="0 0 0" />
-       <inertia ixx="0.001"  ixy="0"  ixz="0" iyy="0.001" iyz="0" izz="0.001" />
-    </xacro:my_link>
-    <!--the grippoint
-    note: not visible, purely kinematic-->
-    <xacro:my_link name="grippoint_${whichside}" mass="0.01" color="Blue">
-       <box size="0.0 0.0 0.0"/>
-       <origin xyz="-0.1 0.0 0.0" rpy="0 0 0"/>
-       <origin xyz="-0.1 0.0 0.0" rpy="0 0 0 " />
-       <inertia ixx="0.0001"  ixy="0"  ixz="0" iyy="0.0001" iyz="0" izz="0.0001" />
-    </xacro:my_link>
-    <!--the joints start here-->
-      <joint name="shoulder_mount_joint_${whichside}" type="fixed">
-        <parent link="trunk"/>
-        <child link="shoulder_mount_${whichside}"/>
-        <origin xyz="0.470 ${sidesign*-0.22} 0.0" rpy="3.14 0 0.0"/><!-- Check length -->
-      </joint>
-    <xacro:my_joint name="shoulder_yaw_joint_${whichside}" type="revolute" parent="shoulder_mount_${whichside}" child="shoulder_link1_${whichside}">
-       <origin xyz="0 0 0" rpy="-1.5708 -1.5708 0"/>
-       <dynamics damping="4.0" friction="4.87"/>
-       <axis xyz="${rollsign}1 0 0"/>
-       <limit effort="13.4" velocity="1.0" lower="-1.57" upper="0.0" />
-    </xacro:my_joint>
-    <xacro:my_joint name="shoulder_pitch_joint_${whichside}" type="revolute" parent="shoulder_link1_${whichside}" child="shoulder_link2_${whichside}">
-       <origin xyz="0.0 0.0 0.0" rpy="-1.5708  0 0"/>
-       <dynamics damping="4.0" friction="6.06"/>
-       <axis xyz="0 -1 0"/>
-       <limit effort="13.4" velocity="1.0" lower="-1.57" upper="1.57" />
-    </xacro:my_joint>
-    <xacro:my_joint name="shoulder_roll_joint_${whichside}" type="revolute" parent="shoulder_link2_${whichside}" child="upper_arm_${whichside}">
-       <origin xyz="0.0 0.0 0.0" rpy="1.5708 0 0.0"/>
-       <dynamics damping="3.8" friction="2.216"/>
-       <axis xyz="0 ${sidesign} 0"/>
-       <limit effort="9.8" velocity="1.0" lower="-1.57" upper="1.57"/>
-    </xacro:my_joint>
-    <xacro:my_joint name="elbow_pitch_joint_${whichside}" type="revolute" parent="upper_arm_${whichside}" child="elbow_link4_${whichside}">
-       <origin xyz="0.01 -0.32 0.0" rpy="-1.5708 0 0"/>
-       <dynamics damping="3" friction="1.18"/>
-       <axis xyz="0 -1 0"/>
-       <limit effort="4.5" velocity="1.0" lower="0.0" upper="2.23" />
-    </xacro:my_joint>
-    <xacro:my_joint name="elbow_roll_joint_${whichside}" type="revolute" parent="elbow_link4_${whichside}" child="fore_arm_${whichside}">
-       <origin xyz="0.0 0.0 0.0" rpy="1.5708 0 0"/>
-       <dynamics damping="3.5" friction="1.35"/>
-       <axis xyz="0 ${sidesign} 0"/>
-       <limit effort="4.5" velocity="1.0" lower="-1.83" upper="1.83"/>
-    </xacro:my_joint>
-    <xacro:my_joint name="wrist_pitch_joint_${whichside}" type="revolute" parent="fore_arm_${whichside}" child="wrist_link6_${whichside}">
-       <origin xyz="0.01 -0.28 0.0" rpy="-1.5708 0 -1.5708"/>
-       <dynamics damping="0.35" friction="0.63"/>
-       <axis xyz="0 -1 0"/>
-       <limit effort="1" velocity="1.0" lower="-0.95" upper="0.95"/>
-    </xacro:my_joint>
-    <xacro:my_joint name="wrist_yaw_joint_${whichside}" type="revolute" parent="wrist_link6_${whichside}" child="hand_${whichside}">
-       <origin xyz="0.0 0.0 0.0" rpy="0 0 0"/>
-       <dynamics damping="0.3" friction="0.68"/>
-       <axis xyz="0 0 ${sidesign}1"/>
-       <limit effort="1" velocity="1.0" lower="-0.61" upper="0.61"/>
-    </xacro:my_joint>
-    <xacro:my_joint name="finger1_joint_${whichside}" type="revolute" parent="hand_${whichside}" child="finger1_${whichside}">
-       <origin xyz=" 0.075 0.02 0" rpy="0 -1.57 0"/>
-       <dynamics damping="0.5" friction="1.0"/>
-       <axis xyz="1 0 0"/>
-       <limit effort="3" velocity="1.0" lower="-1.57" upper="1.57"/>
-    </xacro:my_joint>
-    <joint name="finger1_phalanx_joint_${whichside}" type="fixed">
-        <parent link="finger1_${whichside}"/>
-        <child link="finger1_phalanx_${whichside}"/>
-        <origin xyz="0 0 -0.06" rpy="0 1.57 0"/>
-    </joint>
-    <xacro:my_joint name="finger1_tip_joint_${whichside}" type="revolute" parent="finger1_${whichside}" child="finger1_tip_${whichside}">
-       <origin xyz=" 0 0.0 -0.06" rpy="0 0 0"/>
-       <dynamics damping="0.5" friction="1.0"/>
-       <axis xyz="1 0 0"/>
-       <limit effort="3" velocity="1.0" lower="-1.57" upper="1.57"/>
-    </xacro:my_joint>
-    <joint name="finger1_tip_phalanx_joint_${whichside}" type="fixed">
-        <parent link="finger1_tip_${whichside}"/>
-        <child link="finger1_tip_phalanx_${whichside}"/>
-        <origin xyz="0 0 -0.06" rpy="0 1.57 0"/>
-    </joint>
-    <xacro:my_joint name="finger2_joint_${whichside}" type="revolute" parent="hand_${whichside}" child="finger2_${whichside}">
-       <origin xyz="0.075 -0.02 0" rpy="0 -1.57 0"/>
-       <dynamics damping="0.5" friction="1.0"/>
-       <axis xyz="-1 0 0"/>
-       <limit effort="3" velocity="1.0" lower="-1.57" upper="1.57"/>
-    </xacro:my_joint>
-    <joint name="finger2_phalanx_joint_${whichside}" type="fixed">
-        <parent link="finger2_${whichside}"/>
-        <child link="finger2_phalanx_${whichside}"/>
-        <origin xyz="0 0 -0.06" rpy="0 1.57 0"/>
-    </joint>
-    <xacro:my_joint name="finger2_tip_joint_${whichside}" type="revolute" parent="finger2_${whichside}" child="finger2_tip_${whichside}">
-       <origin xyz="0 0 -0.06" rpy="0 0 0"/>
-       <dynamics damping="0.5" friction="1.0"/>
-       <axis xyz="-1 0 0"/>
-       <limit effort="3" velocity="1.0" lower="-1.57" upper="1.57"/>
-    </xacro:my_joint>
-    <joint name="finger2_tip_phalanx_joint_${whichside}" type="fixed">
-        <parent link="finger2_tip_${whichside}"/>
-        <child link="finger2_tip_phalanx_${whichside}"/>
-        <origin xyz="0 0 -0.06" rpy="0 1.57 0"/>
-    </joint>
-    <joint name="grippoint_joint_${whichside}" type="fixed">
-      <parent link="hand_${whichside}"/>
-      <child link="grippoint_${whichside}"/>
-      <origin xyz="0.14 0.0 0.0" rpy="0 0 0"/>
-    </joint>
+<robot 	xmlns:xacro="http://ros.org/wiki/xacro"
+	xmlns:sensor="http://playerstage.sourceforge.net/gazebo/xmlschema/#sensor"
+	xmlns:controller="http://playerstage.sourceforge.net/gazebo/xmlschema/#controller"
+	xmlns:interface="http://playerstage.sourceforge.net/gazebo/xmlschema/#interface">
+	<author>Rob Janssen, Kris van Tienhoven, Janno Lunenburg</author>
+   <license>BSD</license>
+   <review status="unreviewed" notes=""/>
+<!--Start of the macro
+@param whichside is "left"  or "right"
+@param sidesign is -1 or +1
+@param rollsign is - or +
+The reason sidesign is -1 or +1 and not just - or + aswell is because
+it has to be reversable and xml cannot multiply - or + but can multiply
+ -1 and +1-->
+ <xacro:macro name="arm" params="whichside sidesign rollsign">
+<!--the end of the clavicle, yaw rotation-->
+<xacro:my_link name="shoulder_mount_${whichside}" mass="0.15" color="White">
+   <cylinder radius="0.075" length="0.190" /><!-- Length of tube should be correct (see report), origin depends on placement -->
+   <origin xyz="0.0 ${sidesign*-0.155} 0.0" rpy="1.57 0 0"/>
+   <origin xyz="0.0 ${sidesign*-0.155} 0.0" rpy="1.57 0 0 " />
+   <inertia ixx="0.01"  ixy="0"  ixz="0" iyy="0.01" iyz="0" izz="0.01" /> <!-- 0.45993-->
+</xacro:my_link>
+<!-- ${sidesign*-0.155} -->
+<!--the cylinder on the end of the clavicle, pitch rotation-->
+<xacro:my_link name="shoulder_link1_${whichside}" mass="0.25" color="Black">
+   <cylinder radius="0.045" length="0.015" />
+   <origin xyz="0.0 0.0 0.0" rpy="0 0 0"/>
+   <origin xyz="0.0 0.0 ${sidesign *0.0525}" rpy="0 0 0 " />
+   <inertia ixx="6.0"  ixy="0"  ixz="0" iyy="0.01" iyz="0" izz="0.01" />
+</xacro:my_link>
+<!--the box that connects the clavicle to the upper arm, roll rotation-->
+<xacro:my_link name="shoulder_link2_${whichside}" mass="0.15" color="Black">
+   <box size="0.035 0.01 0.1" />
+   <origin xyz="0.0 0.0 0.0" rpy="0 0 0"/>
+   <origin xyz="0.0 ${-sidesign*0.06} -0.05" rpy="0 0 0" />
+   <inertia ixx="0.01"  ixy="0"  ixz="0" iyy="4.04" iyz="0" izz="0.001" />
+</xacro:my_link>
+<!--the upper arm-->
+<xacro:my_link_texturedmesh name="upper_arm_${whichside}" mass="2.95" texture="white">
+   <origin xyz="0.0 -0.2 0.0" rpy="0 0 0"/>
+   <origin xyz="-0.00959 -0.19131 -0.00001" rpy="0 0 3.1415" />
+   <inertia ixx="0.027"  ixy="0"  ixz="0" iyy="0.45993" iyz="0" izz="0.004" />
+   <mesh filename="package://sergio_description/media/meshes/upperarmtextured.dae" scale="0.0004 0.0004 0.0004"/>
+</xacro:my_link_texturedmesh>
+<!--the elbow
+note: not visible, see arm_extra_visuals for the elbow visuals -->
+<xacro:my_link name="elbow_link4_${whichside}" mass="0.1" color="Grey">
+   <cylinder radius="0.0" length="0.0"/>
+   <origin xyz="0.0 0.0 0.0" rpy="0 0 0"/>
+   <origin xyz="0.0 0.0 0.0" rpy="0 0 0" />
+   <inertia ixx="0.001"  ixy="0"  ixz="0" iyy="0.6" iyz="0" izz="0.001" />
+</xacro:my_link>
+<!--the forearm-->
+<xacro:my_link_texturedmesh name="fore_arm_${whichside}" mass="0.85" texture="white">
+   <origin xyz="0.0 -0.14 0.0" rpy="0.0 0 0"/>
+   <origin xyz="0.00425 -0.14868 0.00547" rpy="0 -1.5708 0" />
+   <inertia ixx="0.001"  ixy="0"  ixz="0" iyy="0.5" iyz="0" izz="0.001" />
+   <mesh filename="package://sergio_description/media/meshes/forearmtextured.dae" scale="0.0004 0.0004 0.0004"/>
+</xacro:my_link_texturedmesh>
+<!--the wrist
+note: not visible, see arm_extra_visuals for the wrist visuals -->
+<xacro:my_link name="wrist_link6_${whichside}" mass="0.01" color="Black">
+   <cylinder radius="0.0" length="0.0"/>
+   <origin xyz="0.0 0.0 0.0" rpy="0 0 0"/>
+   <origin xyz="0.0 0.0 0.0" rpy="1.5708 0 0" />
+   <inertia ixx="0.001"  ixy="0"  ixz="0" iyy="0.03322" iyz="0" izz="0.001" />
+</xacro:my_link>
+<!--the hand -->
+<xacro:my_link name="hand_${whichside}" mass="0.20" color="Grey">
+   <box size="0.080 0.085 0.038"/>
+   <origin xyz="0.048 0.0 0.0" rpy="0 0 0"/>
+   <origin xyz="0.048 0.0 0.0" rpy="0 0 0" />
+   <inertia ixx="0.01"  ixy="0"  ixz="0" iyy="0.01" iyz="0" izz="0.0622" />
+</xacro:my_link>
+<!--the right finger-->
+<xacro:my_link name="finger1_${whichside}" mass="0.01" color="Black">
+   <box size="0.018 0.018 0.06"/>
+   <origin xyz="0.0 0.0 -0.03" rpy="0 0 0"/>
+   <origin xyz="0.0 0.0 -0.03" rpy="0 0 0" />
+   <inertia ixx="0.01"  ixy="0"  ixz="0" iyy="0.01" iyz="0" izz="0.01" />
+</xacro:my_link>
+<gazebo reference="finger1_${whichside}">
+  <mu1 value="100.0" />
+  <mu2 value="100.0" />
+</gazebo>
+<!--the right finger phalanx-->
+<xacro:my_link name="finger1_phalanx_${whichside}" mass="0.01" color="White">
+   <cylinder length="0.019" radius="0.009"/>
+   <origin xyz="0.0 0.0 0" rpy="0 0 0"/>
+   <origin xyz="0.0 0.0 0" rpy="0 0 0" />
+   <inertia ixx="0.001"  ixy="0"  ixz="0" iyy="0.001" iyz="0" izz="0.001" />
+</xacro:my_link>
+<!--the right finger tip-->
+<xacro:my_link name="finger1_tip_${whichside}" mass="0.01" color="Black">
+   <box size="0.018 0.018 0.06"/>
+   <origin xyz="0.0 0.0 -0.03" rpy="0 0 0"/>
+   <origin xyz="0.0 0.0 -0.03" rpy="0 0 0" />
+   <inertia ixx="0.00037"  ixy="0"  ixz="0" iyy="0.00052" iyz="0" izz="0.00052" />
+</xacro:my_link>
+<gazebo reference="finger1_tip_${whichside}">
+  <mu1 value="100.0" />
+  <mu2 value="100.0" />
+</gazebo>
+<!--the right finger tip phalanx-->
+<xacro:my_link name="finger1_tip_phalanx_${whichside}" mass="0.01" color="White">
+   <cylinder length="0.017" radius="0.009"/>
+   <origin xyz="0.0 0.0 0" rpy="0 0 0"/>
+   <origin xyz="0.0 0.0 0" rpy="0 0 0" />
+   <inertia ixx="0.001"  ixy="0"  ixz="0" iyy="0.001" iyz="0" izz="0.001" />
+</xacro:my_link>
+<!--the left finger-->
+<xacro:my_link name="finger2_${whichside}" mass="0.01" color="Black">
+   <box size="0.018 0.018 0.06"/>
+   <origin xyz="0.0 0.0 -0.03" rpy="0 0 0"/>
+   <origin xyz="0.0 0.0 -0.03" rpy="0 0 0" />
+   <inertia ixx="0.01"  ixy="0"  ixz="0" iyy="0.01" iyz="0" izz="0.01" />
+</xacro:my_link>
+<gazebo reference="finger2_${whichside}">
+  <mu1 value="100.0" />
+  <mu2 value="100.0" />
+</gazebo>
+<!--the left finger phalanx-->
+<xacro:my_link name="finger2_phalanx_${whichside}" mass="0.01" color="White">
+   <cylinder length="0.019" radius="0.009"/>
+   <origin xyz="0.0 0.0 0" rpy="0 0 0"/>
+   <origin xyz="0.0 0.0 0" rpy="0 0 0" />
+   <inertia ixx="0.001"  ixy="0"  ixz="0" iyy="0.001" iyz="0" izz="0.001" />
+</xacro:my_link>
+<!--the left finger tip -->
+<xacro:my_link name="finger2_tip_${whichside}" mass="0.01" color="Black">
+   <box size="0.018 0.018 0.06"/>
+   <origin xyz="0.0 0.0 -0.03" rpy="0 0 0"/>
+   <origin xyz="0.0 0.0 -0.03" rpy="0 0 0" />
+   <inertia ixx="0.00037"  ixy="0"  ixz="0" iyy="0.00052" iyz="0" izz="0.00052" />
+</xacro:my_link>
+<gazebo reference="finger2_tip_${whichside}">
+  <mu1 value="100.0" />
+  <mu2 value="100.0" />
+</gazebo>
+<!--the left finger tip phalanx-->
+<xacro:my_link name="finger2_tip_phalanx_${whichside}" mass="0.01" color="White">
+   <cylinder length="0.017" radius="0.009"/>
+   <origin xyz="0.0 0.0 0" rpy="0 0 0"/>
+   <origin xyz="0.0 0.0 0" rpy="0 0 0" />
+   <inertia ixx="0.001"  ixy="0"  ixz="0" iyy="0.001" iyz="0" izz="0.001" />
+</xacro:my_link>
+<!--the grippoint
+note: not visible, purely kinematic-->
+<xacro:my_link name="grippoint_${whichside}" mass="0.01" color="Blue">
+   <box size="0.0 0.0 0.0"/>
+   <origin xyz="-0.1 0.0 0.0" rpy="0 0 0"/>
+   <origin xyz="-0.1 0.0 0.0" rpy="0 0 0 " />
+   <inertia ixx="0.0001"  ixy="0"  ixz="0" iyy="0.0001" iyz="0" izz="0.0001" />
+</xacro:my_link>
+<!--the joints start here-->
+  <joint name="shoulder_mount_joint_${whichside}" type="fixed">
+    <parent link="trunk"/>
+    <child link="shoulder_mount_${whichside}"/>
+    <origin xyz="0.470 ${sidesign*-0.22} 0.0" rpy="3.14 0 0.0"/><!-- Check length -->
+  </joint>
+<xacro:my_joint name="shoulder_yaw_joint_${whichside}" type="revolute" parent="shoulder_mount_${whichside}" child="shoulder_link1_${whichside}">
+   <origin xyz="0 0 0" rpy="-1.5708 -1.5708 0"/>
+   <dynamics damping="4.0" friction="4.87"/>
+   <axis xyz="${rollsign}1 0 0"/>
+   <limit effort="0.2" velocity="0.4" lower="-1.57" upper="0.0" />
+</xacro:my_joint>
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
File: urdf/arms/arm_extra.urdf.xacro (robot description, xacro)
@@ -13,7 +13,7 @@
 <xacro:macro name="arm_extra" params="whichside sidesign rollsign">
 <xacro:my_link name="pitch_axis_${whichside}" mass="0.15" color="White">
-   <cylinder radius="0.035" length="0.220" /><!-- Length of tube should be correct (see report), origin depends on placement -->
-   <origin xyz="0.0 ${sidesign*-0.055} 0.0" rpy="1.57 0 0"/>
-   <origin xyz="0.0 ${sidesign*-0.055} 0.0" rpy="1.57 0 0 " />
+   <cylinder radius="0.035" length="0.11" /><!-- Length of tube should be correct (see report), origin depends on placement -->
+   <origin xyz="0.0 ${sidesign*-0.01} 0.0" rpy="1.57 0 0"/>
+   <origin xyz="0.0 ${sidesign*-0.01} 0.0" rpy="1.57 0 0 " />
    <inertia ixx="0.01"  ixy="0"  ixz="0" iyy="0.01" iyz="0" izz="0.01" /> <!-- 0.45993-->
 </xacro:my_link>

File: urdf/base/base.urdf.xacro (robot description, xacro)
@@ -22,5 +22,5 @@
     </xacro:my_link_texturedmesh>
     <!--base block-->
-    <xacro:my_link name="base_block" mass="0.1" color="White"><!--ToDo: estimate mass-->
+    <xacro:my_link name="base_block" mass="0.1" color="Black"><!--ToDo: estimate mass-->
         <!-- Large box for better self-filtering -->
         <box size="0.68 0.45 0.11" />
