Commit message: Add extra arm visuals

File: urdf/sergio.urdf.xacro (robot description, xacro)
@@ -19,6 +19,10 @@
     <!--========BUILD ARMS======-->
     <xacro:include filename="$(find sergio_description)/urdf/arms/arm.urdf.xacro" />
-    <xacro:arm whichside="right" sidesign="1" rollsign="+"/>
-    <xacro:arm whichside="left"  sidesign="-1" rollsign="-"/>
+    <xacro:arm whichside="right" sidesign="1.0" rollsign="+"/>
+    <xacro:arm whichside="left"  sidesign="-1.0" rollsign="-"/>
+    <!--extra arm visuals-->
+    <xacro:include filename="$(find sergio_description)/urdf/arms/arm_extra.urdf.xacro" />
+    <xacro:arm_extra whichside="right" sidesign="1.0" rollsign="+"/>
+    <xacro:arm_extra whichside="left"  sidesign="-1.0" rollsign="-"/>
     <!--========BUILD HEAD======-->
     <xacro:include filename="$(find sergio_description)/urdf/head/head.urdf.xacro" />

Commit message: Fix loading sergio in gazebo

File: urdf/arms/arm.urdf.xacro (robot description, xacro)
@@ -46,10 +46,11 @@
     <!--the elbow
     note: not visible, see arm_extra_visuals for the elbow visuals -->
-    <xacro:my_link name="elbow_link4_${whichside}" mass="0.1" color="Grey">
-       <cylinder radius="0.0" length="0.0"/>
-       <origin xyz="0.0 0.0 0.0" rpy="0 0 0"/>
-       <origin xyz="0.0 0.0 0.0" rpy="0 0 0" />
-       <inertia ixx="0.001"  ixy="0"  ixz="0" iyy="0.6" iyz="0" izz="0.001" />
-    </xacro:my_link>
+    <link name="elbow_link4_${whichside}">
+      <inertial>
+        <origin rpy="0 0 0" xyz="0.0 0.0 0.0"/>
+        <mass value="0.1"/>
+        <inertia ixx="0.001" ixy="0" ixz="0" iyy="0.6" iyz="0" izz="0.001"/>
+      </inertial>
+    </link>
     <!--the forearm-->
     <xacro:my_link_texturedmesh name="fore_arm_${whichside}" mass="0.85" texture="white">
@@ -61,10 +62,11 @@
     <!--the wrist
     note: not visible, see arm_extra_visuals for the wrist visuals -->
-    <xacro:my_link name="wrist_link6_${whichside}" mass="0.01" color="Black">
-       <cylinder radius="0.0" length="0.0"/>
-       <origin xyz="0.0 0.0 0.0" rpy="0 0 0"/>
-       <origin xyz="0.0 0.0 0.0" rpy="1.5708 0 0" />
-       <inertia ixx="0.001"  ixy="0"  ixz="0" iyy="0.03322" iyz="0" izz="0.001" />
-    </xacro:my_link>
+    <link name="wrist_link6_${whichside}">
+      <inertial>
+        <origin rpy="0 0 0" xyz="0.0 0.0 0.0"/>
+        <mass value="0.01"/>
+        <inertia ixx="0.001" ixy="0" ixz="0" iyy="0.03322" iyz="0" izz="0.001"/>
+      </inertial>
+    </link>
     <!--the hand -->
     <xacro:my_link name="hand_${whichside}" mass="0.20" color="Grey">
@@ -148,10 +150,11 @@
     <!--the grippoint
     note: not visible, purely kinematic-->
-    <xacro:my_link name="grippoint_${whichside}" mass="0.01" color="Blue">
-       <box size="0.0 0.0 0.0"/>
-       <origin xyz="-0.1 0.0 0.0" rpy="0 0 0"/>
-       <origin xyz="-0.1 0.0 0.0" rpy="0 0 0 " />
-       <inertia ixx="0.0001"  ixy="0"  ixz="0" iyy="0.0001" iyz="0" izz="0.0001" />
-    </xacro:my_link>
+    <link name="grippoint_${whichside}">
+      <inertial>
+        <origin rpy="0 0 0" xyz="-0.1 0.0 0.0"/>
+        <mass value="0.01"/>
+        <inertia ixx="0.0001" ixy="0" ixz="0" iyy="0.0001" iyz="0" izz="0.0001"/>
+      </inertial>
+    </link>
     <!--the joints start here-->
       <joint name="shoulder_mount_joint_${whichside}" type="fixed">

File: urdf/base/base.urdf.xacro (robot description, xacro)
@@ -5,10 +5,11 @@
     <review status="unreviewed" notes=""/>
     <!--the root of the tf-tree, because it serves only this function it has no visuals-->
-    <xacro:my_link name="base_link" mass="0" color="White">
-       <cylinder radius="0.0" length="0.00" />
-       <origin xyz="0.0 0.0 0.0" rpy="0 0 0"/>
-       <origin xyz="0.0 0.0 0.0" rpy="0 0 0" />
-       <inertia ixx="0"  ixy="0"  ixz="0" iyy="0" iyz="0" izz="0" />
-    </xacro:my_link>
+    <link name="base_link">
+      <inertial>
+        <origin rpy="0 0 0" xyz="0.0 0.0 0.0"/>
+        <mass value="0"/>
+        <inertia ixx="0" ixy="0" ixz="0" iyy="0" iyz="0" izz="0"/>
+      </inertial>
+    </link>
     <!--the base-->
     <xacro:my_link_texturedmesh name="base" mass="0.1" texture="white">
@@ -43,10 +44,11 @@
     </xacro:my_link>
     <!-- base - torso interface -->
-    <xacro:my_link name="base_torso_mount" mass="0" color="White">
-       <cylinder radius="0.0" length="0.00" />
-       <origin xyz="0.0 0.0 0.0" rpy="0 0 0"/>
-       <origin xyz="0.0 0.0 0.0" rpy="0 0 0" />
-       <inertia ixx="0"  ixy="0"  ixz="0" iyy="0" iyz="0" izz="0" />
-    </xacro:my_link>
+    <link name="base_torso_mount">
+      <inertial>
+        <origin rpy="0 0 0" xyz="0.0 0.0 0.0"/>
+        <mass value="0"/>
+        <inertia ixx="0" ixy="0" ixz="0" iyy="0" iyz="0" izz="0"/>
+      </inertial>
+    </link>
     <!-- base - laser interface -->
     <xacro:my_link name="laser_mount" mass="0.01" color="White">

File: urdf/torso/torso.urdf.xacro (robot description, xacro)
@@ -60,10 +60,11 @@
     </xacro:my_link>-->
     <!-- torso laser joint (center is the center of rotation of the laser)-->
-    <xacro:my_link name="torso_laser_mount" mass="0.01" color="Black">
-        <box size="0.0 0.0 0.0" />
-        <origin xyz="0.0 0.0 0.0" rpy="0 0 0"/>
-        <origin xyz="0.0 0.0 0.0" rpy="0 0 0" />
-        <inertia ixx="0.0001"  ixy="0"  ixz="0" iyy="0.0001" iyz="0" izz="0.0001" />
-    </xacro:my_link>
+    <link name="torso_laser_mount">
+      <inertial>
+        <origin rpy="0 0 0" xyz="0.0 0.0 0.0"/>
+        <mass value="0.01"/>
+        <inertia ixx="0.0001" ixy="0" ixz="0" iyy="0.0001" iyz="0" izz="0.0001"/>
+      </inertial>
+    </link>
     <!-- Matrix creator -->
     <link name="matrix">

Commit message: Fix loading sergio in gazebo

File: urdf/arms/arm.urdf.xacro (robot description, xacro)
@@ -43,10 +43,11 @@
     <!--the elbow
     note: not visible, see arm_extra_visuals for the elbow visuals -->
-    <xacro:my_link name="elbow_link4_${whichside}" mass="0.1" color="Grey">
-       <cylinder radius="0.0" length="0.0"/>
-       <origin xyz="0.0 0.0 0.0" rpy="0 0 0"/>
-       <origin xyz="0.0 0.0 0.0" rpy="0 0 0" />
-       <inertia ixx="0.001"  ixy="0"  ixz="0" iyy="0.6" iyz="0" izz="0.001" />
-    </xacro:my_link>
+    <link name="elbow_link4_${whichside}">
+      <inertial>
+        <origin rpy="0 0 0" xyz="0.0 0.0 0.0"/>
+        <mass value="0.1"/>
+        <inertia ixx="0.001" ixy="0" ixz="0" iyy="0.6" iyz="0" izz="0.001"/>
+      </inertial>
+    </link>
     <!--the forearm-->
     <xacro:my_link_texturedmesh name="fore_arm_${whichside}" mass="0.85" texture="white">
@@ -58,10 +59,11 @@
     <!--the wrist
     note: not visible, see arm_extra_visuals for the wrist visuals -->
-    <xacro:my_link name="wrist_link6_${whichside}" mass="0.01" color="Black">
-       <cylinder radius="0.0" length="0.0"/>
-       <origin xyz="0.0 0.0 0.0" rpy="0 0 0"/>
-       <origin xyz="0.0 0.0 0.0" rpy="1.5708 0 0" />
-       <inertia ixx="0.001"  ixy="0"  ixz="0" iyy="0.03322" iyz="0" izz="0.001" />
-    </xacro:my_link>
+    <link name="wrist_link6_${whichside}">
+      <inertial>
+        <origin rpy="0 0 0" xyz="0.0 0.0 0.0"/>
+        <mass value="0.01"/>
+        <inertia ixx="0.001" ixy="0" ixz="0" iyy="0.03322" iyz="0" izz="0.001"/>
+      </inertial>
+    </link>
     <!--the hand -->
     <xacro:my_link name="hand_${whichside}" mass="0.20" color="Grey">
@@ -129,10 +131,11 @@
     <!--the grippoint
     note: not visible, purely kinematic-->
-    <xacro:my_link name="grippoint_${whichside}" mass="0.01" color="Blue">
-       <box size="0.0 0.0 0.0"/>
-       <origin xyz="-0.1 0.0 0.0" rpy="0 0 0"/>
-       <origin xyz="-0.1 0.0 0.0" rpy="0 0 0 " />
-       <inertia ixx="0.0001"  ixy="0"  ixz="0" iyy="0.0001" iyz="0" izz="0.0001" />
-    </xacro:my_link>
+    <link name="grippoint_${whichside}">
+      <inertial>
+        <origin rpy="0 0 0" xyz="-0.1 0.0 0.0"/>
+        <mass value="0.01"/>
+        <inertia ixx="0.0001" ixy="0" ixz="0" iyy="0.0001" iyz="0" izz="0.0001"/>
+      </inertial>
+    </link>
     <!--the joints start here-->
       <joint name="shoulder_mount_joint_${whichside}" type="fixed">

File: urdf/base/base.urdf.xacro (robot description, xacro)
@@ -4,11 +4,11 @@
     <license>BSD</license>
     <review status="unreviewed" notes=""/>
-    <!--the root of the tf-tree, because it serves only this function it has no visuals-->
-    <xacro:my_link name="base_link" mass="0" color="White">
-       <cylinder radius="0.0" length="0.00" />
-       <origin xyz="0.0 0.0 0.0" rpy="0 0 0"/>
-       <origin xyz="0.0 0.0 0.0" rpy="0 0 0" />
-       <inertia ixx="0"  ixy="0"  ixz="0" iyy="0" iyz="0" izz="0" />
-    </xacro:my_link>
+    <link name="base_link">
+      <inertial>
+        <origin rpy="0 0 0" xyz="0.0 0.0 0.0"/>
+        <mass value="0"/>
+        <inertia ixx="0" ixy="0" ixz="0" iyy="0" iyz="0" izz="0"/>
+      </inertial>
+    </link>
     <!--base block-->
     <xacro:my_link name="base" mass="0.1" color="White"><!--ToDo: estimate mass-->
@@ -40,10 +40,11 @@
     </xacro:my_link>
     <!-- base - torso interface -->
-    <xacro:my_link name="base_torso_mount" mass="0" color="White">
-       <cylinder radius="0.0" length="0.00" />
-       <origin xyz="0.0 0.0 0.0" rpy="0 0 0"/>
-       <origin xyz="0.0 0.0 0.0" rpy="0 0 0" />
-       <inertia ixx="0"  ixy="0"  ixz="0" iyy="0" iyz="0" izz="0" />
-    </xacro:my_link>
+    <link name="base_torso_mount">
+      <inertial>
+        <origin rpy="0 0 0" xyz="0.0 0.0 0.0"/>
+        <mass value="0"/>
+        <inertia ixx="0" ixy="0" ixz="0" iyy="0" iyz="0" izz="0"/>
+      </inertial>
+    </link>
     <!-- base - laser interface -->
     <xacro:my_link name="laser_mount" mass="0.01" color="White">

File: urdf/torso/torso.urdf.xacro (robot description, xacro)
@@ -33,10 +33,11 @@
     </xacro:my_link>
     <!-- torso laser joint (center is the center of rotation of the laser)-->
-    <xacro:my_link name="torso_laser_mount" mass="0.01" color="Black">
-        <box size="0.0 0.0 0.0" />
-        <origin xyz="0.0 0.0 0.0" rpy="0 0 0"/>
-        <origin xyz="0.0 0.0 0.0" rpy="0 0 0" />
-        <inertia ixx="0.0001"  ixy="0"  ixz="0" iyy="0.0001" iyz="0" izz="0.0001" />
-    </xacro:my_link>
+    <link name="torso_laser_mount">
+      <inertial>
+        <origin rpy="0 0 0" xyz="0.0 0.0 0.0"/>
+        <mass value="0.01"/>
+        <inertia ixx="0.0001" ixy="0" ixz="0" iyy="0.0001" iyz="0" izz="0.0001"/>
+      </inertial>
+    </link>
     <!-- Matrix creator -->
     <link name="matrix">
