Commit message: Rebase & squash `cover` branch

File: urdf/arms/arm.urdf.xacro (robot description, xacro)
@@ -1,7 +1,10 @@
 <?xml version="1.0"?>
-<robot 	xmlns:xacro="http://ros.org/wiki/xacro">
-    <author>Rob Janssen, Kris van Tienhoven, Janno Lunenburg</author>
-    <license>BSD</license>
-    <review status="unreviewed" notes=""/>
+<robot 	xmlns:xacro="http://ros.org/wiki/xacro"
+	xmlns:sensor="http://playerstage.sourceforge.net/gazebo/xmlschema/#sensor"
+	xmlns:controller="http://playerstage.sourceforge.net/gazebo/xmlschema/#controller"
+	xmlns:interface="http://playerstage.sourceforge.net/gazebo/xmlschema/#interface">
+	<author>Rob Janssen, Kris van Tienhoven, Janno Lunenburg</author>
+   <license>BSD</license>
+   <review status="unreviewed" notes=""/>
     <!--Start of the macro
     @param whichside is "left"  or "right"
@@ -14,5 +17,5 @@
     <!--the end of the clavicle, yaw rotation-->
     <xacro:my_link name="shoulder_mount_${whichside}" mass="0.15" color="White">
-       <cylinder radius="0.075" length="0.140" /><!-- Length of tube should be correct (see report), origin depends on placement -->
+       <cylinder radius="0.075" length="0.190" /><!-- Length of tube should be correct (see report), origin depends on placement -->
        <origin xyz="0.0 ${sidesign*-0.155} 0.0" rpy="1.57 0 0"/>
        <origin xyz="0.0 ${sidesign*-0.155} 0.0" rpy="1.57 0 0 " />
@@ -78,4 +81,8 @@
        <inertia ixx="0.01"  ixy="0"  ixz="0" iyy="0.01" iyz="0" izz="0.01" />
     </xacro:my_link>
+    <gazebo reference="finger1_${whichside}">
+      <mu1 value="100.0" />
+      <mu2 value="100.0" />
+    </gazebo>
     <!--the right finger phalanx-->
     <xacro:my_link name="finger1_phalanx_${whichside}" mass="0.01" color="White">
@@ -92,4 +99,8 @@
        <inertia ixx="0.00037"  ixy="0"  ixz="0" iyy="0.00052" iyz="0" izz="0.00052" />
     </xacro:my_link>
+    <gazebo reference="finger1_tip_${whichside}">
+      <mu1 value="100.0" />
+      <mu2 value="100.0" />
+    </gazebo>
     <!--the right finger tip phalanx-->
     <xacro:my_link name="finger1_tip_phalanx_${whichside}" mass="0.01" color="White">
@@ -106,4 +117,8 @@
        <inertia ixx="0.01"  ixy="0"  ixz="0" iyy="0.01" iyz="0" izz="0.01" />
     </xacro:my_link>
+    <gazebo reference="finger2_${whichside}">
+      <mu1 value="100.0" />
+      <mu2 value="100.0" />
+    </gazebo>
     <!--the left finger phalanx-->
     <xacro:my_link name="finger2_phalanx_${whichside}" mass="0.01" color="White">
@@ -120,4 +135,8 @@
        <inertia ixx="0.00037"  ixy="0"  ixz="0" iyy="0.00052" iyz="0" izz="0.00052" />
     </xacro:my_link>
+    <gazebo reference="finger2_tip_${whichside}">
+      <mu1 value="100.0" />
+      <mu2 value="100.0" />
+    </gazebo>
     <!--the left finger tip phalanx-->
     <xacro:my_link name="finger2_tip_phalanx_${whichside}" mass="0.01" color="White">
@@ -145,5 +164,5 @@
        <dynamics damping="4.0" friction="4.87"/>
        <axis xyz="${rollsign}1 0 0"/>
-       <limit effort="13.4" velocity="1.0" lower="-1.57" upper="0.0" />
+       <limit effort="0.2" velocity="0.4" lower="-1.57" upper="0.0" />
     </xacro:my_joint>
     <xacro:my_joint name="shoulder_pitch_joint_${whichside}" type="revolute" parent="shoulder_link1_${whichside}" child="shoulder_link2_${whichside}">
@@ -151,5 +170,5 @@
        <dynamics damping="4.0" friction="6.06"/>
        <axis xyz="0 -1 0"/>
-       <limit effort="13.4" velocity="1.0" lower="-1.57" upper="1.57" />
+       <limit effort="0.2" velocity="0.4" lower="-1.57" upper="1.57" />
     </xacro:my_joint>
     <xacro:my_joint name="shoulder_roll_joint_${whichside}" type="revolute" parent="shoulder_link2_${whichside}" child="upper_arm_${whichside}">
@@ -157,5 +176,5 @@
        <dynamics damping="3.8" friction="2.216"/>
        <axis xyz="0 ${sidesign} 0"/>
-       <limit effort="9.8" velocity="1.0" lower="-1.57" upper="1.57"/>
+       <limit effort="0.3" velocity="0.6" lower="-1.57" upper="1.57"/>
     </xacro:my_joint>
     <xacro:my_joint name="elbow_pitch_joint_${whichside}" type="revolute" parent="upper_arm_${whichside}" child="elbow_link4_${whichside}">
@@ -163,5 +182,5 @@
        <dynamics damping="3" friction="1.18"/>
        <axis xyz="0 -1 0"/>
-       <limit effort="4.5" velocity="1.0" lower="0.0" upper="2.23" />
+       <limit effort="0.5" velocity="0.8" lower="0.0" upper="2.23" />
     </xacro:my_joint>
     <xacro:my_joint name="elbow_roll_joint_${whichside}" type="revolute" parent="elbow_link4_${whichside}" child="fore_arm_${whichside}">
@@ -169,5 +188,5 @@
        <dynamics damping="3.5" friction="1.35"/>
        <axis xyz="0 ${sidesign} 0"/>
-       <limit effort="4.5" velocity="1.0" lower="-1.83" upper="1.83"/>
+       <limit effort="0.5" velocity="0.8" lower="-1.83" upper="1.83"/>
     </xacro:my_joint>
     <xacro:my_joint name="wrist_pitch_joint_${whichside}" type="revolute" parent="fore_arm_${whichside}" child="wrist_link6_${whichside}">
@@ -175,5 +194,5 @@
        <dynamics damping="0.35" friction="0.63"/>
        <axis xyz="0 -1 0"/>
-       <limit effort="1" velocity="1.0" lower="-0.95" upper="0.95"/>
+       <limit effort="0.5" velocity="1.0" lower="-0.95" upper="0.95"/>
     </xacro:my_joint>
     <xacro:my_joint name="wrist_yaw_joint_${whichside}" type="revolute" parent="wrist_link6_${whichside}" child="hand_${whichside}">
@@ -181,5 +200,5 @@
        <dynamics damping="0.3" friction="0.68"/>
        <axis xyz="0 0 ${sidesign}1"/>
-       <limit effort="1" velocity="1.0" lower="-0.61" upper="0.61"/>
+       <limit effort="0.5" velocity="1.0" lower="-0.61" upper="0.61"/>
     </xacro:my_joint>
     <xacro:my_joint name="finger1_joint_${whichside}" type="revolute" parent="hand_${whichside}" child="finger1_${whichside}">

File: urdf/base/base.urdf.xacro (robot description, xacro)
@@ -11,30 +11,33 @@
        <inertia ixx="0"  ixy="0"  ixz="0" iyy="0" iyz="0" izz="0" />
     </xacro:my_link>
+    <!--the base-->
+    <xacro:my_link_texturedmesh name="base" mass="0.1" texture="white">
+        <origin xyz="-0.295 0.10 -0.14" rpy="0 0 1.57"/>
+        <origin xyz="-0.295 0.10 -0.14" rpy="0 0 1.57" />
+        <inertia ixx="0.001"  ixy="0"  ixz="0" iyy="0.001" iyz="0" izz="0.001" />
+        <!--<mesh filename="package://sergio_description/media/meshes/Base2_reduced.dae" scale="0.01 0.01 0.01"/>-->
+        <!--<mesh filename="package://sergio_description/media/meshes/Base2_reduced10000.dae" scale="0.01 0.01 0.01"/>-->
+        <!--<mesh filename="package://sergio_description/media/meshes/BaseWithTexture.dae" scale="0.01 0.01 0.01"/>-->
+        <mesh filename="package://sergio_description/media/meshes/Base2.dae" scale="0.01 0.01 0.01"/>
+    </xacro:my_link_texturedmesh>
     <!--base block-->
-    <xacro:my_link name="base" mass="0.1" color="White"><!--ToDo: estimate mass-->
-        <!--box size="0.713 0.500 0.11" /--><!--ToDo: check dimensions, adjust height-->
+    <xacro:my_link name="base_block" mass="0.1" color="Black"><!--ToDo: estimate mass-->
         <!-- Large box for better self-filtering -->
-        <box size="0.73 0.650 0.14" />
-        <origin xyz="-0.02 0.0 -0.015" rpy="0 0 0"/>
-        <origin xyz="-0.02 0.0 -0.015" rpy="0 0 0"/>
+        <box size="0.68 0.45 0.11" />
+        <origin xyz="-0.02 0.0 0.0" rpy="0 0 0"/>
+        <origin xyz="-0.02 0.0 0.0" rpy="0 0 0"/>
         <inertia ixx="0.001"  ixy="0"  ixz="0" iyy="0.001" iyz="0" izz="0.001" /><!--Estimate inertia-->
     </xacro:my_link>
     <!-- side pots -->
     <xacro:my_link name="sidepot_left" mass="0.1" color="White"><!--ToDo: estimate mass-->
-        <box size="0.43 0.165 0.13" /><!--ToDo: check dimensions, adjust height-->
-        <origin xyz="0.0 0.0 0.065" rpy="0 0 0"/>
-        <origin xyz="0.0 0.0 0.065" rpy="0 0 0"/>
+        <box size="0.360 0.0615 0.1" /><!--ToDo: check dimensions, adjust height-->
+        <origin xyz="0.0 0.0 0.0" rpy="0 0 0"/>
+        <origin xyz="0.0 0.0 0.0" rpy="0 0 0"/>
         <inertia ixx="0.001"  ixy="0"  ixz="0" iyy="0.001" iyz="0" izz="0.001" /><!--Estimate inertia-->
     </xacro:my_link>
     <xacro:my_link name="sidepot_right" mass="0.1" color="White"><!--ToDo: estimate mass-->
-        <box size="0.43 0.165 0.13" /><!--ToDo: check dimensions, adjust height-->
-        <origin xyz="0.0 0.0 0.065" rpy="0 0 0"/>
-        <origin xyz="0.0 0.0 0.065" rpy="0 0 0"/>
-        <inertia ixx="0.001"  ixy="0"  ixz="0" iyy="0.001" iyz="0" izz="0.001" /><!--Estimate inertia-->
-    </xacro:my_link>
-    <xacro:my_link name="sidepot_back" mass="0.1" color="White"><!--ToDo: estimate mass-->
-        <box size="0.16 0.65 0.13" /><!--ToDo: check dimensions, adjust height-->
-        <origin xyz="0.0 0.0 0.065" rpy="0 0 0"/>
-        <origin xyz="0.0 0.0 0.065" rpy="0 0 0"/>
+        <box size="0.360 0.0615 0.1" /><!--ToDo: check dimensions, adjust height-->
+        <origin xyz="0.0 0.0 0.0" rpy="0 0 0"/>
+        <origin xyz="0.0 0.0 0.0" rpy="0 0 0"/>
         <inertia ixx="0.001"  ixy="0"  ixz="0" iyy="0.001" iyz="0" izz="0.001" /><!--Estimate inertia-->
     </xacro:my_link>
@@ -60,4 +63,36 @@
        <inertia ixx="0.0001"  ixy="0"  ixz="0" iyy="0.0001" iyz="0" izz="0.0001" />
     </xacro:my_link>
+    <!-- wheels -->
+    <xacro:my_link name="wheel_right_front" mass="0" color="DarkGrey">
+       <cylinder radius="0.075" length="0.055" />
+       <origin xyz="0.0 0.0 0.0" rpy="0.0 0 0"/>
+       <origin xyz="0.0 0.0 0.0" rpy="0.0 0 0" />
+       <inertia ixx="0"  ixy="0"  ixz="0" iyy="0" iyz="0" izz="0" />
+    </xacro:my_link>
+    <xacro:my_link name="wheel_left_front" mass="0" color="DarkGrey">
+       <cylinder radius="0.075" length="0.055" />
+       <origin xyz="0.0 0.0 0.0" rpy="0.0 0 0"/>
+       <origin xyz="0.0 0.0 0.0" rpy="0.0 0 0" />
+       <inertia ixx="0"  ixy="0"  ixz="0" iyy="0" iyz="0" izz="0" />
+    </xacro:my_link>
+    <xacro:my_link name="wheel_right_rear" mass="0" color="DarkGrey">
+       <cylinder radius="0.075" length="0.055" />
+       <origin xyz="0.0 0.0 0.0" rpy="0.0 0 0"/>
+       <origin xyz="0.0 0.0 0.0" rpy="0.0 0 0" />
+       <inertia ixx="0"  ixy="0"  ixz="0" iyy="0" iyz="0" izz="0" />
+    </xacro:my_link>
+    <xacro:my_link name="wheel_left_rear" mass="0" color="DarkGrey">
+       <cylinder radius="0.075" length="0.055" />
+       <origin xyz="0.0 0.0 0.0" rpy="0.0 0 0"/>
+       <origin xyz="0.0 0.0 0.0" rpy="0.0 0 0" />
+       <inertia ixx="0"  ixy="0"  ixz="0" iyy="0" iyz="0" izz="0" />
+    </xacro:my_link>
+    <!-- Batteries -->
+    <xacro:my_link name="batteries" mass="0.1" color="Black"><!--ToDo: estimate mass-->
+        <box size="0.332 0.120 0.1" /><!--ToDo: check dimensions, adjust height-->
+        <origin xyz="0.0 0.0 0.05" rpy="0 0 0"/>
+        <origin xyz="0.0 0.0 0.05" rpy="0 0 0"/>
+        <inertia ixx="0.001"  ixy="0"  ixz="0" iyy="0.001" iyz="0" izz="0.001" /><!--Estimate inertia-->
+    </xacro:my_link>
     <!-- joints -->
     <joint name="base_link_joint" type="fixed">
@@ -67,9 +102,15 @@
         <origin xyz="0.0 0.0 0.085" rpy="0 0 0"/><!--ToDO: adjust height-->
     </joint>
+    <joint name="base_block_joint" type="fixed">
+        <parent link="base"/>
+        <child link="base_block"/>
+        <axis xyz="1 0 0"/>
+        <origin xyz="0.0 0.0 0.0" rpy="0 0 0"/><!--ToDO: adjust height-->
+    </joint>
     <joint name="sidepot_left_joint" type="fixed">
         <parent link="base"/>
         <child link="sidepot_left"/>
         <axis xyz="1 0 0"/>
-        <origin xyz="-0.01 0.2425 0.045" rpy="0 0 0"/><!--ToDO: adjust distance-->
+        <origin xyz="0.0 0.2425 0.045" rpy="0 0 0"/><!--ToDO: adjust distance-->
     </joint>
     <joint name="sidepot_right_joint" type="fixed">
@@ -77,11 +118,5 @@
         <child link="sidepot_right"/>
         <axis xyz="1 0 0"/>
-        <origin xyz="-0.01 -0.2425 0.045" rpy="0 0 0"/><!--ToDO: adjust distance-->
-    </joint>
-    <joint name="sidepot_back_joint" type="fixed">
-        <parent link="base"/>
-        <child link="sidepot_back"/>
-        <axis xyz="1 0 0"/>
-        <origin xyz="-0.305 0.0 0.045" rpy="0 0 0"/><!--ToDO: adjust distance-->
+        <origin xyz="0.0 -0.2425 0.045" rpy="0 0 0"/><!--ToDO: adjust distance-->
     </joint>
     <joint name="base_mount_joint" type="fixed">
@@ -100,3 +135,28 @@
         <origin xyz="-0.293 0.0 0.157" rpy="0.0 0.0 0.0"/>
     </joint>
+    <joint name="wheel_right_front_joint" type="fixed">
+        <parent link="base_link"/>
+        <child link="wheel_right_front"/>
+        <origin xyz="0.265 -0.275 0.075" rpy="1.57 0.0 0.0"/>
+    </joint>
+    <joint name="wheel_left_front_joint" type="fixed">
+        <parent link="base_link"/>
+        <child link="wheel_left_front"/>
+        <origin xyz="0.265 0.275 0.075" rpy="1.57 0.0 0.0"/>
+    </joint>
+    <joint name="wheel_right_rear_joint" type="fixed">
+        <parent link="base_link"/>
+        <child link="wheel_right_rear"/>
+        <origin xyz="-0.265 -0.275 0.075" rpy="1.57 0.0 0.0"/>
+    </joint>
+    <joint name="wheel_left_rear_joint" type="fixed">
+        <parent link="base_link"/>
+        <child link="wheel_left_rear"/>
+        <origin xyz="-0.265 0.275 0.075" rpy="1.57 0.0 0.0"/>
+    </joint>
+    <joint name="battery_joint" type="fixed">
+        <parent link="base"/>
+        <child link="batteries"/>
+        <origin xyz="0.0 0.23 0.055" rpy="0.0 0.0 0.0"/>
+    </joint>
 </robot>

File: urdf/torso/torso.urdf.xacro (robot description, xacro)
@@ -5,5 +5,5 @@
     <review status="unreviewed" notes=""/>
    <!--mounting frame-->
-    <xacro:my_link name="torso_mounting_frame" mass="0.1" color="White"><!--ToDo: estimate mass-->
+    <xacro:my_link name="torso_mounting_frame" mass="0.1" color="Grey"><!--ToDo: estimate mass-->
         <box size="0.500 0.400 0.05" /><!--ToDo: check dimensions, adjust height-->
         <origin xyz="0.0 0.0 0.025" rpy="0 0 0"/>
@@ -12,5 +12,5 @@
     </xacro:my_link>
     <!-- Lower rear leg -->
-    <xacro:my_link name="lower_rear_leg" mass="5" color="White"><!--ToDo: estimate mass-->
+    <xacro:my_link name="lower_rear_leg" mass="5" color="Grey"><!--ToDo: estimate mass-->
         <box size="0.390 0.200 0.05" /><!--ToDo: check dimensions, adjust height-->
         <origin xyz="0.195 0.0 0.0" rpy="0 0 0"/><!--ToDo: check dimensions, adjust height-->
@@ -19,17 +19,44 @@
     </xacro:my_link>
     <!-- Upper leg (part from lower rear leg joint to trunk joint) -->
-    <xacro:my_link name="upper_leg" mass="5" color="White"><!--ToDo: estimate mass-->
-        <box size="0.4115 0.200 0.1" /><!--ToDo: check dimensions, adjust height-->
-        <origin xyz="0.20575 0.0 0.0" rpy="0 0 0"/><!--ToDo: check dimensions, adjust height-->
-        <origin xyz="0.20575 0.0 0.0" rpy="0 0 0"/><!--ToDo: check dimensions, adjust height-->
-        <inertia ixx="0.001"  ixy="0"  ixz="0" iyy="0.001" iyz="0" izz="0.001" /><!--Estimate inertia-->
+    <!--
+    <xacro:my_link name="upper_leg" mass="5" color="White">
+        <box size="0.4115 0.200 0.1" />
+        <origin xyz="0.20575 0.0 0.0" rpy="0 0 0"/>
+        <origin xyz="0.20575 0.0 0.0" rpy="0 0 0"/>
+        <inertia ixx="0.001"  ixy="0"  ixz="0" iyy="0.001" iyz="0" izz="0.001" />
+    </xacro:my_link>-->
+    <xacro:my_link_texturedmesh name="upper_leg" mass="5" texture="white"><!-- ToDo: estimate mass -->
+        <origin xyz="0.41575 -0.10 -0.02" rpy="0 0 1.57"/>
+        <origin xyz="0.41575 -0.10 -0.02" rpy="0 0 1.57"/>
+        <inertia ixx="0.001"  ixy="0"  ixz="0" iyy="0.001" iyz="0" izz="0.001" /><!-- ToDo: estimate mass -->
+        <mesh filename="package://sergio_description/media/meshes/upper_leg_reduced10000.dae" scale="0.01 0.01 0.01"/>
+    </xacro:my_link_texturedmesh>
+    <xacro:my_link name="upper_leg_inside" mass="0.001" color="Black">
+        <box size="0.5115 0.200 0.06" />
+        <origin xyz="0.20 0.0 0.0" rpy="0 0 0"/>
+        <origin xyz="0.20 0.0 0.0" rpy="0 0 0"/>
+        <inertia ixx="0.001"  ixy="0"  ixz="0" iyy="0.001" iyz="0" izz="0.001" />
     </xacro:my_link>
     <!-- Trunk -->
-    <xacro:my_link name="trunk" mass="10" color="White"><!--ToDo: estimate mass-->
-        <box size="0.470 0.200 0.15" /><!--ToDo: check dimensions, adjust height-->
-        <origin xyz="0.235 0.0 0.0" rpy="0 0 0"/><!--ToDo: check dimensions, adjust height-->
-        <origin xyz="0.235 0.0 0.0" rpy="0 0 0"/><!--ToDo: check dimensions, adjust height-->
-        <inertia ixx="0.001"  ixy="0"  ixz="0" iyy="0.001" iyz="0" izz="0.001" /><!--Estimate inertia-->
-    </xacro:my_link>
+    <!--
+    <xacro:my_link name="trunk" mass="10" color="White">
+        <box size="0.470 0.200 0.15" />
+        <origin xyz="0.235 0.0 0.0" rpy="0 0 0"/>
+        <origin xyz="0.235 0.0 0.0" rpy="0 0 0"/>
+        <inertia ixx="0.001"  ixy="0"  ixz="0" iyy="0.001" iyz="0" izz="0.001" />
+    </xacro:my_link>-->
+    <xacro:my_link_texturedmesh name="trunk" mass="10" texture="white"><!-- ToDo: estimate mass -->
+        <origin xyz="0.16 -0.11 0.0" rpy="3.1415 1.73 0"/>
+        <origin xyz="0.16 -0.11 0.0" rpy="3.1415 1.73 0"/>
+        <inertia ixx="0.001"  ixy="0"  ixz="0" iyy="0.001" iyz="0" izz="0.001" /><!-- ToDo: estimate mass -->
+        <!--<mesh filename="package://sergio_description/media/meshes/torso_reduced10000.dae" scale="0.01 0.01 0.01"/>-->
+        <mesh filename="package://sergio_description/media/meshes/torso.dae" scale="0.01 0.01 0.01"/>
+    </xacro:my_link_texturedmesh>
+    <xacro:my_link name="trunk_inside" mass="0.001" color="Black">
+        <box size="0.470 0.200 0.075" />
+        <origin xyz="0.235 0.0 0.0" rpy="0 0 0"/>
+        <origin xyz="0.235 0.0 0.0" rpy="0 0 0"/>
+        <inertia ixx="0.001"  ixy="0"  ixz="0" iyy="0.001" iyz="0" izz="0.001" />
+    </xacro:my_link>-->
     <!-- torso laser joint (center is the center of rotation of the laser)-->
     <xacro:my_link name="torso_laser_mount" mass="0.01" color="Black">
@@ -54,5 +81,5 @@
         <dynamics damping="6.0" friction="4.87"/><!-- ToDo: adjust dynamics-->
         <axis xyz="0 -1 0"/><!--ToDo: DH parameters?-->
-        <limit effort="1000" velocity="0.265" lower="0.152" upper="1.00" /> <!--ToDo: adjust parameters-->
+        <limit effort="0.3" velocity="0.265" lower="0.152" upper="1.00" /> <!--ToDo: adjust parameters-->
         <!--<limit effort="1000" velocity="10" lower="0.87" upper="0.87" />--> <!--TEMP: fixed joint positions until control is fixed-->
     </xacro:my_joint>
@@ -61,14 +88,24 @@
         <dynamics damping="6.0" friction="4.87"/><!-- ToDo: adjust dynamics-->
         <axis xyz="0 -1 0"/><!--ToDo: DH parameters?-->
-        <limit effort="1000" velocity="0.539" lower="0.419" upper="2.059" /> <!--ToDo: adjust parameters -->
+        <limit effort="0.3" velocity="0.539" lower="0.419" upper="2.059" /> <!--ToDo: adjust parameters -->
         <!--<limit effort="1000" velocity="10" lower="2.0" upper="2.0" />--> <!--TEMP: fixed joint positions until control is fixed -->
     </xacro:my_joint>
+    <joint name="upper_leg_inside_joint" type="fixed">
+        <parent link="upper_leg"/>
+        <child link="upper_leg_inside"/>
+        <origin xyz="0.0 0.0 0.0" rpy="0 0 0.0"/>
+    </joint>
     <xacro:my_joint name="hip_joint" type="revolute" parent="upper_leg" child="trunk">
         <origin xyz="0.4115 0.0 0.0" rpy="3.14 3.14 0.0"/><!-- ToDo: adjust height-->
         <dynamics damping="6.0" friction="4.87"/><!-- ToDo: adjust dynamics-->
         <axis xyz="0 -1 0"/><!--ToDo: DH parameters?-->
-        <limit effort="1000" velocity="0.375" lower="1.007" upper="2.31" /> <!--ToDo: adjust parameters --><!--Velocity: move in 4 s-->
+        <limit effort="0.3" velocity="0.375" lower="1.007" upper="2.31" /> <!--ToDo: adjust parameters --><!--Velocity: move in 4 s-->
         <!--<limit effort="1000" velocity="10" lower="2.36" upper="2.36" />--> <!--TEMP: fixed joint positions until control is fixed-->
     </xacro:my_joint>
+    <joint name="trunk_inside_joint" type="fixed">
+        <parent link="trunk"/>
+        <child link="trunk_inside"/>
+        <origin xyz="0.0 0.0 0.0" rpy="0 0 0.0"/>
+    </joint>
     <joint name="laser_tilt_joint" type="revolute" >
         <parent link="trunk" />
